File: ShimbleBoard_Hardware/ShimbleBoard_Hardware.sch (KiCad schematic (older format))
At the start: 14 parts

Commit message: Schematic Finished Draft
Parts:
- removed Conn?: AndersonPP, symbol MRDT_Connectors:AndersonPP
- added C1, C2: 10uF, symbol Device:C
- added Conn8, Conn9: Molex_SL_03, symbol MRDT_Connectors:Molex_SL_03
- gave numbers to parts that had none: 8
Connections:
- net labels added: +5V, GND, Servo_1_Ctrl, Servo_2_Ctrl, Servo_3_Ctrl, Servo_4_Ctrl, Servo_5_Ctrl, Servo_6_Ctrl, Servo_7_Ctrl, Servo_8_Ctrl
- wire segments 0 -> 62
Other:
- note added: "Power Filtering\n"
- note added: "Servo 1"
- note added: "Servo 2"
- note added: "Servo 3"
- note added: "Servo 4"
- note added: "Servo 5"
- note added: "Servo 6"
- note added: "Servo 7"
- note added: "Servo 8"
- note added: "Servo Connectors"
- note added: "TIVA Headers"
- moved on the sheet: Conn1A, Conn1B, Conn2, Conn3, Conn4, Conn5, Conn6, Conn7, U1E, U1F, U1G, U1H

Commit message: Preliminary Board Layout
Parts:
- C1, C2: footprint (none) -> Capacitor_SMD:C_0603_1608Metric_Pad1.05x0.95mm_HandSolder
- Conn1: footprint (none) -> MRDT_Connectors:Anderson_2_Horisontal_Side_by_Side
- Conn2, Conn3, Conn4, Conn5, Conn6, Conn7, Conn8, Conn9: footprint (none) -> MRDT_Connectors:MOLEX_SL_03_Horizontal
- U1: footprint (none) -> MRDT_Shields:TM4C129E_Launchpad_X7
- U2: renamed from U?; footprint (none) -> MRDT_Devices:OKI_Horizontal
Changed lines of the file:
@@
 F 0 "Conn1" H 3650 2200 60  0000 C CNN
 F 1 "AndersonPP" H 3650 2800 60  0000 C CNN
-F 2 "" H 3350 1700 60  0001 C CNN
+F 2 "MRDT_Connectors:Anderson_2_Horisontal_Side_by_Side" H 3350 1700 60  0001 C CNN
 F 3 "" H 3350 1700 60  0001 C CNN
 	1    3500 2250
@@
 F 0 "Conn1" H 3650 1900 60  0000 C CNN
 F 1 "AndersonPP" H 3706 2231 60  0001 C CNN
-F 2 "" H 3350 1400 60  0001 C CNN
+F 2 "MRDT_Connectors:Anderson_2_Horisontal_Side_by_Side" H 3350 1400 60  0001 C CNN
 F 3 "" H 3350 1400 60  0001 C CNN
 	2    3500 1950
@@
 $EndComp
 $Comp
-L MRDT_Devices:OKI U?
+L MRDT_Devices:OKI U2
 U 1 1 5BCBB624
 P 4600 1950
-F 0 "U?" H 4650 1900 60  0001 C CNN
+F 0 "U2" H 4650 1900 60  0001 C CNN
 F 1 "OKI" H 4800 2231 60  0000 C CNN
-F 2 "" H 4400 1850 60  0001 C CNN
+F 2 "MRDT_Devices:OKI_Horizontal" H 4400 1850 60  0001 C CNN
 F 3 "" H 4400 1850 60  0001 C CNN
 	1    4600 1950
@@
 F 0 "U1" H 3400 4300 60  0000 L CNN
 F 1 "TM4C129E_Launchpad" H 3150 5500 60  0000 L CNN
-F 2 "" H 3400 4350 60  0001 C CNN
+F 2 "MRDT_Shields:TM4C129E_Launchpad_X7" H 3400 4350 60  0001 C CNN
 F 3 "" H 3400 4350 60  0001 C CNN
 	5    3400 4350
@@
 F 0 "U1" H 3900 4300 60  0000 L CNN
 F 1 "TM4C129E_Launchpad" H 4205 4842 60  0001 L CNN
-F 2 "" H 3900 4350 60  0001 C CNN
+F 2 "MRDT_Shields:TM4C129E_Launchpad_X7" H 3900 4350 60  0001 C CNN
 F 3 "" H 3900 4350 60  0001 C CNN
 	6    3900 4350
@@
 F 0 "U1" H 3400 5500 60  0000 L CNN
 F 1 "TM4C129E_Launchpad" H 3705 6042 60  0001 L CNN
-F 2 "" H 3400 5550 60  0001 C CNN
+F 2 "MRDT_Shields:TM4C129E_Launchpad_X7" H 3400 5550 60  0001 C CNN
 F 3 "" H 3400 5550 60  0001 C CNN
 	7    3400 5550
@@
 F 0 "U1" H 3900 5500 60  0000 L CNN
 F 1 "TM4C129E_Launchpad" H 4205 6042 60  0001 L CNN
-F 2 "" H 3900 5550 60  0001 C CNN
+F 2 "MRDT_Shields:TM4C129E_Launchpad_X7" H 3900 5550 60  0001 C CNN
 F 3 "" H 3900 5550 60  0001 C CNN
 	8    3900 5550
@@
 F 0 "Conn2" H 6227 3608 60  0000 L CNN
 F 1 "Molex_SL_03" H 6227 3502 60  0000 L CNN
-F 2 "" H 6100 3400 60  0001 C CNN
+F 2 "MRDT_Connectors:MOLEX_SL_03_Horizontal" H 6100 3400 60  0001 C CNN
 F 3 "" H 6100 3400 60  0001 C CNN
 	1    6100 3400
@@
 F 0 "Conn3" H 6227 3958 60  0000 L CNN
 F 1 "Molex_SL_03" H 6227 3852 60  0000 L CNN
-F 2 "" H 6100 3750 60  0001 C CNN
+F 2 "MRDT_Connectors:MOLEX_SL_03_Horizontal" H 6100 3750 60  0001 C CNN
 F 3 "" H 6100 3750 60  0001 C CNN
 	1    6100 3750
@@
 F 0 "Conn4" H 6227 4308 60  0000 L CNN
 F 1 "Molex_SL_03" H 6227 4202 60  0000 L CNN
-F 2 "" H 6100 4100 60  0001 C CNN
+F 2 "MRDT_Connectors:MOLEX_SL_03_Horizontal" H 6100 4100 60  0001 C CNN
 F 3 "" H 6100 4100 60  0001 C CNN
 	1    6100 4100
@@
 F 0 "Conn5" H 6227 4658 60  0000 L CNN
 F 1 "Molex_SL_03" H 6227 4552 60  0000 L CNN
-F 2 "" H 6100 4450 60  0001 C CNN
+F 2 "MRDT_Connectors:MOLEX_SL_03_Horizontal" H 6100 4450 60  0001 C CNN
 F 3 "" H 6100 4450 60  0001 C CNN
 	1    6100 4450
@@
 F 0 "Conn6" H 6227 5008 60  0000 L CNN
 F 1 "Molex_SL_03" H 6227 4902 60  0000 L CNN
-F 2 "" H 6100 4800 60  0001 C CNN
+F 2 "MRDT_Connectors:MOLEX_SL_03_Horizontal" H 6100 4800 60  0001 C CNN
 F 3 "" H 6100 4800 60  0001 C CNN
 	1    6100 4800
@@
 F 0 "Conn7" H 6227 5358 60  0000 L CNN
 F 1 "Molex_SL_03" H 6227 5252 60  0000 L CNN
-F 2 "" H 6100 5150 60  0001 C CNN
+F 2 "MRDT_Connectors:MOLEX_SL_03_Horizontal" H 6100 5150 60  0001 C CNN
 F 3 "" H 6100 5150 60  0001 C CNN
 	1    6100 5150
@@
 $EndComp
 $Comp
-L power:+5V #PWR?
+L power:+5V #PWR0101
 U 1 1 5BCD68E7
 P 5700 1850
-F 0 "#PWR?" H 5700 1700 50  0001 C CNN
+F 0 "#PWR0101" H 5700 1700 50  0001 C CNN
 F 1 "+5V" H 5715 2023 50  0000 C CNN
 F 2 "" H 5700 1850 50  0001 C CNN
@@
 $EndComp
 $Comp
-L power:GND #PWR?
+L power:GND #PWR0102
 U 1 1 5BCD6940
 P 5700 2150
-F 0 "#PWR?" H 5700 1900 50  0001 C CNN
+F 0 "#PWR0102" H 5700 1900 50  0001 C CNN
 F 1 "GND" H 5705 1977 50  0000 C CNN
 F 2 "" H 5700 2150 50  0001 C CNN
@@
 $EndComp
 $Comp
-L power:GND #PWR?
+L power:GND #PWR0103
 U 1 1 5BCD697A
 P 5800 5850
-F 0 "#PWR?" H 5800 5600 50  0001 C CNN
+F 0 "#PWR0103" H 5800 5600 50  0001 C CNN
 F 1 "GND" H 5805 5677 50  0000 C CNN
 F 2 "" H 5800 5850 50  0001 C CNN
@@
 F 0 "C1" H 4315 2046 50  0000 L CNN
 F 1 "10uF" H 4315 1955 50  0000 L CNN
-F 2 "" H 4238 1850 50  0001 C CNN
+F 2 "Capacitor_SMD:C_0603_1608Metric_Pad1.05x0.95mm_HandSolder" H 4238 1850 50  0001 C CNN
 F 3 "~" H 4200 2000 50  0001 C CNN
 	1    4200 2000
@@
 F 0 "C2" H 5515 2046 50  0000 L CNN
 F 1 "10uF" H 5515 1955 50  0000 L CNN
-F 2 "" H 5438 1850 50  0001 C CNN
+F 2 "Capacitor_SMD:C_0603_1608Metric_Pad1.05x0.95mm_HandSolder" H 5438 1850 50  0001 C CNN
 F 3 "~" H 5400 2000 50  0001 C CNN
 	1    5400 2000
@@
 Connection ~ 4200 2150
 $Comp
-L power:+5V #PWR?
+L power:+5V #PWR0104
 U 1 1 5BCDAF51
 P 4250 3400
-F 0 "#PWR?" H 4250 3250 50  0001 C CNN
+F 0 "#PWR0104" H 4250 3250 50  0001 C CNN
 F 1 "+5V" H 4265 3573 50  0000 C CNN
 F 2 "" H 4250 3400 50  0001 C CNN
@@
 $EndComp
 $Comp
-L power:GND #PWR?
+L power:GND #PWR0105
 U 1 1 5BCDB62B
 P 4250 4450
-F 0 "#PWR?" H 4250 4200 50  0001 C CNN
+F 0 "#PWR0105" H 4250 4200 50  0001 C CNN
 F 1 "GND" H 4255 4277 50  0000 C CNN
 F 2 "" H 4250 4450 50  0001 C CNN
@@
 $EndComp
 $Comp
-L power:GND #PWR?
+L power:GND #PWR0106
 U 1 1 5BCDBCE0
 P 4250 3500
-F 0 "#PWR?" H 4250 3250 50  0001 C CNN
+F 0 "#PWR0106" H 4250 3250 50  0001 C CNN
 F 1 "GND" H 4255 3327 50  0000 C CNN
 F 2 "" H 4250 3500 50  0001 C CNN
@@
 F 0 "Conn8" H 6227 5708 60  0000 L CNN
 F 1 "Molex_SL_03" H 6227 5602 60  0000 L CNN
-F 2 "" H 6100 5500 60  0001 C CNN
+F 2 "MRDT_Connectors:MOLEX_SL_03_Horizontal" H 6100 5500 60  0001 C CNN
 F 3 "" H 6100 5500 60  0001 C CNN
 	1    6100 5500
@@
 F 0 "Conn9" H 6227 6058 60  0000 L CNN
 F 1 "Molex_SL_03" H 6227 5952 60  0000 L CNN
-F 2 "" H 6100 5850 60  0001 C CNN
+F 2 "MRDT_Connectors:MOLEX_SL_03_Horizontal" H 6100 5850 60  0001 C CNN
 F 3 "" H 6100 5850 60  0001 C CNN
 	1    6100 5850
@@
 	5700 5250 5700 4900
 $Comp
-L power:+5V #PWR?
+L power:+5V #PWR0107
 U 1 1 5BD1C266
 P 5700 3050
-F 0 "#PWR?" H 5700 2900 50  0001 C CNN
+F 0 "#PWR0107" H 5700 2900 50  0001 C CNN
 F 1 "+5V" H 5715 3223 50  0000 C CNN
 F 2 "" H 5700 3050 50  0001 C CNN

Commit message: fixed board connectors
Parts:
- Conn7, Conn8, Conn9: footprint MRDT_Connectors:MOLEX_SL_03_Horizontal -> MRDT_Connectors:MOLEX_SL_03_Vertical
Changed lines of the file:
@@
 F 0 "Conn7" H 6227 5358 60  0000 L CNN
 F 1 "Molex_SL_03" H 6227 5252 60  0000 L CNN
-F 2 "MRDT_Connectors:MOLEX_SL_03_Horizontal" H 6100 5150 60  0001 C CNN
+F 2 "MRDT_Connectors:MOLEX_SL_03_Vertical" H 6100 5150 60  0001 C CNN
 F 3 "" H 6100 5150 60  0001 C CNN
 	1    6100 5150
@@
 F 0 "Conn8" H 6227 5708 60  0000 L CNN
 F 1 "Molex_SL_03" H 6227 5602 60  0000 L CNN
-F 2 "MRDT_Connectors:MOLEX_SL_03_Horizontal" H 6100 5500 60  0001 C CNN
+F 2 "MRDT_Connectors:MOLEX_SL_03_Vertical" H 6100 5500 60  0001 C CNN
 F 3 "" H 6100 5500 60  0001 C CNN
 	1    6100 5500
@@
 F 0 "Conn9" H 6227 6058 60  0000 L CNN
 F 1 "Molex_SL_03" H 6227 5952 60  0000 L CNN
-F 2 "MRDT_Connectors:MOLEX_SL_03_Horizontal" H 6100 5850 60  0001 C CNN
+F 2 "MRDT_Connectors:MOLEX_SL_03_Vertical" H 6100 5850 60  0001 C CNN
 F 3 "" H 6100 5850 60  0001 C CNN
 	1    6100 5850
