File: ShimbleBoard_Hardware/ShimbleBoard_Hardware.sch (KiCad schematic (older format))
At the start: 13 parts, among them U1 TM4C129E_Launchpad, U2 OKI

Commit message: Removed Servo 8 & Increased Power Track Width
Parts:
- removed Conn9: Molex_SL_03, MRDT_Connectors:MOLEX_SL_03_Horizontal, symbol MRDT_Connectors:Molex_SL_03
Connections:
- net labels removed: Servo_8_Ctrl
- wire segments 62 -> 55
Other:
- note removed: "Servo 8"
- moved on the sheet: Conn2, Conn3, Conn4, Conn5, Conn6, Conn7, Conn8

Commit message: Fixed Minor Issues
Parts:
- added Conn9: Molex_SL_03, MRDT_Connectors:MOLEX_SL_03_Horizontal, symbol MRDT_Connectors:Molex_SL_03
Connections:
- net labels added: Servo_8_Ctrl
- wire segments 55 -> 61
Other:
- note added: "Servo 8"
Changed lines of the file:
@@
 L power:GND #PWR0103
 U 1 1 5BCD697A
-P 5800 5650
-F 0 "#PWR0103" H 5800 5400 50  0001 C CNN
-F 1 "GND" H 5805 5477 50  0000 C CNN
-F 2 "" H 5800 5650 50  0001 C CNN
-F 3 "" H 5800 5650 50  0001 C CNN
-	1    5800 5650
+P 5800 6000
+F 0 "#PWR0103" H 5800 5750 50  0001 C CNN
+F 1 "GND" H 5805 5827 50  0000 C CNN
+F 2 "" H 5800 6000 50  0001 C CNN
+F 3 "" H 5800 6000 50  0001 C CNN
+	1    5800 6000
 	1    0    0    -1
 $EndComp
@@
 Wire Wire Line
 	5900 5200 5800 5200
-Connection ~ 5800 5200
-Wire Wire Line
-	5800 5200 5800 5550
-Wire Wire Line
-	5900 5550 5800 5550
 Wire Wire Line
 	5550 3350 5900 3350
@@
 	6900 1250 6900 6100
 Wire Notes Line
-	6900 6100 2400 6100
+	6900 6250 2400 6250
 Wire Notes Line
 	6900 1250 2400 1250
@@
 Text Notes 6200 5550 1    39   ~ 0
 Servo 7
-Wire Wire Line
-	5800 5550 5800 5650
+$Comp
+L MRDT_Connectors:Molex_SL_03 Conn9
+U 1 1 5BD49544
+P 6100 5950
+F 0 "Conn9" H 6227 6158 60  0000 L CNN
+F 1 "Molex_SL_03" H 6227 6052 60  0000 L CNN
+F 2 "MRDT_Connectors:MOLEX_SL_03_Horizontal" H 6100 5950 60  0001 C CNN
+F 3 "" H 6100 5950 60  0001 C CNN
+	1    6100 5950
+	1    0    0    -1
+$EndComp
+Text GLabel 5550 5800 0    50   Input ~ 0
+Servo_8_Ctrl
+Wire Wire Line
+	5900 5900 5800 5900
+Wire Wire Line
+	5900 5800 5550 5800
+Wire Wire Line
+	5700 5700 5700 5350
+Text Notes 6200 5900 1    39   ~ 0
+Servo 8
+Wire Wire Line
+	5800 5900 5800 6000
+Wire Wire Line
+	5700 5700 5900 5700
+Wire Wire Line
+	5800 5200 5800 5550
+Wire Wire Line
+	5800 5550 5900 5550
+Connection ~ 5800 5200
+Wire Wire Line
+	5800 5550 5800 5900
 Connection ~ 5800 5550
+Connection ~ 5800 5900
+Text GLabel 4250 4300 2    50   Input ~ 0
+Servo_8_Ctrl
+Wire Wire Line
+	4100 4300 4250 4300
 $EndSCHEMATC
