File: ShimbleBoard_Hardware/ShimbleBoard_Hardware.sch (KiCad schematic (older format))
At the start: 13 parts, among them U1 TM4C129E_Launchpad, U2 OKI

Commit message: Board Review
Changed lines of the file:
@@
 Wire Wire Line
 	4100 4700 4250 4700
-Wire Wire Line
-	3050 3500 3200 3500
-Wire Wire Line
-	4250 4200 4100 4200
-Text GLabel 4250 4200 2    50   Input ~ 0
+Text GLabel 3050 4700 0    50   Input ~ 0
 Servo_7_Ctrl
 Text GLabel 5550 5100 0    50   Input ~ 0
 Servo_6_Ctrl
+Text GLabel 3050 4900 0    50   Input ~ 0
+Servo_5_Ctrl
+Text GLabel 3050 5000 0    50   Input ~ 0
+Servo_4_Ctrl
+Text GLabel 4250 5500 2    50   Input ~ 0
+Servo_3_Ctrl
+Text GLabel 4250 4900 2    50   Input ~ 0
+Servo_2_Ctrl
 Text GLabel 4250 4700 2    50   Input ~ 0
-Servo_5_Ctrl
-Text GLabel 3050 4900 0    50   Input ~ 0
-Servo_4_Ctrl
+Servo_1_Ctrl
 Text GLabel 3050 4800 0    50   Input ~ 0
-Servo_3_Ctrl
-Text GLabel 3050 4700 0    50   Input ~ 0
-Servo_2_Ctrl
-Text GLabel 3050 4600 0    50   Input ~ 0
-Servo_1_Ctrl
-Text GLabel 3050 3500 0    50   Input ~ 0
 Servo_6_Ctrl
 Text GLabel 5550 4750 0    50   Input ~ 0
@@
 Connection ~ 5800 5550
 Connection ~ 5800 5900
-Text GLabel 4250 4300 2    50   Input ~ 0
+Text GLabel 3050 4600 0    50   Input ~ 0
 Servo_8_Ctrl
-Wire Wire Line
-	4100 4300 4250 4300
 Wire Notes Line
 	2400 1250 2400 6250
 Wire Notes Line
 	6900 1250 6900 6250
+Wire Wire Line
+	3050 5000 3200 5000
+Wire Wire Line
+	4250 5500 4100 5500
+Wire Wire Line
+	4250 4900 4100 4900
 $EndSCHEMATC

Commit message: Revised Schematic
Parts:
- removed U2: OKI, MRDT_Devices:OKI_Horizontal, symbol MRDT_Devices:OKI
- added C3, C4: 10uF, Capacitor_SMD:C_0603_1608Metric_Pad1.05x0.95mm_HandSolder, symbol Device:C
- added unit 3 of Conn1
- added D1, D2: D_Schottky, Diode_SMD:D_0603_1608Metric_Pad1.05x0.95mm_HandSolder, symbol Device:D_Schottky_ALT
- added D10: Ctrl_6_LED, Diode_SMD:D_0603_1608Metric_Pad1.05x0.95mm_HandSolder, symbol Device:LED
- added D11: Ctrl_7_LED, Diode_SMD:D_0603_1608Metric_Pad1.05x0.95mm_HandSolder, symbol Device:LED
- added D12: Ctrl_8_LED, Diode_SMD:D_0603_1608Metric_Pad1.05x0.95mm_HandSolder, symbol Device:LED
- added D3: 5V_Act_LED, Diode_SMD:D_0603_1608Metric_Pad1.05x0.95mm_HandSolder, symbol Device:LED
- added D4: 5V_Log_LED, Diode_SMD:D_0603_1608Metric_Pad1.05x0.95mm_HandSolder, symbol Device:LED
- added D5: Ctrl_1_LED, Diode_SMD:D_0603_1608Metric_Pad1.05x0.95mm_HandSolder, symbol Device:LED
- added D6: Ctrl_2_LED, Diode_SMD:D_0603_1608Metric_Pad1.05x0.95mm_HandSolder, symbol Device:LED
- added D7: Ctrl_3_LED, Diode_SMD:D_0603_1608Metric_Pad1.05x0.95mm_HandSolder, symbol Device:LED
- added D8: Ctrl_4_LED, Diode_SMD:D_0603_1608Metric_Pad1.05x0.95mm_HandSolder, symbol Device:LED
- added D9: Ctrl_5_LED, Diode_SMD:D_0603_1608Metric_Pad1.05x0.95mm_HandSolder, symbol Device:LED
- added L1: 47uH, Inductor_SMD:L_0603_1608Metric_Pad1.05x0.95mm_HandSolder, symbol Device:L
- added L2: 47uH, Diode_SMD:D_0603_1608Metric_Pad1.05x0.95mm_HandSolder, symbol Device:L
- added R1, R10, R2, R3, R4, R5, R6, R7, R8, R9: 500, Resistor_SMD:R_0603_1608Metric_Pad1.05x0.95mm_HandSolder, symbol Device:R
- added U2, U3: AP1059, Package_SO:SOIC-8_3.9x4.9mm_P1.27mm, symbol MRDT_ICs:AP1059
- Conn1: footprint MRDT_Connectors:Anderson_2_Horisontal_Side_by_Side -> MRDT_Connectors:Anderson_3_Horisontal_Side_by_Side
Connections:
- net labels added: +5VA, +5VL, V+Act, V+Log
- net labels removed: +5V
- wire segments 61 -> 154
Other:
- note added: "Indicators"
- note added: "Power Inputs"
- moved on the sheet: Conn1A, Conn1B, Conn2, Conn3, Conn4, Conn5, Conn6, Conn7, Conn8, Conn9

Commit message: Work hours 2018-11-17
Other:
- note added: "AnalogWrite"
- note added: "PWM"
- moved on the sheet: C1, C2, C3, C4, Conn1A, Conn1B, Conn1C

Commit message: BOM and Redesigned AP1509 Area
Parts:
- L1: footprint Inductor_SMD:L_0603_1608Metric_Pad1.05x0.95mm_HandSolder -> ShimbleBoard_Hardware:ETQ-P4M470YFN_Inductor
- L2: footprint Diode_SMD:D_0603_1608Metric_Pad1.05x0.95mm_HandSolder -> ShimbleBoard_Hardware:ETQ-P4M470YFN_Inductor
Changed lines of the file:
@@
 F 0 "L1" H 3950 1700 50  0000 L BNN
 F 1 "47uH" H 3950 1800 50  0000 L CNN
-F 2 "Inductor_SMD:L_0603_1608Metric_Pad1.05x0.95mm_HandSolder" H 3900 1800 50  0001 C CNN
+F 2 "ShimbleBoard_Hardware:ETQ-P4M470YFN_Inductor" H 3900 1800 50  0001 C CNN
 F 3 "~" H 3900 1800 50  0001 C CNN
 	1    3900 1800
@@
 F 0 "L2" H 6650 1700 50  0000 L BNN
 F 1 "47uH" H 6650 1800 50  0000 L CNN
-F 2 "Diode_SMD:D_0603_1608Metric_Pad1.05x0.95mm_HandSolder" H 6600 1800 50  0001 C CNN
+F 2 "ShimbleBoard_Hardware:ETQ-P4M470YFN_Inductor" H 6600 1800 50  0001 C CNN
 F 3 "~" H 6600 1800 50  0001 C CNN
 	1    6600 1800

Commit message: PRR Take 2: OKI Boogaloo
Parts:
- removed D1, D2: D_Schottky, Diode_SMD:D_0603_1608Metric_Pad1.05x0.95mm_HandSolder, symbol Device:D_Schottky_ALT
- removed L1, L2: 47uH, ShimbleBoard_Hardware:ETQ-P4M470YFN_Inductor, symbol Device:L
- removed U2, U3: AP1059, Package_SO:SOIC-8_3.9x4.9mm_P1.27mm, symbol MRDT_ICs:AP1059
- added U2, U3: OKI, MRDT_Devices:OKI_Horizontal, symbol MRDT_Devices:OKI
Connections:
- wire segments 154 -> 110
Other:
- moved on the sheet: C3, C4

Commit message: Finalized board and made adjustments
Connections:
- net labels added: +12L, +12VA
- net labels removed: V+Act, V+Log
- wire segments 110 -> 114
Other:
- note added: "Green"
- note added: "Orange"
- note added: "PWM 5"
- note added: "PWM 6"
- note added: "PWM 7\n"
- note removed: "PWM"
Changed lines of the file:
@@
 P 1800 1700
 F 0 "Conn1" H 1950 1650 60  0000 C CNN
-F 1 "AndersonPP" H 1950 2250 60  0000 C CNN
+F 1 "AndersonPP" H 1900 2250 60  0000 C CNN
 F 2 "MRDT_Connectors:Anderson_3_Horisontal_Side_by_Side" H 1650 1150 60  0001 C CNN
 F 3 "" H 1650 1150 60  0001 C CNN
@@
 Text GLabel 7250 6000 0    50   Input ~ 0
 Servo_8_Ctrl
-Text GLabel 2400 1950 2    50   Input ~ 0
-V+Act
-Text GLabel 2400 1250 2    50   Input ~ 0
-V+Log
 Wire Wire Line
 	2350 1300 2350 1250
-Wire Wire Line
-	2350 1250 2400 1250
 Connection ~ 2350 1300
-Wire Wire Line
-	2350 1900 2350 1950
-Wire Wire Line
-	2350 1950 2400 1950
 Connection ~ 2350 1900
 $Comp
@@
 	1    0    0    -1
 $EndComp
-Text GLabel 6700 1400 0    50   Input ~ 0
-V+Log
-Text GLabel 4050 1400 0    50   Input ~ 0
-V+Act
 $Comp
 L Device:C C4
@@
 	1400 6400 8400 6400
 Text Notes 1850 4650 2    47   ~ 0
-PWM
+PWM 5
 Text Notes 1850 4750 2    47   ~ 0
-PWM
+PWM 6
 Text Notes 1850 4850 2    47   ~ 0
-PWM
+PWM 7\n
 Text Notes 1850 4950 2    47   ~ 0
 AnalogWrite
@@
 	7750 1400 7500 1400
 Connection ~ 7500 1400
+$Comp
+L power:+12VA #PWR?
+U 1 1 5C16D80D
+P 2550 2100
+F 0 "#PWR?" H 2550 1950 50  0001 C CNN
+F 1 "+12VA" H 2565 2273 50  0000 C CNN
+F 2 "" H 2550 2100 50  0001 C CNN
+F 3 "" H 2550 2100 50  0001 C CNN
+	1    2550 2100
+	1    0    0    -1
+$EndComp
+$Comp
+L power:+12L #PWR?
+U 1 1 5C16D884
+P 2350 1250
+F 0 "#PWR?" H 2350 1100 50  0001 C CNN
+F 1 "+12L" H 2365 1423 50  0000 C CNN
+F 2 "" H 2350 1250 50  0001 C CNN
+F 3 "" H 2350 1250 50  0001 C CNN
+	1    2350 1250
+	1    0    0    -1
+$EndComp
+Wire Wire Line
+	2350 2150 2550 2150
+Wire Wire Line
+	2550 2150 2550 2100
+Wire Wire Line
+	2350 1900 2350 2150
+$Comp
+L power:+12VA #PWR?
+U 1 1 5C171904
+P 4000 1350
+F 0 "#PWR?" H 4000 1200 50  0001 C CNN
+F 1 "+12VA" H 4015 1523 50  0000 C CNN
+F 2 "" H 4000 1350 50  0001 C CNN
+F 3 "" H 4000 1350 50  0001 C CNN
+	1    4000 1350
+	1    0    0    -1
+$EndComp
+$Comp
+L power:+12L #PWR?
+U 1 1 5C17195D
+P 6650 1350
+F 0 "#PWR?" H 6650 1200 50  0001 C CNN
+F 1 "+12L" H 6665 1523 50  0000 C CNN
+F 2 "" H 6650 1350 50  0001 C CNN
+F 3 "" H 6650 1350 50  0001 C CNN
+	1    6650 1350
+	1    0    0    -1
+$EndComp
+Wire Wire Line
+	4000 1350 4000 1400
+Wire Wire Line
+	4000 1400 4050 1400
+Wire Wire Line
+	6650 1350 6650 1400
+Wire Wire Line
+	6650 1400 6700 1400
+Text Notes 7650 2850 0    50   ~ 0
+Green
+Text Notes 7650 3200 0    50   ~ 0
+Green
+Text Notes 7600 3900 0    50   ~ 0
+Orange
+Text Notes 7600 3550 0    50   ~ 0
+Orange
+Text Notes 7600 4250 0    50   ~ 0
+Orange
+Text Notes 7600 4600 0    50   ~ 0
+Orange
+Text Notes 7600 4950 0    50   ~ 0
+Orange
+Text Notes 7600 5300 0    50   ~ 0
+Orange
+Text Notes 7600 5650 0    50   ~ 0
+Orange
+Text Notes 7600 6000 0    50   ~ 0
+Orange
 $EndSCHEMATC

Commit message: Updated Rev2 Libraries
Parts:
- Conn1: footprint MRDT_Connectors:Anderson_3_Horisontal_Side_by_Side -> MRDT_Connectors:Anderson_3_Horizontal_Side_by_Side
- U1: footprint MRDT_Shields:TM4C129E_Launchpad_X7 -> MRDT_Shields:TM4C129E_Launchpad_X7_THT_BOTTOM
Changed lines of the file:
@@
 F 0 "Conn1" H 1950 1650 60  0000 C CNN
 F 1 "AndersonPP" H 1900 2250 60  0000 C CNN
-F 2 "MRDT_Connectors:Anderson_3_Horisontal_Side_by_Side" H 1650 1150 60  0001 C CNN
+F 2 "MRDT_Connectors:Anderson_3_Horizontal_Side_by_Side" H 1650 1150 60  0001 C CNN
 F 3 "" H 1650 1150 60  0001 C CNN
 	1    1800 1700
@@
 F 0 "Conn1" H 1950 1350 60  0000 C CNN
 F 1 "AndersonPP" H 2006 1681 60  0001 C CNN
-F 2 "MRDT_Connectors:Anderson_3_Horisontal_Side_by_Side" H 1650 850 60  0001 C CNN
+F 2 "MRDT_Connectors:Anderson_3_Horizontal_Side_by_Side" H 1650 850 60  0001 C CNN
 F 3 "" H 1650 850 60  0001 C CNN
 	2    1800 1400
@@
 F 0 "U1" H 2750 4300 60  0000 L CNN
 F 1 "TM4C129E_Launchpad" H 2500 5500 60  0000 L CNN
-F 2 "MRDT_Shields:TM4C129E_Launchpad_X7" H 2750 4350 60  0001 C CNN
+F 2 "MRDT_Shields:TM4C129E_Launchpad_X7_THT_BOTTOM" H 2750 4350 60  0001 C CNN
 F 3 "" H 2750 4350 60  0001 C CNN
 	5    2750 4350
@@
 F 0 "U1" H 3250 4300 60  0000 L CNN
 F 1 "TM4C129E_Launchpad" H 3555 4842 60  0001 L CNN
-F 2 "MRDT_Shields:TM4C129E_Launchpad_X7" H 3250 4350 60  0001 C CNN
+F 2 "MRDT_Shields:TM4C129E_Launchpad_X7_THT_BOTTOM" H 3250 4350 60  0001 C CNN
 F 3 "" H 3250 4350 60  0001 C CNN
 	6    3250 4350
@@
 F 0 "U1" H 2750 5500 60  0000 L CNN
 F 1 "TM4C129E_Launchpad" H 3055 6042 60  0001 L CNN
-F 2 "MRDT_Shields:TM4C129E_Launchpad_X7" H 2750 5550 60  0001 C CNN
+F 2 "MRDT_Shields:TM4C129E_Launchpad_X7_THT_BOTTOM" H 2750 5550 60  0001 C CNN
 F 3 "" H 2750 5550 60  0001 C CNN
 	7    2750 5550
@@
 F 0 "U1" H 3250 5500 60  0000 L CNN
 F 1 "TM4C129E_Launchpad" H 3555 6042 60  0001 L CNN
-F 2 "MRDT_Shields:TM4C129E_Launchpad_X7" H 3250 5550 60  0001 C CNN
+F 2 "MRDT_Shields:TM4C129E_Launchpad_X7_THT_BOTTOM" H 3250 5550 60  0001 C CNN
 F 3 "" H 3250 5550 60  0001 C CNN
 	8    3250 5550
@@
 F 0 "Conn1" H 1950 1950 60  0000 C CNN
 F 1 "AndersonPP" H 2006 2281 60  0001 C CNN
-F 2 "MRDT_Connectors:Anderson_3_Horisontal_Side_by_Side" H 1650 1450 60  0001 C CNN
+F 2 "MRDT_Connectors:Anderson_3_Horizontal_Side_by_Side" H 1650 1450 60  0001 C CNN
 F 3 "" H 1650 1450 60  0001 C CNN
 	3    1800 2000
@@
 Connection ~ 7500 1400
 $Comp
-L power:+12VA #PWR?
+L power:+12VA #PWR0114
 U 1 1 5C16D80D
 P 2550 2100
-F 0 "#PWR?" H 2550 1950 50  0001 C CNN
+F 0 "#PWR0114" H 2550 1950 50  0001 C CNN
 F 1 "+12VA" H 2565 2273 50  0000 C CNN
 F 2 "" H 2550 2100 50  0001 C CNN
@@
 $EndComp
 $Comp
-L power:+12L #PWR?
+L power:+12L #PWR0115
 U 1 1 5C16D884
 P 2350 1250
-F 0 "#PWR?" H 2350 1100 50  0001 C CNN
+F 0 "#PWR0115" H 2350 1100 50  0001 C CNN
 F 1 "+12L" H 2365 1423 50  0000 C CNN
 F 2 "" H 2350 1250 50  0001 C CNN
@@
 	2350 1900 2350 2150
 $Comp
-L power:+12VA #PWR?
+L power:+12VA #PWR0116
 U 1 1 5C171904
 P 4000 1350
-F 0 "#PWR?" H 4000 1200 50  0001 C CNN
+F 0 "#PWR0116" H 4000 1200 50  0001 C CNN
 F 1 "+12VA" H 4015 1523 50  0000 C CNN
 F 2 "" H 4000 1350 50  0001 C CNN
@@
 $EndComp
 $Comp
-L power:+12L #PWR?
+L power:+12L #PWR0117
 U 1 1 5C17195D
 P 6650 1350
-F 0 "#PWR?" H 6650 1200 50  0001 C CNN
+F 0 "#PWR0117" H 6650 1200 50  0001 C CNN
 F 1 "+12L" H 6665 1523 50  0000 C CNN
 F 2 "" H 6650 1350 50  0001 C CNN

Commit message: Fixed Servo Wiring
Parts:
- U1: symbol MRDT_Shields:TM4C129E_Launchpad -> ShimbleBoard_Hardware-rescue:TM4C129E_Launchpad-MRDT_Shields
Changed lines of the file:
@@
 $EndComp
 $Comp
-L MRDT_Shields:TM4C129E_Launchpad U1
+L ShimbleBoard_Hardware-rescue:TM4C129E_Launchpad-MRDT_Shields U1
 U 5 1 5BCBB9FF
 P 2750 4350
@@
 $EndComp
 $Comp
-L MRDT_Shields:TM4C129E_Launchpad U1
+L ShimbleBoard_Hardware-rescue:TM4C129E_Launchpad-MRDT_Shields U1
 U 6 1 5BCBBA80
 P 3250 4350
@@
 $EndComp
 $Comp
-L MRDT_Shields:TM4C129E_Launchpad U1
+L ShimbleBoard_Hardware-rescue:TM4C129E_Launchpad-MRDT_Shields U1
 U 7 1 5BCBBAD0
 P 2750 5550
@@
 $EndComp
 $Comp
-L MRDT_Shields:TM4C129E_Launchpad U1
+L ShimbleBoard_Hardware-rescue:TM4C129E_Launchpad-MRDT_Shields U1
 U 8 1 5BCBBB1F
 P 3250 5550
@@
 Wire Wire Line
 	3450 4700 3600 4700
-Text GLabel 2400 4700 0    50   Input ~ 0
+Text GLabel 2400 4700 0    50   Output ~ 0
 Servo_7_Ctrl
-Text GLabel 5250 5000 0    50   Input ~ 0
+Text GLabel 5250 4900 0    50   Input ~ 0
 Servo_6_Ctrl
-Text GLabel 2400 4900 0    50   Input ~ 0
+Text GLabel 2400 4900 0    50   Output ~ 0
 Servo_5_Ctrl
-Text GLabel 2400 5000 0    50   Input ~ 0
+Text GLabel 2400 5000 0    50   Output ~ 0
 Servo_4_Ctrl
-Text GLabel 3600 5500 2    50   Input ~ 0
+Text GLabel 3600 5500 2    50   Output ~ 0
 Servo_3_Ctrl
-Text GLabel 3600 4900 2    50   Input ~ 0
+Text GLabel 3600 4900 2    50   Output ~ 0
 Servo_2_Ctrl
-Text GLabel 3600 4700 2    50   Input ~ 0
+Text GLabel 3600 4700 2    50   Output ~ 0
 Servo_1_Ctrl
-Text GLabel 2400 4800 0    50   Input ~ 0
+Text GLabel 2400 4800 0    50   Output ~ 0
 Servo_6_Ctrl
-Text GLabel 5250 4650 0    50   Input ~ 0
+Text GLabel 5250 4550 0    50   Input ~ 0
 Servo_5_Ctrl
-Text GLabel 5250 4300 0    50   Input ~ 0
+Text GLabel 5250 4200 0    50   Input ~ 0
 Servo_4_Ctrl
-Text GLabel 5250 3950 0    50   Input ~ 0
+Text GLabel 5250 3850 0    50   Input ~ 0
 Servo_3_Ctrl
-Text GLabel 5250 3600 0    50   Input ~ 0
+Text GLabel 5250 3500 0    50   Input ~ 0
 Servo_2_Ctrl
-Text GLabel 5250 3250 0    50   Input ~ 0
+Text GLabel 5250 3150 0    50   Input ~ 0
 Servo_1_Ctrl
 Wire Wire Line
@@
 	1    0    0    -1
 $EndComp
-Text GLabel 5250 5350 0    50   Input ~ 0
+Text GLabel 5250 5250 0    50   Input ~ 0
 Servo_7_Ctrl
 Wire Wire Line
@@
 	5600 5100 5500 5100
 Wire Wire Line
-	5250 3250 5600 3250
-Wire Wire Line
-	5600 3600 5250 3600
-Wire Wire Line
-	5600 3950 5250 3950
-Wire Wire Line
-	5600 4300 5250 4300
-Wire Wire Line
-	5600 4650 5250 4650
-Wire Wire Line
-	5600 5000 5250 5000
-Wire Wire Line
-	5600 5350 5250 5350
-Wire Wire Line
-	5600 3150 5400 3150
-Connection ~ 5400 3150
-Wire Wire Line
-	5400 3150 5400 3050
-Wire Wire Line
-	5600 3500 5400 3500
-Connection ~ 5400 3500
-Wire Wire Line
-	5400 3500 5400 3150
-Wire Wire Line
-	5600 3850 5400 3850
-Connection ~ 5400 3850
-Wire Wire Line
-	5400 3850 5400 3500
-Wire Wire Line
-	5600 4200 5400 4200
-Connection ~ 5400 4200
-Wire Wire Line
-	5400 4200 5400 3850
-Wire Wire Line
-	5600 4550 5400 4550
-Connection ~ 5400 4550
-Wire Wire Line
-	5400 4550 5400 4200
-Connection ~ 5400 4900
-Wire Wire Line
-	5400 4900 5400 4550
-Wire Wire Line
-	5400 4900 5600 4900
-Wire Wire Line
-	5600 5250 5400 5250
-Wire Wire Line
-	5400 5250 5400 4900
+	5250 3150 5600 3150
+Wire Wire Line
+	5600 3500 5250 3500
+Wire Wire Line
+	5600 3850 5250 3850
+Wire Wire Line
+	5600 4200 5250 4200
+Wire Wire Line
+	5600 4550 5250 4550
+Wire Wire Line
+	5600 4900 5250 4900
+Wire Wire Line
+	5600 5250 5250 5250
 Text Notes 2400 2450 0    118  ~ 24
 TIVA Headers
@@
 	1    0    0    -1
 $EndComp
-Text GLabel 5250 5700 0    50   Input ~ 0
+Text GLabel 5250 5600 0    50   Input ~ 0
 Servo_8_Ctrl
 Wire Wire Line
 	5600 5800 5500 5800
-Wire Wire Line
-	5600 5700 5250 5700
-Wire Wire Line
-	5400 5600 5400 5250
 Text Notes 5900 5800 1    39   ~ 0
 Servo 8
 Wire Wire Line
 	5500 5800 5500 5900
-Wire Wire Line
-	5400 5600 5600 5600
 Wire Wire Line
 	5500 5100 5500 5450
@@
 Connection ~ 5500 5450
 Connection ~ 5500 5800
-Text GLabel 2400 4600 0    50   Input ~ 0
+Text GLabel 2400 4600 0    50   Output ~ 0
 Servo_8_Ctrl
 Wire Wire Line
@@
 Wire Notes Line
 	3100 2100 3100 700
-Connection ~ 5400 5250
 Text Notes 7050 2450 0    118  ~ 24
 Indicators
@@
 Text Notes 7600 6000 0    50   ~ 0
 Orange
+Wire Wire Line
+	5600 5700 5400 5700
+Wire Wire Line
+	5400 3050 5400 3250
+Wire Wire Line
+	5600 5600 5250 5600
+Wire Wire Line
+	5400 5350 5600 5350
+Connection ~ 5400 5350
+Wire Wire Line
+	5400 5350 5400 5700
+Wire Wire Line
+	5600 5000 5400 5000
+Connection ~ 5400 5000
+Wire Wire Line
+	5400 5000 5400 5350
+Wire Wire Line
+	5600 4650 5400 4650
+Connection ~ 5400 4650
+Wire Wire Line
+	5400 4650 5400 5000
+Wire Wire Line
+	5600 4300 5400 4300
+Connection ~ 5400 4300
+Wire Wire Line
+	5400 4300 5400 4650
+Wire Wire Line
+	5600 3600 5400 3600
+Connection ~ 5400 3600
+Wire Wire Line
+	5600 3250 5400 3250
+Connection ~ 5400 3250
+Wire Wire Line
+	5400 3250 5400 3600
+Wire Wire Line
+	5400 3600 5400 3950
+Wire Wire Line
+	5600 3950 5400 3950
+Connection ~ 5400 3950
+Wire Wire Line
+	5400 3950 5400 4300
 $EndSCHEMATC
