File: ShimbleBoard_Hardware/ShimbleBoard_Hardware.kicad_pcb (KiCad board)
At the start: 2 copper layers, 61 x 91.6 mm, 42 parts, among them U1 TM4C129E_Launchpad, U2 AP1059, U3 AP1059

Commit message: PRR Take 2: OKI Boogaloo
Parts:
- removed D1, D2: D_Schottky, Diode_SMD:D_0603_1608Metric_Pad1.05x0.95mm_HandSolder
- removed L1, L2: 47uH, ShimbleBoard_Hardware:ETQ-P4M470YFN_Inductor
- U2, U3: value AP1059 -> OKI; footprint Package_SO:SOIC-8_3.9x4.9mm_P1.27mm -> MRDT_Devices:OKI_Horizontal
- moved U2 23.2 mm to (95.5, 106.2)
- moved U3 13.1 mm to (120.4, 122.7), turned to 180 degrees
- moved C2 4.93 mm to (108.0, 113.8), turned to 180 degrees
- moved C4 1.87 mm to (108.0, 111.2)
- moved C1 1.83 mm to (108.0, 118.6), turned to 0 degrees
- moved C3 1.05 mm to (108.0, 120.7)
Connections:
- C3 pad 1: GND -> +5VL
- C3 pad 2: +5VL -> GND
- C4 pad 1: GND -> +5VA
- C4 pad 2: +5VA -> GND
- U2 pad 1: V+Log -> V+Act
- U2 pad 2: Net-(D1-Pad1) -> GND
- U2 pad 3: +5VL -> +5VA
- U3 pad 1: V+Act -> V+Log
- U3 pad 2: Net-(D2-Pad1) -> GND
- U3 pad 3: +5VA -> +5VL
Routing:
- net GND: track 70.1 -> 45.9 mm, vias 13 -> 15
- net V+Act: track 18.3 -> 39.6 mm
- net Net-(D2-Pad1): track 10.3 -> 0.00 mm
- net Net-(D1-Pad1): track 10.3 -> 0.00 mm
- net V+Log: track 17.4 -> 27.7 mm
- net +5VA: track 82.9 -> 75.2 mm
- net +5VL: track 59.6 -> 58.9 mm
- net (no net): vias 5 -> 0

Commit message: Finalized board and made adjustments
Parts:
- C2: moved to B.Cu
- Conn2, Conn3, Conn4, Conn5, Conn6, Conn7, Conn8: footprint MRDT_Connectors:MOLEX_SL_03_Horizontal -> MRDT_Connectors:MOLEX_SL_03_Horizontal_NO_HOLE
- moved C2 7.51 mm to (108.0, 106.3), turned to 90 degrees
Routing:
- net +5VA: track 75.2 -> 13.9 mm
- net V+Act: track 39.6 -> 29.9 mm
- net V+Log: track 27.7 -> 26.1 mm
- net GND: track 45.9 -> 44.8 mm
Other:
- board text added: "+ PWM -"
- board text added: "5VA"
- board text added: "5VL"
