File: ShimbleBoard_Hardware/Gimbal_Board.sch (KiCad schematic (older format))
At the start: 89 parts, among them Q1 Q_NMOS_GDS, Q2 Q_NMOS_GDS, Q3 Q_NMOS_GDS, Q4 Q_NMOS_GDS, Q5 Q_NMOS_GDS, Q6 Q_NMOS_GDS, Q7 Q_NMOS_GDS, Q8 Q_NMOS_GDS, SW1 SW_Push, SW10 SW_SPDT, SW2 SW_Push, SW3 SW_Push, SW4 SW_Push, SW5 SW_Push, SW6 SW_Push, SW7 SW_Push, SW8 SW_Push, SW9 SW_Push, U1 TM4C129E_Launchpad, U2 OKI, U3 OKI

Commit message: Gerbs
Parts:
- D20: value 5V_Log_LED -> 3V_LED
- R1, R2, R28, R3, R4, R5, R6, R7, R8: value 500 -> 330
Connections:
- net +3V3: now also C3.1, R1.1, R2.1, R28.2, R3.1, R4.1, R5.1, R6.1, R7.1, R8.1, U2.3 (Vo)
- removed net +5VL: C3.1, R1.1, R2.1, R28.2, R3.1, R4.1, R5.1, R6.1, R7.1, R8.1, U1.+5V (B1_1), U1.+5V' (B2_1), U2.3 (Vo)
- no-connect marks 55 -> 57
Changed lines of the file:
@@
 P 1050 6000
 F 0 "R6" V 1150 5950 50  0000 L CNN
-F 1 "500" V 1050 5950 50  0000 L CNN
+F 1 "330" V 1050 5950 50  0000 L CNN
 F 2 "Resistor_SMD:R_0603_1608Metric_Pad1.05x0.95mm_HandSolder" V 980 6000 50  0001 C CNN
 F 3 "~" H 1050 6000 50  0001 C CNN
@@
 Wire Wire Line
 	1200 2250 1300 2250
-Wire Wire Line
-	800  2250 850  2250
 $Comp
 L power:+5VA #PWR010
@@
 P 1050 4700
 F 0 "R4" V 1150 4650 50  0000 L CNN
-F 1 "500" V 1050 4650 50  0000 L CNN
+F 1 "330" V 1050 4650 50  0000 L CNN
 F 2 "Resistor_SMD:R_0603_1608Metric_Pad1.05x0.95mm_HandSolder" V 980 4700 50  0001 C CNN
 F 3 "~" H 1050 4700 50  0001 C CNN
@@
 P 1050 4050
 F 0 "R3" V 1150 4000 50  0000 L CNN
-F 1 "500" V 1050 4000 50  0000 L CNN
+F 1 "330" V 1050 4000 50  0000 L CNN
 F 2 "Resistor_SMD:R_0603_1608Metric_Pad1.05x0.95mm_HandSolder" V 980 4050 50  0001 C CNN
 F 3 "~" H 1050 4050 50  0001 C CNN
@@
 P 1050 3400
 F 0 "R2" V 1150 3350 50  0000 L CNN
-F 1 "500" V 1050 3350 50  0000 L CNN
+F 1 "330" V 1050 3350 50  0000 L CNN
 F 2 "Resistor_SMD:R_0603_1608Metric_Pad1.05x0.95mm_HandSolder" V 980 3400 50  0001 C CNN
 F 3 "~" H 1050 3400 50  0001 C CNN
@@
 P 1050 7300
 F 0 "R8" V 1150 7250 50  0000 L CNN
-F 1 "500" V 1050 7250 50  0000 L CNN
+F 1 "330" V 1050 7250 50  0000 L CNN
 F 2 "Resistor_SMD:R_0603_1608Metric_Pad1.05x0.95mm_HandSolder" V 980 7300 50  0001 C CNN
 F 3 "~" H 1050 7300 50  0001 C CNN
@@
 P 1050 6650
 F 0 "R7" V 1150 6600 50  0000 L CNN
-F 1 "500" V 1050 6600 50  0000 L CNN
+F 1 "330" V 1050 6600 50  0000 L CNN
 F 2 "Resistor_SMD:R_0603_1608Metric_Pad1.05x0.95mm_HandSolder" V 980 6650 50  0001 C CNN
 F 3 "~" H 1050 6650 50  0001 C CNN
@@
 P 1450 2250
 F 0 "D20" H 1450 2150 50  0000 C CNN
-F 1 "5V_Log_LED" H 1450 2350 50  0000 C CNN
+F 1 "3V_LED" H 1450 2350 50  0000 C CNN
 F 2 "Diode_SMD:D_0603_1608Metric_Pad1.05x0.95mm_HandSolder" H 1450 2250 50  0001 C CNN
 F 3 "~" H 1450 2250 50  0001 C CNN
@@
 P 1050 2250
 F 0 "R28" V 950 2250 50  0000 C CNN
-F 1 "500" V 1050 2250 50  0000 C CNN
+F 1 "330" V 1050 2250 50  0000 C CNN
 F 2 "Resistor_SMD:R_0603_1608Metric_Pad1.05x0.95mm_HandSolder" V 980 2250 50  0001 C CNN
 F 3 "~" H 1050 2250 50  0001 C CNN
 	1    1050 2250
 	0    1    -1   0
-$EndComp
-$Comp
-L power:+5VL #PWR09
-U 1 1 5D93B524
-P 800 2250
-F 0 "#PWR09" H 800 2100 50  0001 C CNN
-F 1 "+5VL" H 815 2423 50  0000 C CNN
-F 2 "" H 800 2250 50  0001 C CNN
-F 3 "" H 800 2250 50  0001 C CNN
-	1    800  2250
-	-1   0    0    -1
 $EndComp
 Wire Wire Line
@@
 $EndComp
 $Comp
-L power:+5VL #PWR04
-U 1 1 5DB37DF7
-P 4550 1050
-F 0 "#PWR04" H 4550 900 50  0001 C CNN
-F 1 "+5VL" H 4565 1223 50  0000 C CNN
-F 2 "" H 4550 1050 50  0001 C CNN
-F 3 "" H 4550 1050 50  0001 C CNN
-	1    4550 1050
-	1    0    0    -1
-$EndComp
-$Comp
 L power:GND #PWR05
 U 1 1 5DB3823D
@@
 Wire Notes Line
 	2600 2900 7400 2900
-$Comp
-L power:+5VL #PWR0109
-U 1 1 5DA29F3F
-P 4500 3300
-F 0 "#PWR0109" H 4500 3150 50  0001 C CNN
-F 1 "+5VL" H 4515 3473 50  0000 C CNN
-F 2 "" H 4500 3300 50  0001 C CNN
-F 3 "" H 4500 3300 50  0001 C CNN
-	1    4500 3300
-	1    0    0    -1
-$EndComp
 $Comp
 L power:GND #PWR0108
@@
 TIVA Logic
 $Comp
-L power:+5VL #PWR0106
-U 1 1 5DA9133E
-P 6650 3250
-F 0 "#PWR0106" H 6650 3100 50  0001 C CNN
-F 1 "+5VL" H 6665 3423 50  0000 C CNN
-F 2 "" H 6650 3250 50  0001 C CNN
-F 3 "" H 6650 3250 50  0001 C CNN
-	1    6650 3250
-	1    0    0    -1
-$EndComp
-$Comp
 L power:GND #PWR0102
 U 1 1 5DA7416D
@@
 Wire Wire Line
 	4500 3400 4400 3400
-Wire Wire Line
-	4500 3300 4400 3300
-Wire Wire Line
-	6650 3250 6550 3250
 Wire Wire Line
 	3500 4800 3450 4800
@@
 P 1050 5350
 F 0 "R5" V 1150 5300 50  0000 L CNN
-F 1 "500" V 1050 5300 50  0000 L CNN
+F 1 "330" V 1050 5300 50  0000 L CNN
 F 2 "Resistor_SMD:R_0603_1608Metric_Pad1.05x0.95mm_HandSolder" V 980 5350 50  0001 C CNN
 F 3 "~" H 1050 5350 50  0001 C CNN
@@
 P 1050 2750
 F 0 "R1" V 1150 2700 50  0000 L CNN
-F 1 "500" V 1050 2700 50  0000 L CNN
+F 1 "330" V 1050 2700 50  0000 L CNN
 F 2 "Resistor_SMD:R_0603_1608Metric_Pad1.05x0.95mm_HandSolder" V 980 2750 50  0001 C CNN
 F 3 "~" H 1050 2750 50  0001 C CNN
@@
 	1    0    0    -1
 $EndComp
+Wire Wire Line
+	800  2250 850  2250
+$Comp
+L power:+3V3 #PWR?
+U 1 1 5E4FC442
+P 4550 1050
+F 0 "#PWR?" H 4550 900 50  0001 C CNN
+F 1 "+3V3" H 4565 1223 50  0000 C CNN
+F 2 "" H 4550 1050 50  0001 C CNN
+F 3 "" H 4550 1050 50  0001 C CNN
+	1    4550 1050
+	1    0    0    -1
+$EndComp
+$Comp
+L power:+3V3 #PWR?
+U 1 1 5E51951A
+P 800 2250
+F 0 "#PWR?" H 800 2100 50  0001 C CNN
+F 1 "+3V3" H 815 2423 50  0000 C CNN
+F 2 "" H 800 2250 50  0001 C CNN
+F 3 "" H 800 2250 50  0001 C CNN
+	1    800  2250
+	1    0    0    -1
+$EndComp
+NoConn ~ 6550 3250
+NoConn ~ 4400 3300
 $EndSCHEMATC

Commit message: BOM
Parts:
- U2: value OKI -> OKI_3V3
- U3: value OKI -> OKI_5V
Changed lines of the file:
@@
 P 3900 1200
 F 0 "U2" H 3950 1150 60  0001 C CNN
-F 1 "OKI" H 4100 1481 60  0000 C CNN
+F 1 "OKI_3V3" H 4100 1481 60  0000 C CNN
 F 2 "MRDT_Devices:OKI_Horizontal" H 3700 1100 60  0001 C CNN
 F 3 "" H 3700 1100 60  0001 C CNN
@@
 P 3100 1950
 F 0 "U3" H 3150 1900 60  0001 C CNN
-F 1 "OKI" H 3300 2231 60  0000 C CNN
+F 1 "OKI_5V" H 3300 2231 60  0000 C CNN
 F 2 "MRDT_Devices:OKI_Horizontal" H 2900 1850 60  0001 C CNN
 F 3 "" H 2900 1850 60  0001 C CNN
@@
 	800  2250 850  2250
 $Comp
-L power:+3V3 #PWR?
+L power:+3V3 #PWR0106
 U 1 1 5E4FC442
 P 4550 1050
-F 0 "#PWR?" H 4550 900 50  0001 C CNN
+F 0 "#PWR0106" H 4550 900 50  0001 C CNN
 F 1 "+3V3" H 4565 1223 50  0000 C CNN
 F 2 "" H 4550 1050 50  0001 C CNN
@@
 $EndComp
 $Comp
-L power:+3V3 #PWR?
+L power:+3V3 #PWR0109
 U 1 1 5E51951A
 P 800 2250
-F 0 "#PWR?" H 800 2100 50  0001 C CNN
+F 0 "#PWR0109" H 800 2100 50  0001 C CNN
 F 1 "+3V3" H 815 2423 50  0000 C CNN
 F 2 "" H 800 2250 50  0001 C CNN
