File: Gimbal_Board.kicad_pcb (KiCad board)
At the start: 2 copper layers, 54 parts, among them Q1 2N3904, Q2 2N3904, Q3 2N3904, Q4 2N3904, Q5 2N3904, Q6 2N3904, Q7 2N3904, Q8 2N3904, U1 TM4C129E_Launchpad, U2 OKI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

Commit message: PCB first layout complete
Finished first PCB layout and ratsnest.
Parts:
- moved D8 136.4 mm to (186.9, 74.8), turned to 90 degrees
- moved Q2 127.7 mm to (91.9, 84.8), turned to 270 degrees
- moved R8 110.1 mm to (186.9, 70.1), turned to 270 degrees
- moved R16 109.4 mm to (181.9, 70.2), turned to 90 degrees
- moved R7 105.8 mm to (170.2, 70.2), turned to 270 degrees
- moved R15 100.6 mm to (165.1, 70.1), turned to 90 degrees
- moved C1 91.2 mm to (164.6, 96.2), turned to 270 degrees
- moved R3 89.8 mm to (86.9, 69.1)
- moved Q7 89.0 mm to (166.6, 75.7), turned to 180 degrees
- moved D6 88.2 mm to (128.0, 74.7), turned to 90 degrees
- moved Q8 87.0 mm to (183.4, 75.7), turned to 180 degrees
- moved D5 85.5 mm to (115.3, 74.7), turned to 90 degrees
- moved D3 79.8 mm to (91.4, 69.1), turned to 180 degrees
- moved R13 77.9 mm to (110.7, 70.2), turned to 90 degrees
- moved U2 77.3 mm to (160.0, 91.9), turned to 270 degrees
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- renumbered R17 to R16, R8 to R17, R7 to R18, R16 to R7, R18 to R8
Routing:
- net +5VL: track 0.00 -> 91.0 mm
- net Servo_Ctrl_3: track 0.00 -> 78.4 mm
- net Servo_Ctrl_2: track 0.00 -> 69.9 mm
- net Servo_Ctrl_4: track 0.00 -> 68.0 mm
- net Servo_Ctrl_1: track 0.00 -> 61.6 mm
- net GND: track 0.00 -> 47.3 mm
- net Servo_Ctrl_8: track 0.00 -> 46.9 mm
- net Servo_Ctrl_7: track 0.00 -> 32.1 mm
- net Servo_Ctrl_5: track 0.00 -> 27.5 mm
- net Servo_Ctrl_6: track 0.00 -> 19.1 mm
- net +12VA: track 0.00 -> 12.0 mm
- net +12L: track 0.00 -> 10.9 mm
- net Net-(D3-Pad1): track 0.00 -> 7.40 mm
- net Net-(D2-Pad1): track 0.00 -> 7.40 mm
- net Net-(D5-Pad1): track 0.00 -> 7.25 mm
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- added copper zone on F.Cu, net +5VA
- added copper zone on B.Cu, net GND
