File: Gimbal_Board.sch (KiCad schematic (older format))
At the start: 54 parts, among them Q1 2N3904, Q2 2N3904, Q3 2N3904, Q4 2N3904, Q5 2N3904, Q6 2N3904, Q7 2N3904, Q8 2N3904, U1 TM4C129E_Launchpad, U2 OKI, U3 OKI

Commit message: Footprints Assigned, Netlist Generated, and PCB layout started
As it is in the title.  Connecters and anderson placed on board. Servo pins changed.
Parts:
- C1, C2, C3, C4: footprint (none) -> Capacitor_SMD:C_0603_1608Metric_Pad1.05x0.95mm_HandSolder
- C5, C6: footprint (none) -> Capacitor_THT:CP_Radial_D8.0mm_P3.50mm
- Conn1, Conn2, Conn3, Conn4, Conn5, Conn6, Conn7, Conn8: footprint (none) -> MRDT_Connectors:MOLEX_SL_03_Horizontal
- Conn9: footprint (none) -> MRDT_Connectors:Anderson_3_Horizontal_Side_by_Side
- D1, D10, D2, D3, D4, D5, D6, D7, D8, D9: footprint (none) -> Diode_SMD:D_0603_1608Metric_Pad1.05x0.95mm_HandSolder
- R1, R10, R11, R12, R13, R14, R15, R16, R17, R18, R2, R3, R4, R5, R6, R7, R8, R9: footprint (none) -> Resistor_SMD:R_0603_1608Metric_Pad1.05x0.95mm_HandSolder
- U1: footprint (none) -> MRDT_Shields:TM4C129E_Launchpad_FULL_THT_BOTTOM
- U2, U3: footprint (none) -> MRDT_Devices:OKI_Horizontal
Connections:
- net Servo_Ctrl_1: now also U1.PD2 (A2_2); no longer U1.PM7 (D2_2)
- net Servo_Ctrl_2: now also U1.PP0 (A2_3); no longer U1.PA7 (D2_4)
- net Servo_Ctrl_3: now also U1.PP1 (A2_4); no longer U1.PM6 (D2_10)
- net Servo_Ctrl_4: now also U1.PD4 (A2_5); no longer U1.PM1 (C2_5)
- net Servo_Ctrl_5: now also U1.PG1 (C2_1); no longer U1.PM0 (C2_4)
- net Servo_Ctrl_6: now also U1.PK4 (C2_2); no longer U1.PK5 (C2_3)
- net Servo_Ctrl_7: now also U1.PK5 (C2_3); no longer U1.PK4 (C2_2)
- net Servo_Ctrl_8: now also U1.PM0 (C2_4); no longer U1.PG1 (C2_1)
Other:
- note added: "PMW 1"
- note added: "PMW 2"
- note added: "PMW 3"
- note added: "PMW 4"

Commit message: PMW to PWM
Other:
- note added: "PWM 1"
- note added: "PWM 2"
- note added: "PWM 3"
- note added: "PWM 4"
- note added: "PWM 5"
- note added: "PWM 6"
- note added: "PWM 7"
- note removed: "PMW 1"
- note removed: "PMW 2"
- note removed: "PMW 3"
- note removed: "PMW 4"
- note removed: "PMW 5"
- note removed: "PMW 6"
- note removed: "PMW 7"
Changed lines of the file:
@@
 Wire Notes Line
 	7350 500  7350 2950
-Text Notes 2700 4900 0    50   ~ 0
-PMW 5
-Text Notes 2700 5000 0    50   ~ 0
-PMW 6
 Wire Wire Line
 	3600 4850 3500 4850
@@
 Wire Wire Line
 	4550 4850 4500 4850
-Text Notes 2700 5100 0    50   ~ 0
-PMW 7
 Text Notes 2550 5200 0    50   ~ 0
 AlalogWrite
@@
 Wire Wire Line
 	3500 5150 3600 5150
+Text Notes 2700 3800 0    50   ~ 0
+PWM 1
+Text Notes 2700 3900 0    50   ~ 0
+PWM 2
+Text Notes 2700 4000 0    50   ~ 0
+PWM 3
 Text Notes 2700 4100 0    50   ~ 0
-PMW 4
-Text Notes 2700 4000 0    50   ~ 0
-PMW 3
-Text Notes 2700 3900 0    50   ~ 0
-PMW 2
-Text Notes 2700 3800 0    50   ~ 0
-PMW 1
+PWM 4
+Text Notes 2700 4900 0    50   ~ 0
+PWM 5
+Text Notes 2700 5000 0    50   ~ 0
+PWM 6
+Text Notes 2700 5100 0    50   ~ 0
+PWM 7
 $EndSCHEMATC

Commit message: Minor Schematic changes
Labeling and numbering for resistors
Parts:
- renumbered R17 to R16, R8 to R17, R7 to R18, R16 to R7, R18 to R8
Changed lines of the file:
@@
 $EndComp
 $Comp
-L Device:R R7
+L Device:R R18
 U 1 1 5D93B51A
 P 700 1450
-F 0 "R7" V 493 1450 50  0001 C CNN
+F 0 "R18" V 493 1450 50  0001 C CNN
 F 1 "1000" V 700 1450 50  0000 C CNN
 F 2 "Resistor_SMD:R_0603_1608Metric_Pad1.05x0.95mm_HandSolder" V 630 1450 50  0001 C CNN
@@
 $EndComp
 $Comp
-L Device:R R8
+L Device:R R17
 U 1 1 5D93B508
 P 1050 1450
-F 0 "R8" V 843 1450 50  0001 C CNN
+F 0 "R17" V 843 1450 50  0001 C CNN
 F 1 "1000" V 1050 1450 50  0000 C CNN
 F 2 "Resistor_SMD:R_0603_1608Metric_Pad1.05x0.95mm_HandSolder" V 980 1450 50  0001 C CNN
@@
 	6550 1800 6550 1900
 $Comp
-L Device:R R18
+L Device:R R8
 U 1 1 5D98C67E
 P 6900 1450
-F 0 "R18" H 6970 1496 50  0000 L CNN
+F 0 "R8" H 6970 1496 50  0000 L CNN
 F 1 "100" V 6900 1400 50  0000 L CNN
 F 2 "Resistor_SMD:R_0603_1608Metric_Pad1.05x0.95mm_HandSolder" V 6830 1450 50  0001 C CNN
@@
 $EndComp
 $Comp
-L Device:R R17
+L Device:R R16
 U 1 1 5D98C690
 P 6550 2050
-F 0 "R17" V 6450 2050 50  0000 C CNN
+F 0 "R16" V 6450 2050 50  0000 C CNN
 F 1 "100" V 6550 2050 50  0000 C CNN
 F 2 "Resistor_SMD:R_0603_1608Metric_Pad1.05x0.95mm_HandSolder" V 6480 2050 50  0001 C CNN
@@
 	5800 1800 5800 1900
 $Comp
-L Device:R R16
+L Device:R R7
 U 1 1 5D98C69D
 P 6150 1450
-F 0 "R16" H 6220 1496 50  0000 L CNN
+F 0 "R7" H 6220 1496 50  0000 L CNN
 F 1 "100" V 6150 1400 50  0000 L CNN
 F 2 "Resistor_SMD:R_0603_1608Metric_Pad1.05x0.95mm_HandSolder" V 6080 1450 50  0001 C CNN
