File: Hardware/gimble_board/GimbleBoard04.sch (KiCad schematic (older format))
At the start: 1 part, among them U3 TM4C129E_Launchpad

Commit message: footprints
Parts:
- U3: footprint (none) -> MRDT_Shields:TM4C129E_Launchpad_FULL_THT_TOP
Changed lines of the file:
@@
 EESchema Schematic File Version 4
+LIBS:gimble_board-cache
 EELAYER 30 0
 EELAYER END
@@
 F 0 "U3" H 2500 2450 60  0000 L CNN
 F 1 "TM4C129E_Launchpad" H 3150 2600 60  0001 L CNN
-F 2 "" H 2450 2500 60  0001 C CNN
+F 2 "MRDT_Shields:TM4C129E_Launchpad_FULL_THT_TOP" H 2450 2500 60  0001 C CNN
 F 3 "" H 2450 2500 60  0001 C CNN
 	1    2450 2500
@@
 F 0 "U3" H 3200 2450 60  0000 C CNN
 F 1 "TM4C129E_Launchpad" H 3081 3671 60  0001 C CNN
-F 2 "" H 3050 2500 60  0001 C CNN
+F 2 "MRDT_Shields:TM4C129E_Launchpad_FULL_THT_TOP" H 3050 2500 60  0001 C CNN
 F 3 "" H 3050 2500 60  0001 C CNN
 	2    3050 2500
@@
 F 0 "U3" H 4550 2450 60  0000 L CNN
 F 1 "TM4C129E_Launchpad" H 4805 2992 60  0001 L CNN
-F 2 "" H 4500 2500 60  0001 C CNN
+F 2 "MRDT_Shields:TM4C129E_Launchpad_FULL_THT_TOP" H 4500 2500 60  0001 C CNN
 F 3 "" H 4500 2500 60  0001 C CNN
 	3    4500 2500
@@
 F 0 "U3" H 5250 2450 60  0000 C CNN
 F 1 "TM4C129E_Launchpad" H 5131 3671 60  0001 C CNN
-F 2 "" H 5100 2500 60  0001 C CNN
+F 2 "MRDT_Shields:TM4C129E_Launchpad_FULL_THT_TOP" H 5100 2500 60  0001 C CNN
 F 3 "" H 5100 2500 60  0001 C CNN
 	4    5100 2500
@@
 F 0 "U3" H 2500 3900 60  0000 L CNN
 F 1 "TM4C129E_Launchpad" H 2751 4442 60  0001 L CNN
-F 2 "" H 2450 3950 60  0001 C CNN
+F 2 "MRDT_Shields:TM4C129E_Launchpad_FULL_THT_TOP" H 2450 3950 60  0001 C CNN
 F 3 "" H 2450 3950 60  0001 C CNN
 	5    2450 3950
@@
 F 0 "U3" H 3200 3900 60  0000 C CNN
 F 1 "TM4C129E_Launchpad" H 3081 5121 60  0001 C CNN
-F 2 "" H 3050 3950 60  0001 C CNN
+F 2 "MRDT_Shields:TM4C129E_Launchpad_FULL_THT_TOP" H 3050 3950 60  0001 C CNN
 F 3 "" H 3050 3950 60  0001 C CNN
 	6    3050 3950
@@
 F 0 "U3" H 4550 3900 60  0000 L CNN
 F 1 "TM4C129E_Launchpad" H 4805 4442 60  0001 L CNN
-F 2 "" H 4500 3950 60  0001 C CNN
+F 2 "MRDT_Shields:TM4C129E_Launchpad_FULL_THT_TOP" H 4500 3950 60  0001 C CNN
 F 3 "" H 4500 3950 60  0001 C CNN
 	7    4500 3950
@@
 F 0 "U3" H 5250 3900 60  0000 C CNN
 F 1 "TM4C129E_Launchpad" H 5131 5121 60  0001 C CNN
-F 2 "" H 5100 3950 60  0001 C CNN
+F 2 "MRDT_Shields:TM4C129E_Launchpad_FULL_THT_TOP" H 5100 3950 60  0001 C CNN
 F 3 "" H 5100 3950 60  0001 C CNN
 	8    5100 3950
@@
 $EndComp
 $Comp
-L power:+3.3V #PWR049
+L power:+3.3V #PWR028
 U 1 1 5F8A68ED
 P 2100 1400
-F 0 "#PWR049" H 2100 1250 50  0001 C CNN
+F 0 "#PWR028" H 2100 1250 50  0001 C CNN
 F 1 "+3.3V" H 2115 1573 50  0000 C CNN
 F 2 "" H 2100 1400 50  0001 C CNN
@@
 	4150 1750 4300 1750
 $Comp
-L power:GND #PWR053
+L power:GND #PWR032
 U 1 1 5F8AA7DC
 P 5450 1550
-F 0 "#PWR053" H 5450 1300 50  0001 C CNN
+F 0 "#PWR032" H 5450 1300 50  0001 C CNN
 F 1 "GND" H 5455 1377 50  0000 C CNN
 F 2 "" H 5450 1550 50  0001 C CNN
@@
 $EndComp
 $Comp
-L power:GND #PWR054
+L power:GND #PWR033
 U 1 1 5F8ABA51
 P 5450 3000
-F 0 "#PWR054" H 5450 2750 50  0001 C CNN
+F 0 "#PWR033" H 5450 2750 50  0001 C CNN
 F 1 "GND" H 5455 2827 50  0000 C CNN
 F 2 "" H 5450 3000 50  0001 C CNN
@@
 NoConn ~ 4300 2450
 $Comp
-L power:GND #PWR051
+L power:GND #PWR030
 U 1 1 5F8ADF38
 P 3400 1650
-F 0 "#PWR051" H 3400 1400 50  0001 C CNN
+F 0 "#PWR030" H 3400 1400 50  0001 C CNN
 F 1 "GND" H 3405 1477 50  0000 C CNN
 F 2 "" H 3400 1650 50  0001 C CNN
@@
 NoConn ~ 4300 3900
 $Comp
-L power:GND #PWR052
+L power:GND #PWR031
 U 1 1 5F8EF5BF
 P 3400 3100
-F 0 "#PWR052" H 3400 2850 50  0001 C CNN
+F 0 "#PWR031" H 3400 2850 50  0001 C CNN
 F 1 "GND" H 3405 2927 50  0000 C CNN
 F 2 "" H 3400 3100 50  0001 C CNN
@@
 	3250 3100 3400 3100
 $Comp
-L power:+3.3V #PWR050
+L power:+3.3V #PWR029
 U 1 1 5F8F0066
 P 2100 2850
-F 0 "#PWR050" H 2100 2700 50  0001 C CNN
+F 0 "#PWR029" H 2100 2700 50  0001 C CNN
 F 1 "+3.3V" H 2115 3023 50  0000 C CNN
 F 2 "" H 2100 2850 50  0001 C CNN

Commit message: start layout
Connections:
- net Servo_8_PWM is gone; now on net Servo_7_PWM: U3.PK5 (C2_3)
- net Servo_1_SW: now also U3.PM5 (B1_10); no longer U3.PE4 (A1_2)
- net Servo_2_SW: now also U3.PM4 (B1_9); no longer U3.PC4 (A1_3)
- net Servo_3_SW: now also U3.PA6 (B1_8); no longer U3.PC5 (A1_4)
- net Servo_4_SW: now also U3.PD7 (B1_7); no longer U3.PC6 (A1_5)
- net Servo_5_SW: now also U3.PE3 (B1_6); no longer U3.PE5 (A1_6)
- net Servo_6_PWM: now also U3.PK4 (C2_2); no longer U3.PG1 (C2_1)
- net Servo_6_SW: now also U3.PE2 (B1_5); no longer U3.PD3 (A1_7)
- net Servo_7_PWM: no longer U3.PK4 (C2_2)
- net Servo_7_SW: now also U3.PE1 (B1_4); no longer U3.PC7 (A1_8)
- net Servo_8_SW: now also U3.PE0 (B1_3); no longer U3.PB2 (A1_9)
- net Servo_Digital_Control: now also U3.PA4 (B2_9); no longer U3.PP0 (A2_3)
- net Servo_Manual_Control: now also U3.PA5 (B2_10); no longer U3.PD2 (A2_2)
- net Servo_8_AW: now reaches U3.PM0 (C2_4)
- net Servo_5_AW: no longer names the net of U3.PL4 (C1_5)
- new net Servo_5_PWM: U3.PG1 (C2_1)
Other:
- moved on the sheet: U3A, U3B, U3E, U3F
Changed lines of the file:
@@
 EESchema Schematic File Version 4
-LIBS:gimble_board-cache
 EELAYER 30 0
 EELAYER END
@@
 L MRDT_Shields:TM4C129E_Launchpad U3
 U 1 1 5F85C869
+P 1850 2500
+F 0 "U3" H 1900 2450 60  0000 L CNN
+F 1 "TM4C129E_Launchpad" H 2550 2600 60  0001 L CNN
+F 2 "MRDT_Shields:TM4C129E_Launchpad_FULL_THT_TOP" H 1850 2500 60  0001 C CNN
+F 3 "" H 1850 2500 60  0001 C CNN
+	1    1850 2500
+	1    0    0    -1
+$EndComp
+$Comp
+L MRDT_Shields:TM4C129E_Launchpad U3
+U 2 1 5F860DB3
 P 2450 2500
-F 0 "U3" H 2500 2450 60  0000 L CNN
-F 1 "TM4C129E_Launchpad" H 3150 2600 60  0001 L CNN
+F 0 "U3" H 2600 2450 60  0000 C CNN
+F 1 "TM4C129E_Launchpad" H 2481 3671 60  0001 C CNN
 F 2 "MRDT_Shields:TM4C129E_Launchpad_FULL_THT_TOP" H 2450 2500 60  0001 C CNN
 F 3 "" H 2450 2500 60  0001 C CNN
-	1    2450 2500
-	1    0    0    -1
-$EndComp
-$Comp
-L MRDT_Shields:TM4C129E_Launchpad U3
-U 2 1 5F860DB3
-P 3050 2500
-F 0 "U3" H 3200 2450 60  0000 C CNN
-F 1 "TM4C129E_Launchpad" H 3081 3671 60  0001 C CNN
-F 2 "MRDT_Shields:TM4C129E_Launchpad_FULL_THT_TOP" H 3050 2500 60  0001 C CNN
-F 3 "" H 3050 2500 60  0001 C CNN
-	2    3050 2500
+	2    2450 2500
 	-1   0    0    -1
 $EndComp
@@
 L MRDT_Shields:TM4C129E_Launchpad U3
 U 5 1 5F873BAC
+P 1850 3950
+F 0 "U3" H 1900 3900 60  0000 L CNN
+F 1 "TM4C129E_Launchpad" H 2151 4442 60  0001 L CNN
+F 2 "MRDT_Shields:TM4C129E_Launchpad_FULL_THT_TOP" H 1850 3950 60  0001 C CNN
+F 3 "" H 1850 3950 60  0001 C CNN
+	5    1850 3950
+	1    0    0    -1
+$EndComp
+$Comp
+L MRDT_Shields:TM4C129E_Launchpad U3
+U 6 1 5F87567D
 P 2450 3950
-F 0 "U3" H 2500 3900 60  0000 L CNN
-F 1 "TM4C129E_Launchpad" H 2751 4442 60  0001 L CNN
+F 0 "U3" H 2600 3900 60  0000 C CNN
+F 1 "TM4C129E_Launchpad" H 2481 5121 60  0001 C CNN
 F 2 "MRDT_Shields:TM4C129E_Launchpad_FULL_THT_TOP" H 2450 3950 60  0001 C CNN
 F 3 "" H 2450 3950 60  0001 C CNN
-	5    2450 3950
-	1    0    0    -1
-$EndComp
-$Comp
-L MRDT_Shields:TM4C129E_Launchpad U3
-U 6 1 5F87567D
-P 3050 3950
-F 0 "U3" H 3200 3900 60  0000 C CNN
-F 1 "TM4C129E_Launchpad" H 3081 5121 60  0001 C CNN
-F 2 "MRDT_Shields:TM4C129E_Launchpad_FULL_THT_TOP" H 3050 3950 60  0001 C CNN
-F 3 "" H 3050 3950 60  0001 C CNN
-	6    3050 3950
+	6    2450 3950
 	-1   0    0    -1
 $EndComp
@@
 L power:+3.3V #PWR028
 U 1 1 5F8A68ED
-P 2100 1400
-F 0 "#PWR028" H 2100 1250 50  0001 C CNN
-F 1 "+3.3V" H 2115 1573 50  0000 C CNN
-F 2 "" H 2100 1400 50  0001 C CNN
-F 3 "" H 2100 1400 50  0001 C CNN
-	1    2100 1400
-	1    0    0    -1
-$EndComp
-Wire Wire Line
-	2100 1400 2100 1550
-Wire Wire Line
-	2100 1550 2250 1550
+P 1500 1400
+F 0 "#PWR028" H 1500 1250 50  0001 C CNN
+F 1 "+3.3V" H 1515 1573 50  0000 C CNN
+F 2 "" H 1500 1400 50  0001 C CNN
+F 3 "" H 1500 1400 50  0001 C CNN
+	1    1500 1400
+	1    0    0    -1
+$EndComp
+Wire Wire Line
+	1500 1400 1500 1550
+Wire Wire Line
+	1500 1550 1650 1550
 Text GLabel 4150 1550 0    39   Output ~ 0
 Servo_1_PWM
@@
 L power:GND #PWR030
 U 1 1 5F8ADF38
-P 3400 1650
-F 0 "#PWR030" H 3400 1400 50  0001 C CNN
-F 1 "GND" H 3405 1477 50  0000 C CNN
-F 2 "" H 3400 1650 50  0001 C CNN
-F 3 "" H 3400 1650 50  0001 C CNN
-	1    3400 1650
-	1    0    0    -1
-$EndComp
-Wire Wire Line
-	3250 1650 3400 1650
-NoConn ~ 3250 1550
-Text GLabel 4150 3000 0    39   Output ~ 0
+P 2800 1650
+F 0 "#PWR030" H 2800 1400 50  0001 C CNN
+F 1 "GND" H 2805 1477 50  0000 C CNN
+F 2 "" H 2800 1650 50  0001 C CNN
+F 3 "" H 2800 1650 50  0001 C CNN
+	1    2800 1650
+	-1   0    0    1
+$EndComp
+Wire Wire Line
+	2650 1650 2800 1650
+NoConn ~ 2650 1550
+Text GLabel 4150 3100 0    39   Output ~ 0
 Servo_6_PWM
-Text GLabel 4150 3100 0    39   Output ~ 0
+Text GLabel 4150 3200 0    39   Output ~ 0
 Servo_7_PWM
-Text GLabel 4150 3200 0    39   Output ~ 0
-Servo_8_PWM
+Text GLabel 4150 3300 0    39   Output ~ 0
+Servo_8_AW
 Wire Wire Line
 	4150 3000 4300 3000
@@
 Text GLabel 4150 1850 0    39   Output ~ 0
 Servo_4_PWM
-Text GLabel 4150 1950 0    39   Output ~ 0
-Servo_5_AW
 Wire Wire Line
 	4150 1850 4300 1850
-Wire Wire Line
-	4150 1950 4300 1950
-NoConn ~ 4300 3300
+NoConn ~ 4300 1950
 NoConn ~ 4300 3400
 NoConn ~ 4300 3500
@@
 L power:GND #PWR031
 U 1 1 5F8EF5BF
-P 3400 3100
-F 0 "#PWR031" H 3400 2850 50  0001 C CNN
-F 1 "GND" H 3405 2927 50  0000 C CNN
-F 2 "" H 3400 3100 50  0001 C CNN
-F 3 "" H 3400 3100 50  0001 C CNN
-	1    3400 3100
-	1    0    0    -1
-$EndComp
-Wire Wire Line
-	3250 3100 3400 3100
+P 2800 3100
+F 0 "#PWR031" H 2800 2850 50  0001 C CNN
+F 1 "GND" H 2805 2927 50  0000 C CNN
+F 2 "" H 2800 3100 50  0001 C CNN
+F 3 "" H 2800 3100 50  0001 C CNN
+	1    2800 3100
+	1    0    0    -1
+$EndComp
+Wire Wire Line
+	2650 3100 2800 3100
 $Comp
 L power:+3.3V #PWR029
 U 1 1 5F8F0066
-P 2100 2850
-F 0 "#PWR029" H 2100 2700 50  0001 C CNN
-F 1 "+3.3V" H 2115 3023 50  0000 C CNN
-F 2 "" H 2100 2850 50  0001 C CNN
-F 3 "" H 2100 2850 50  0001 C CNN
-	1    2100 2850
-	1    0    0    -1
-$EndComp
-Wire Wire Line
-	2100 2850 2100 3000
-Wire Wire Line
-	2100 3000 2250 3000
-NoConn ~ 3250 3000
-Text GLabel 2100 1650 0    39   Input ~ 0
+P 1500 2850
+F 0 "#PWR029" H 1500 2700 50  0001 C CNN
+F 1 "+3.3V" H 1515 3023 50  0000 C CNN
+F 2 "" H 1500 2850 50  0001 C CNN
+F 3 "" H 1500 2850 50  0001 C CNN
+	1    1500 2850
+	1    0    0    -1
+$EndComp
+Wire Wire Line
+	1500 2850 1500 3000
+Wire Wire Line
+	1500 3000 1650 3000
+NoConn ~ 2650 3000
+Text GLabel 2650 2450 2    39   Input ~ 0
 Servo_1_SW
-Text GLabel 2100 1750 0    39   Input ~ 0
+Text GLabel 2650 2350 2    39   Input ~ 0
 Servo_2_SW
-Text GLabel 2100 1850 0    39   Input ~ 0
+Text GLabel 2650 2250 2    39   Input ~ 0
 Servo_3_SW
 Wire Wire Line
-	2100 1650 2250 1650
-Wire Wire Line
-	2100 1750 2250 1750
-Wire Wire Line
-	2100 1850 2250 1850
-Text GLabel 2100 1950 0    39   Input ~ 0
+	1500 1650 1650 1650
+Wire Wire Line
+	1500 1750 1650 1750
+Wire Wire Line
+	1500 1850 1650 1850
+Text GLabel 2650 2150 2    39   Input ~ 0
 Servo_4_SW
-Text GLabel 2100 2050 0    39   Input ~ 0
+Text GLabel 2650 2050 2    39   Input ~ 0
 Servo_5_SW
 Wire Wire Line
-	2100 1950 2250 1950
-Wire Wire Line
-	2100 2050 2250 2050
-Text GLabel 2100 2150 0    39   Input ~ 0
+	1500 1950 1650 1950
+Wire Wire Line
+	1500 2050 1650 2050
+Text GLabel 2650 1950 2    39   Input ~ 0
 Servo_6_SW
-Text GLabel 2100 2250 0    39   Input ~ 0
+Text GLabel 2650 1850 2    39   Input ~ 0
 Servo_7_SW
-Text GLabel 2100 2350 0    39   Input ~ 0
+Text GLabel 2650 1750 2    39   Input ~ 0
 Servo_8_SW
 Wire Wire Line
-	2100 2150 2250 2150
-Wire Wire Line
-	2100 2250 2250 2250
-Wire Wire Line
-	2100 2350 2250 2350
-Text GLabel 2100 3100 0    39   Input ~ 0
+	1500 2150 1650 2150
+Wire Wire Line
+	1500 2250 1650 2250
+Wire Wire Line
+	1500 2350 1650 2350
+Text GLabel 2800 3900 2    39   Input ~ 0
 Servo_Manual_Control
 Wire Wire Line
-	2100 2450 2250 2450
+	1500 2450 1650 2450
 NoConn ~ 4300 2050
 NoConn ~ 5300 3100
@@
 NoConn ~ 5300 1750
 NoConn ~ 5300 1650
-NoConn ~ 3250 2450
-NoConn ~ 3250 2350
-NoConn ~ 3250 2250
-NoConn ~ 3250 2150
-NoConn ~ 3250 2050
-NoConn ~ 3250 1950
-NoConn ~ 3250 1850
-NoConn ~ 3250 1750
-NoConn ~ 2250 3300
-NoConn ~ 2250 3400
-NoConn ~ 2250 3500
-NoConn ~ 2250 3600
-NoConn ~ 2250 3700
-NoConn ~ 2250 3800
-NoConn ~ 2250 3900
-NoConn ~ 3250 3200
-NoConn ~ 3250 3300
-NoConn ~ 3250 3400
-NoConn ~ 3250 3500
-NoConn ~ 3250 3800
-NoConn ~ 3250 3900
-NoConn ~ 3250 3600
-NoConn ~ 3250 3700
-Text GLabel 2100 3200 0    39   Input ~ 0
+NoConn ~ 1500 1950
+NoConn ~ 1500 2350
+NoConn ~ 1500 2250
+NoConn ~ 1500 2150
+NoConn ~ 1500 2050
+NoConn ~ 1500 1850
+NoConn ~ 1500 1750
+NoConn ~ 1500 1650
+NoConn ~ 1650 3300
+NoConn ~ 1650 3400
+NoConn ~ 1650 3500
+NoConn ~ 1650 3600
+NoConn ~ 1650 3700
+NoConn ~ 1650 3800
+NoConn ~ 1650 3900
+NoConn ~ 2650 3200
+NoConn ~ 2650 3300
+NoConn ~ 2650 3400
+NoConn ~ 2650 3500
+NoConn ~ 1650 3200
+NoConn ~ 1650 3100
+NoConn ~ 2650 3600
+NoConn ~ 2650 3700
+Text GLabel 2800 3800 2    39   Input ~ 0
 Servo_Digital_Control
-Wire Wire Line
-	2100 3100 2250 3100
-Wire Wire Line
-	2100 3200 2250 3200
 Text Notes 3050 1000 0    79   ~ 0
 Tiva Headers
 Text Notes 7200 6950 0    157  ~ 0
 Sheet 04: Tiva
-NoConn ~ 2100 2450
+NoConn ~ 1500 2450
+Wire Wire Line
+	4150 3300 4300 3300
+Text GLabel 4150 3000 0    39   Output ~ 0
+Servo_5_PWM
+Wire Wire Line
+	2650 3800 2800 3800
+Wire Wire Line
+	2650 3900 2800 3900
 $EndSCHEMATC

Commit message: layout 2
Connections:
- net Servo_1_SW: now also U3.PE0 (B1_3); no longer U3.PM5 (B1_10)
- net Servo_2_SW: now also U3.PE1 (B1_4); no longer U3.PM4 (B1_9)
- net Servo_3_SW: now also U3.PE2 (B1_5); no longer U3.PA6 (B1_8)
- net Servo_4_SW: now also U3.PE3 (B1_6); no longer U3.PD7 (B1_7)
- net Servo_5_SW: now also U3.PD7 (B1_7); no longer U3.PE3 (B1_6)
- net Servo_6_SW: now also U3.PA6 (B1_8); no longer U3.PE2 (B1_5)
- net Servo_7_SW: now also U3.PM4 (B1_9); no longer U3.PE1 (B1_4)
- net Servo_8_SW: now also U3.PM5 (B1_10); no longer U3.PE0 (B1_3)
Changed lines of the file:
@@
 	1500 3000 1650 3000
 NoConn ~ 2650 3000
-Text GLabel 2650 2450 2    39   Input ~ 0
+Text GLabel 2650 1750 2    39   Input ~ 0
 Servo_1_SW
-Text GLabel 2650 2350 2    39   Input ~ 0
+Text GLabel 2650 1850 2    39   Input ~ 0
 Servo_2_SW
-Text GLabel 2650 2250 2    39   Input ~ 0
+Text GLabel 2650 1950 2    39   Input ~ 0
 Servo_3_SW
 Wire Wire Line
@@
 Wire Wire Line
 	1500 1850 1650 1850
+Text GLabel 2650 2050 2    39   Input ~ 0
+Servo_4_SW
 Text GLabel 2650 2150 2    39   Input ~ 0
-Servo_4_SW
-Text GLabel 2650 2050 2    39   Input ~ 0
 Servo_5_SW
 Wire Wire Line
@@
 Wire Wire Line
 	1500 2050 1650 2050
-Text GLabel 2650 1950 2    39   Input ~ 0
+Text GLabel 2650 2250 2    39   Input ~ 0
 Servo_6_SW
-Text GLabel 2650 1850 2    39   Input ~ 0
+Text GLabel 2650 2350 2    39   Input ~ 0
 Servo_7_SW
-Text GLabel 2650 1750 2    39   Input ~ 0
+Text GLabel 2650 2450 2    39   Input ~ 0
 Servo_8_SW
 Wire Wire Line

Commit message: layout 3
Parts:
- U3: footprint MRDT_Shields:TM4C129E_Launchpad_FULL_THT_TOP -> MRDT_Shields:TM4C129E_Launchpad_FULL_THT_BOTTOM
Changed lines of the file:
@@
 EESchema Schematic File Version 4
+LIBS:gimble_board-cache
 EELAYER 30 0
 EELAYER END
@@
 F 0 "U3" H 1900 2450 60  0000 L CNN
 F 1 "TM4C129E_Launchpad" H 2550 2600 60  0001 L CNN
-F 2 "MRDT_Shields:TM4C129E_Launchpad_FULL_THT_TOP" H 1850 2500 60  0001 C CNN
+F 2 "MRDT_Shields:TM4C129E_Launchpad_FULL_THT_BOTTOM" H 1850 2500 60  0001 C CNN
 F 3 "" H 1850 2500 60  0001 C CNN
 	1    1850 2500
@@
 F 0 "U3" H 2600 2450 60  0000 C CNN
 F 1 "TM4C129E_Launchpad" H 2481 3671 60  0001 C CNN
-F 2 "MRDT_Shields:TM4C129E_Launchpad_FULL_THT_TOP" H 2450 2500 60  0001 C CNN
+F 2 "MRDT_Shields:TM4C129E_Launchpad_FULL_THT_BOTTOM" H 2450 2500 60  0001 C CNN
 F 3 "" H 2450 2500 60  0001 C CNN
 	2    2450 2500
@@
 F 0 "U3" H 4550 2450 60  0000 L CNN
 F 1 "TM4C129E_Launchpad" H 4805 2992 60  0001 L CNN
-F 2 "MRDT_Shields:TM4C129E_Launchpad_FULL_THT_TOP" H 4500 2500 60  0001 C CNN
+F 2 "MRDT_Shields:TM4C129E_Launchpad_FULL_THT_BOTTOM" H 4500 2500 60  0001 C CNN
 F 3 "" H 4500 2500 60  0001 C CNN
 	3    4500 2500
@@
 F 0 "U3" H 5250 2450 60  0000 C CNN
 F 1 "TM4C129E_Launchpad" H 5131 3671 60  0001 C CNN
-F 2 "MRDT_Shields:TM4C129E_Launchpad_FULL_THT_TOP" H 5100 2500 60  0001 C CNN
+F 2 "MRDT_Shields:TM4C129E_Launchpad_FULL_THT_BOTTOM" H 5100 2500 60  0001 C CNN
 F 3 "" H 5100 2500 60  0001 C CNN
 	4    5100 2500
@@
 F 0 "U3" H 1900 3900 60  0000 L CNN
 F 1 "TM4C129E_Launchpad" H 2151 4442 60  0001 L CNN
-F 2 "MRDT_Shields:TM4C129E_Launchpad_FULL_THT_TOP" H 1850 3950 60  0001 C CNN
+F 2 "MRDT_Shields:TM4C129E_Launchpad_FULL_THT_BOTTOM" H 1850 3950 60  0001 C CNN
 F 3 "" H 1850 3950 60  0001 C CNN
 	5    1850 3950
@@
 F 0 "U3" H 2600 3900 60  0000 C CNN
 F 1 "TM4C129E_Launchpad" H 2481 5121 60  0001 C CNN
-F 2 "MRDT_Shields:TM4C129E_Launchpad_FULL_THT_TOP" H 2450 3950 60  0001 C CNN
+F 2 "MRDT_Shields:TM4C129E_Launchpad_FULL_THT_BOTTOM" H 2450 3950 60  0001 C CNN
 F 3 "" H 2450 3950 60  0001 C CNN
 	6    2450 3950
@@
 F 0 "U3" H 4550 3900 60  0000 L CNN
 F 1 "TM4C129E_Launchpad" H 4805 4442 60  0001 L CNN
-F 2 "MRDT_Shields:TM4C129E_Launchpad_FULL_THT_TOP" H 4500 3950 60  0001 C CNN
+F 2 "MRDT_Shields:TM4C129E_Launchpad_FULL_THT_BOTTOM" H 4500 3950 60  0001 C CNN
 F 3 "" H 4500 3950 60  0001 C CNN
 	7    4500 3950
@@
 F 0 "U3" H 5250 3900 60  0000 C CNN
 F 1 "TM4C129E_Launchpad" H 5131 5121 60  0001 C CNN
-F 2 "MRDT_Shields:TM4C129E_Launchpad_FULL_THT_TOP" H 5100 3950 60  0001 C CNN
+F 2 "MRDT_Shields:TM4C129E_Launchpad_FULL_THT_BOTTOM" H 5100 3950 60  0001 C CNN
 F 3 "" H 5100 3950 60  0001 C CNN
 	8    5100 3950

Commit message: layout 6
Connections:
- net Servo_Digital_Control: now also U3.PE4 (A1_2); no longer U3.PA4 (B2_9)
- net Servo_Manual_Control: now also U3.PC4 (A1_3); no longer U3.PA5 (B2_10)
Changed lines of the file:
@@
 Wire Wire Line
 	1500 2350 1650 2350
-Text GLabel 2800 3900 2    39   Input ~ 0
+Text GLabel 1500 1750 0    39   Input ~ 0
 Servo_Manual_Control
 Wire Wire Line
@@
 NoConn ~ 1500 2050
 NoConn ~ 1500 1850
-NoConn ~ 1500 1750
-NoConn ~ 1500 1650
+NoConn ~ 2650 3800
+NoConn ~ 2650 3900
 NoConn ~ 1650 3300
 NoConn ~ 1650 3400
@@
 NoConn ~ 2650 3600
 NoConn ~ 2650 3700
-Text GLabel 2800 3800 2    39   Input ~ 0
+Text GLabel 1500 1650 0    39   Input ~ 0
 Servo_Digital_Control
 Text Notes 3050 1000 0    79   ~ 0
@@
 Text GLabel 4150 3000 0    39   Output ~ 0
 Servo_5_PWM
-Wire Wire Line
-	2650 3800 2800 3800
-Wire Wire Line
-	2650 3900 2800 3900
 $EndSCHEMATC
