File: Hardware/gimble_board/GimableBoard05.sch (KiCad schematic (older format))
At the start: 32 parts, among them Q1 Q_NMOS_GDS, Q2 Q_NMOS_GDS, Q3 Q_NMOS_GDS, Q4 Q_NMOS_GDS, Q5 Q_NMOS_GDS, Q6 Q_NMOS_GDS, Q7 Q_NMOS_GDS, Q8 Q_NMOS_GDS

Commit message: layout 9
Parts:
- renumbered D22 to D15, D23 to D16, D24 to D17, D25 to D18, D26 to D19, D27 to D20, D28 to D21, D29 to D22, R18 to R13, R19 to R14, R20 to R15, R21 to R16, R22 to R17, R23 to R18, R24 to R19, R25 to R20, R26 to R21, R27 to R22, R28 to R23, R29 to R24, R30 to R25, R31 to R26, R32 to R27, R33 to R28
Changed lines of the file:
@@
 $EndDescr
 $Comp
-L power:+3.3V #PWR039
+L power:+3.3V #PWR027
 U 1 1 5FB5387A
 P 4050 1300
-F 0 "#PWR039" H 4050 1150 50  0001 C CNN
+F 0 "#PWR027" H 4050 1150 50  0001 C CNN
 F 1 "+3.3V" H 4065 1473 50  0000 C CNN
 F 2 "" H 4050 1300 50  0001 C CNN
@@
 Servo_1_PWM
 $Comp
-L Device:R R26
+L Device:R R21
 U 1 1 5FB58774
 P 3750 1450
-F 0 "R26" V 3650 1450 50  0000 C CNN
+F 0 "R21" V 3650 1450 50  0000 C CNN
 F 1 "330" V 3750 1450 50  0000 C CNN
 F 2 "Resistor_SMD:R_0603_1608Metric_Pad1.05x0.95mm_HandSolder" V 3680 1450 50  0001 C CNN
@@
 $EndComp
 $Comp
-L Device:LED D22
+L Device:LED D15
 U 1 1 5FB5A15A
 P 3300 1450
-F 0 "D22" H 3300 1350 50  0000 C CNN
+F 0 "D15" H 3300 1350 50  0000 C CNN
 F 1 "LED" H 3300 1550 50  0000 C CNN
 F 2 "LED_SMD:LED_0603_1608Metric_Pad1.05x0.95mm_HandSolder" H 3300 1450 50  0001 C CNN
@@
 $EndComp
 $Comp
-L Device:R R18
+L Device:R R13
 U 1 1 5FB5CA90
 P 3100 1150
-F 0 "R18" V 3000 1150 50  0000 C CNN
+F 0 "R13" V 3000 1150 50  0000 C CNN
 F 1 "500" V 3100 1150 50  0000 C CNN
 F 2 "Resistor_SMD:R_0603_1608Metric_Pad1.05x0.95mm_HandSolder" V 3030 1150 50  0001 C CNN
@@
 $EndComp
 $Comp
-L power:GND #PWR038
+L power:GND #PWR026
 U 1 1 5FBA968B
 P 2450 6150
-F 0 "#PWR038" H 2450 5900 50  0001 C CNN
+F 0 "#PWR026" H 2450 5900 50  0001 C CNN
 F 1 "GND" H 2455 5977 50  0000 C CNN
 F 2 "" H 2450 6150 50  0001 C CNN
@@
 Servo_2_PWM
 $Comp
-L Device:R R27
+L Device:R R22
 U 1 1 5F8988CD
 P 3750 2100
-F 0 "R27" V 3650 2100 50  0000 C CNN
+F 0 "R22" V 3650 2100 50  0000 C CNN
 F 1 "330" V 3750 2100 50  0000 C CNN
 F 2 "Resistor_SMD:R_0603_1608Metric_Pad1.05x0.95mm_HandSolder" V 3680 2100 50  0001 C CNN
@@
 $EndComp
 $Comp
-L Device:LED D23
+L Device:LED D16
 U 1 1 5F8988D3
 P 3300 2100
-F 0 "D23" H 3300 2000 50  0000 C CNN
+F 0 "D16" H 3300 2000 50  0000 C CNN
 F 1 "LED" H 3300 2200 50  0000 C CNN
 F 2 "LED_SMD:LED_0603_1608Metric_Pad1.05x0.95mm_HandSolder" H 3300 2100 50  0001 C CNN
@@
 $EndComp
 $Comp
-L Device:R R19
+L Device:R R14
 U 1 1 5F8988DF
 P 3100 1800
-F 0 "R19" V 3000 1800 50  0000 C CNN
+F 0 "R14" V 3000 1800 50  0000 C CNN
 F 1 "500" V 3100 1800 50  0000 C CNN
 F 2 "Resistor_SMD:R_0603_1608Metric_Pad1.05x0.95mm_HandSolder" V 3030 1800 50  0001 C CNN
@@
 Servo_3_PWM
 $Comp
-L Device:R R28
+L Device:R R23
 U 1 1 5F8A6B43
 P 3750 2750
-F 0 "R28" V 3650 2750 50  0000 C CNN
+F 0 "R23" V 3650 2750 50  0000 C CNN
 F 1 "330" V 3750 2750 50  0000 C CNN
 F 2 "Resistor_SMD:R_0603_1608Metric_Pad1.05x0.95mm_HandSolder" V 3680 2750 50  0001 C CNN
@@
 $EndComp
 $Comp
-L Device:LED D24
+L Device:LED D17
 U 1 1 5F8A6B49
 P 3300 2750
-F 0 "D24" H 3300 2650 50  0000 C CNN
+F 0 "D17" H 3300 2650 50  0000 C CNN
 F 1 "LED" H 3300 2850 50  0000 C CNN
 F 2 "LED_SMD:LED_0603_1608Metric_Pad1.05x0.95mm_HandSolder" H 3300 2750 50  0001 C CNN
@@
 $EndComp
 $Comp
-L Device:R R20
+L Device:R R15
 U 1 1 5F8A6B55
 P 3100 2450
-F 0 "R20" V 3000 2450 50  0000 C CNN
+F 0 "R15" V 3000 2450 50  0000 C CNN
 F 1 "500" V 3100 2450 50  0000 C CNN
 F 2 "Resistor_SMD:R_0603_1608Metric_Pad1.05x0.95mm_HandSolder" V 3030 2450 50  0001 C CNN
@@
 Servo_4_PWM
 $Comp
-L Device:R R29
+L Device:R R24
 U 1 1 5F8A6B62
 P 3750 3400
-F 0 "R29" V 3650 3400 50  0000 C CNN
+F 0 "R24" V 3650 3400 50  0000 C CNN
 F 1 "330" V 3750 3400 50  0000 C CNN
 F 2 "Resistor_SMD:R_0603_1608Metric_Pad1.05x0.95mm_HandSolder" V 3680 3400 50  0001 C CNN
@@
 $EndComp
 $Comp
-L Device:LED D25
+L Device:LED D18
 U 1 1 5F8A6B68
 P 3300 3400
-F 0 "D25" H 3300 3300 50  0000 C CNN
+F 0 "D18" H 3300 3300 50  0000 C CNN
 F 1 "LED" H 3300 3500 50  0000 C CNN
 F 2 "LED_SMD:LED_0603_1608Metric_Pad1.05x0.95mm_HandSolder" H 3300 3400 50  0001 C CNN
@@
 $EndComp
 $Comp
-L Device:R R21
+L Device:R R16
 U 1 1 5F8A6B74
 P 3100 3100
-F 0 "R21" V 3000 3100 50  0000 C CNN
+F 0 "R16" V 3000 3100 50  0000 C CNN
 F 1 "500" V 3100 3100 50  0000 C CNN
 F 2 "Resistor_SMD:R_0603_1608Metric_Pad1.05x0.95mm_HandSolder" V 3030 3100 50  0001 C CNN
@@
 Servo_5_PWM
 $Comp
-L Device:R R30
+L Device:R R25
 U 1 1 5F8C6A5B
 P 3750 4050
-F 0 "R30" V 3650 4050 50  0000 C CNN
+F 0 "R25" V 3650 4050 50  0000 C CNN
 F 1 "330" V 3750 4050 50  0000 C CNN
 F 2 "Resistor_SMD:R_0603_1608Metric_Pad1.05x0.95mm_HandSolder" V 3680 4050 50  0001 C CNN
@@
 $EndComp
 $Comp
-L Device:LED D26
+L Device:LED D19
 U 1 1 5F8C6A61
 P 3300 4050
-F 0 "D26" H 3300 3950 50  0000 C CNN
+F 0 "D19" H 3300 3950 50  0000 C CNN
 F 1 "LED" H 3300 4150 50  0000 C CNN
 F 2 "LED_SMD:LED_0603_1608Metric_Pad1.05x0.95mm_HandSolder" H 3300 4050 50  0001 C CNN
@@
 $EndComp
 $Comp
-L Device:R R22
+L Device:R R17
 U 1 1 5F8C6A6D
 P 3100 3750
-F 0 "R22" V 3000 3750 50  0000 C CNN
+F 0 "R17" V 3000 3750 50  0000 C CNN
 F 1 "500" V 3100 3750 50  0000 C CNN
 F 2 "Resistor_SMD:R_0603_1608Metric_Pad1.05x0.95mm_HandSolder" V 3030 3750 50  0001 C CNN
@@
 Servo_6_PWM
 $Comp
-L Device:R R31
+L Device:R R26
 U 1 1 5F8C6A7A
 P 3750 4700
-F 0 "R31" V 3650 4700 50  0000 C CNN
+F 0 "R26" V 3650 4700 50  0000 C CNN
 F 1 "330" V 3750 4700 50  0000 C CNN
 F 2 "Resistor_SMD:R_0603_1608Metric_Pad1.05x0.95mm_HandSolder" V 3680 4700 50  0001 C CNN
@@
 $EndComp
 $Comp
-L Device:LED D27
+L Device:LED D20
 U 1 1 5F8C6A80
 P 3300 4700
-F 0 "D27" H 3300 4600 50  0000 C CNN
+F 0 "D20" H 3300 4600 50  0000 C CNN
 F 1 "LED" H 3300 4800 50  0000 C CNN
 F 2 "LED_SMD:LED_0603_1608Metric_Pad1.05x0.95mm_HandSolder" H 3300 4700 50  0001 C CNN
@@
 $EndComp
 $Comp
-L Device:R R23
+L Device:R R18
 U 1 1 5F8C6A8C
 P 3100 4400
-F 0 "R23" V 3000 4400 50  0000 C CNN
+F 0 "R18" V 3000 4400 50  0000 C CNN
 F 1 "500" V 3100 4400 50  0000 C CNN
 F 2 "Resistor_SMD:R_0603_1608Metric_Pad1.05x0.95mm_HandSolder" V 3030 4400 50  0001 C CNN
@@
 Servo_7_PWM
 $Comp
-L Device:R R32
+L Device:R R27
 U 1 1 5F8C6A99
 P 3750 5350
-F 0 "R32" V 3650 5350 50  0000 C CNN
+F 0 "R27" V 3650 5350 50  0000 C CNN
 F 1 "330" V 3750 5350 50  0000 C CNN
 F 2 "Resistor_SMD:R_0603_1608Metric_Pad1.05x0.95mm_HandSolder" V 3680 5350 50  0001 C CNN
@@
 $EndComp
 $Comp
-L Device:LED D28
+L Device:LED D21
 U 1 1 5F8C6A9F
 P 3300 5350
-F 0 "D28" H 3300 5250 50  0000 C CNN
+F 0 "D21" H 3300 5250 50  0000 C CNN
 F 1 "LED" H 3300 5450 50  0000 C CNN
 F 2 "LED_SMD:LED_0603_1608Metric_Pad1.05x0.95mm_HandSolder" H 3300 5350 50  0001 C CNN
@@
 $EndComp
 $Comp
-L Device:R R24
+L Device:R R19
 U 1 1 5F8C6AAB
 P 3100 5050
-F 0 "R24" V 3000 5050 50  0000 C CNN
+F 0 "R19" V 3000 5050 50  0000 C CNN
 F 1 "500" V 3100 5050 50  0000 C CNN
 F 2 "Resistor_SMD:R_0603_1608Metric_Pad1.05x0.95mm_HandSolder" V 3030 5050 50  0001 C CNN
@@
 Servo_8_AW
 $Comp
-L Device:R R33
+L Device:R R28
 U 1 1 5F8C6AB8
 P 3750 6000
-F 0 "R33" V 3650 6000 50  0000 C CNN
+F 0 "R28" V 3650 6000 50  0000 C CNN
 F 1 "330" V 3750 6000 50  0000 C CNN
 F 2 "Resistor_SMD:R_0603_1608Metric_Pad1.05x0.95mm_HandSolder" V 3680 6000 50  0001 C CNN
@@
 $EndComp
 $Comp
-L Device:LED D29
+L Device:LED D22
 U 1 1 5F8C6ABE
 P 3300 6000
-F 0 "D29" H 3300 5900 50  0000 C CNN
+F 0 "D22" H 3300 5900 50  0000 C CNN
 F 1 "LED" H 3300 6100 50  0000 C CNN
 F 2 "LED_SMD:LED_0603_1608Metric_Pad1.05x0.95mm_HandSolder" H 3300 6000 50  0001 C CNN
@@
 $EndComp
 $Comp
-L Device:R R25
+L Device:R R20
 U 1 1 5F8C6ACA
 P 3100 5700
-F 0 "R25" V 3000 5700 50  0000 C CNN
+F 0 "R20" V 3000 5700 50  0000 C CNN
 F 1 "500" V 3100 5700 50  0000 C CNN
 F 2 "Resistor_SMD:R_0603_1608Metric_Pad1.05x0.95mm_HandSolder" V 3030 5700 50  0001 C CNN

Commit message: layout 11
Parts:
- added D21, D22, D23, D24: LED, LED_SMD:LED_0603_1608Metric_Pad1.05x0.95mm_HandSolder, symbol Device:LED
- added R27, R28: 1000, Resistor_SMD:R_0603_1608Metric_Pad1.05x0.95mm_HandSolder, symbol Device:R
- added R29, R30: 330, Resistor_SMD:R_0603_1608Metric_Pad1.05x0.95mm_HandSolder, symbol Device:R
- renumbered D15 to D13, D16 to D14, D17 to D15, D18 to D16, D19 to D17, D20 to D18, D21 to D19, D22 to D20, R13 to R11, R14 to R12, R15 to R13, R16 to R14, R17 to R15, R18 to R16, R19 to R17, R20 to R18, R21 to R19, R22 to R20, R23 to R21, R24 to R22, R25 to R23, R26 to R24, R27 to R25, R28 to R26
Connections:
- net +3V3: now also R29.2
- net GND: now also D21.1 (K), D22.1 (K), D23.1 (K), D24.1 (K)
- new net: D21.2 (A), R27.1
- new net: D22.2 (A), R28.1
- new net: D23.2 (A), R29.1
- new net: D24.2 (A), R30.1
- new net +12L: R27.2
- new net +12VA: R28.2
- new net +5V: R30.2
