File: Hardware/gimble_board/GimbleBoard02.sch (KiCad schematic (older format))
At the start: 45 parts, among them SW1 SW_Push, SW2 SW_Push, SW3 SW_Push, SW4 SW_Push, SW5 SW_Push, SW6 SW_Push, SW7 SW_Push, SW8 SW_Push

Commit message: Replaced zener with schottky
Parts:
- gave numbers to parts that had none: 5
Changed lines of the file:
@@
 $EndComp
 $Comp
-L MRDT_Switches:2P2T SW?
+L MRDT_Switches:2P2T SW9
 U 1 1 5FC02AEA
 P 8650 2150
-F 0 "SW?" H 8775 2847 60  0000 C CNN
+F 0 "SW9" H 8775 2847 60  0000 C CNN
 F 1 "2P2T" H 8775 2741 60  0000 C CNN
 F 2 "" H 8250 2100 60  0001 C CNN
@@
 $EndComp
 $Comp
-L Device:R R?
+L Device:R R20
 U 1 1 5FC035C3
 P 9400 1700
-F 0 "R?" V 9500 1750 50  0000 R CNN
+F 0 "R20" V 9500 1750 50  0000 R CNN
 F 1 "330" V 9400 1800 50  0000 R CNN
 F 2 "" V 9330 1700 50  0001 C CNN
@@
 $EndComp
 $Comp
-L Device:R R?
+L Device:R R21
 U 1 1 5FC046BB
 P 9400 2100
-F 0 "R?" V 9500 2150 50  0000 R CNN
+F 0 "R21" V 9500 2150 50  0000 R CNN
 F 1 "330" V 9400 2200 50  0000 R CNN
 F 2 "" V 9330 2100 50  0001 C CNN
@@
 $EndComp
 $Comp
-L Device:LED D?
+L Device:LED D15
 U 1 1 5FC05378
 P 10000 1700
-F 0 "D?" H 10000 1600 50  0000 C CNN
+F 0 "D15" H 10000 1600 50  0000 C CNN
 F 1 "LED" H 10000 1800 50  0000 C CNN
 F 2 "" H 10000 1700 50  0001 C CNN
@@
 $EndComp
 $Comp
-L Device:LED D?
+L Device:LED D27
 U 1 1 5FC0654D
 P 10000 2100
-F 0 "D?" H 10000 2000 50  0000 C CNN
+F 0 "D27" H 10000 2000 50  0000 C CNN
 F 1 "LED" H 10000 2200 50  0000 C CNN
 F 2 "" H 10000 2100 50  0001 C CNN
@@
 $EndComp
 $Comp
-L power:GND #PWR?
+L power:GND #PWR044
 U 1 1 5FC0BD93
 P 10600 2550
-F 0 "#PWR?" H 10600 2300 50  0001 C CNN
+F 0 "#PWR044" H 10600 2300 50  0001 C CNN
 F 1 "GND" H 10605 2377 50  0000 C CNN
 F 2 "" H 10600 2550 50  0001 C CNN

Commit message: Fixed Switch and Buttons
Parts:
- removed C10, C11, C12, C5, C6, C7, C8, C9: 0.1uF, symbol Device:C
- removed R11, R14, R15, R18, R19: 1k, symbol Device:R
- removed R12, R13, R16: 330, symbol Device:R
- removed SW9: 2P2T, symbol MRDT_Switches:2P2T
- added SW9: SW_SPDT, symbol Switch:SW_SPDT
- R10, R6, R7: value 1k -> 330
Connections:
- net labels added: Servo_5_SW
- net labels removed: Servo_5_AW
- wire segments 106 -> 88
- no-connect marks 2 -> 0
Other:
- moved on the sheet: D14, D15, D27, R17, R20, R21, SW8

Commit message: footprints
Parts:
- D10: renamed from D7; footprint (none) -> LED_SMD:LED_0603_1608Metric_Pad1.05x0.95mm_HandSolder
- D11: renamed from D8; footprint (none) -> LED_SMD:LED_0603_1608Metric_Pad1.05x0.95mm_HandSolder
- D12: renamed from D9; footprint (none) -> LED_SMD:LED_0603_1608Metric_Pad1.05x0.95mm_HandSolder
- D13: renamed from D10; footprint (none) -> LED_SMD:LED_0603_1608Metric_Pad1.05x0.95mm_HandSolder
- D14: renamed from D11; footprint (none) -> LED_SMD:LED_0603_1608Metric_Pad1.05x0.95mm_HandSolder
- D15: renamed from D12; footprint (none) -> LED_SMD:LED_0603_1608Metric_Pad1.05x0.95mm_HandSolder
- D16: renamed from D13; footprint (none) -> LED_SMD:LED_0603_1608Metric_Pad1.05x0.95mm_HandSolder
- D17: renamed from D15; footprint (none) -> LED_SMD:LED_0603_1608Metric_Pad1.05x0.95mm_HandSolder
- D18: renamed from D27; footprint (none) -> LED_SMD:LED_0603_1608Metric_Pad1.05x0.95mm_HandSolder
- D9: renamed from D14; footprint (none) -> LED_SMD:LED_0603_1608Metric_Pad1.05x0.95mm_HandSolder
- R10: renamed from R8; footprint (none) -> Resistor_SMD:R_0603_1608Metric_Pad1.05x0.95mm_HandSolder
- R11: renamed from R9; footprint (none) -> Resistor_SMD:R_0603_1608Metric_Pad1.05x0.95mm_HandSolder
- R12: renamed from R10; footprint (none) -> Resistor_SMD:R_0603_1608Metric_Pad1.05x0.95mm_HandSolder
- R13: renamed from R20; footprint (none) -> Resistor_SMD:R_0603_1608Metric_Pad1.05x0.95mm_HandSolder
- R14: renamed from R21; footprint (none) -> Resistor_SMD:R_0603_1608Metric_Pad1.05x0.95mm_HandSolder
- R5: renamed from R17; footprint (none) -> Resistor_SMD:R_0603_1608Metric_Pad1.05x0.95mm_HandSolder
- R6: renamed from R4; footprint (none) -> Resistor_SMD:R_0603_1608Metric_Pad1.05x0.95mm_HandSolder
- R7: renamed from R5; footprint (none) -> Resistor_SMD:R_0603_1608Metric_Pad1.05x0.95mm_HandSolder
- R8: renamed from R6; footprint (none) -> Resistor_SMD:R_0603_1608Metric_Pad1.05x0.95mm_HandSolder
- R9: renamed from R7; footprint (none) -> Resistor_SMD:R_0603_1608Metric_Pad1.05x0.95mm_HandSolder
- SW1: renamed from SW8; footprint (none) -> Button_Switch_SMD:SW_SPST_TL3305A
- SW2: renamed from SW1; footprint (none) -> Button_Switch_SMD:SW_SPST_TL3305A
- SW3: renamed from SW2; footprint (none) -> Button_Switch_SMD:SW_SPST_TL3305A
- SW4: renamed from SW3; footprint (none) -> Button_Switch_SMD:SW_SPST_TL3305A
- SW5: renamed from SW4; footprint (none) -> Button_Switch_SMD:SW_SPST_TL3305A
- SW6: renamed from SW5; footprint (none) -> Button_Switch_SMD:SW_SPST_TL3305A
- SW7: renamed from SW6; footprint (none) -> Button_Switch_SMD:SW_SPST_TL3305A
- SW8: renamed from SW7; footprint (none) -> Button_Switch_SMD:SW_SPST_TL3305A
- SW9: footprint (none) -> Button_Switch_THT:SW_CuK_OS102011MA1QN1_SPDT_Angled

Commit message: layout 9
Parts:
- renumbered D14 to D10, D15 to D11, D16 to D12, D17 to D13, D18 to D14, D9 to D5, D10 to D6, D11 to D7, D12 to D8, D13 to D9, R12 to R10, R13 to R11, R14 to R12, R5 to R3, R6 to R4, R7 to R5, R8 to R6, R9 to R7, R10 to R8, R11 to R9
Changed lines of the file:
@@
 Sheet 02: Buttons
 $Comp
-L Device:LED D9
+L Device:LED D5
 U 1 1 5FB32644
 P 2550 1650
-F 0 "D9" H 2600 1550 50  0000 R CNN
+F 0 "D5" H 2600 1550 50  0000 R CNN
 F 1 "LED" H 2600 1750 50  0000 R CNN
 F 2 "LED_SMD:LED_0603_1608Metric_Pad1.05x0.95mm_HandSolder" H 2550 1650 50  0001 C CNN
@@
 $EndComp
 $Comp
-L Device:R R5
+L Device:R R3
 U 1 1 5FB3264A
 P 2100 1650
-F 0 "R5" V 2000 1700 50  0000 R CNN
+F 0 "R3" V 2000 1700 50  0000 R CNN
 F 1 "330" V 2100 1700 50  0000 R CNN
 F 2 "Resistor_SMD:R_0603_1608Metric_Pad1.05x0.95mm_HandSolder" V 2030 1650 50  0001 C CNN
@@
 Servo_1_SW
 $Comp
-L power:+3.3V #PWR021
+L power:+3.3V #PWR013
 U 1 1 5FB3F7E5
 P 1100 1500
-F 0 "#PWR021" H 1100 1350 50  0001 C CNN
+F 0 "#PWR013" H 1100 1350 50  0001 C CNN
 F 1 "+3.3V" H 1115 1673 50  0000 C CNN
 F 2 "" H 1100 1500 50  0001 C CNN
@@
 $EndComp
 $Comp
-L power:+3.3V #PWR023
+L power:+3.3V #PWR015
 U 1 1 5FBFCB75
 P 3450 1750
-F 0 "#PWR023" H 3450 1600 50  0001 C CNN
+F 0 "#PWR015" H 3450 1600 50  0001 C CNN
 F 1 "+3.3V" H 3465 1923 50  0000 C CNN
 F 2 "" H 3450 1750 50  0001 C CNN
@@
 $EndComp
 $Comp
-L Device:R R13
+L Device:R R11
 U 1 1 5FC035C3
 P 4300 1800
-F 0 "R13" V 4400 1850 50  0000 R CNN
+F 0 "R11" V 4400 1850 50  0000 R CNN
 F 1 "330" V 4300 1900 50  0000 R CNN
 F 2 "Resistor_SMD:R_0603_1608Metric_Pad1.05x0.95mm_HandSolder" V 4230 1800 50  0001 C CNN
@@
 $EndComp
 $Comp
-L Device:R R14
+L Device:R R12
 U 1 1 5FC046BB
 P 4300 2000
-F 0 "R14" V 4400 2050 50  0000 R CNN
+F 0 "R12" V 4400 2050 50  0000 R CNN
 F 1 "330" V 4300 2100 50  0000 R CNN
 F 2 "Resistor_SMD:R_0603_1608Metric_Pad1.05x0.95mm_HandSolder" V 4230 2000 50  0001 C CNN
@@
 $EndComp
 $Comp
-L Device:LED D17
+L Device:LED D13
 U 1 1 5FC05378
 P 4900 1500
-F 0 "D17" H 4900 1400 50  0000 C CNN
+F 0 "D13" H 4900 1400 50  0000 C CNN
 F 1 "LED" H 4900 1600 50  0000 C CNN
 F 2 "LED_SMD:LED_0603_1608Metric_Pad1.05x0.95mm_HandSolder" H 4900 1500 50  0001 C CNN
@@
 $EndComp
 $Comp
-L Device:LED D18
+L Device:LED D14
 U 1 1 5FC0654D
 P 4900 2300
-F 0 "D18" H 4900 2200 50  0000 C CNN
+F 0 "D14" H 4900 2200 50  0000 C CNN
 F 1 "LED" H 4900 2400 50  0000 C CNN
 F 2 "LED_SMD:LED_0603_1608Metric_Pad1.05x0.95mm_HandSolder" H 4900 2300 50  0001 C CNN
@@
 $EndComp
 $Comp
-L power:GND #PWR024
+L power:GND #PWR016
 U 1 1 5FC0BD93
 P 5550 2450
-F 0 "#PWR024" H 5550 2200 50  0001 C CNN
+F 0 "#PWR016" H 5550 2200 50  0001 C CNN
 F 1 "GND" H 5555 2277 50  0000 C CNN
 F 2 "" H 5550 2450 50  0001 C CNN
@@
 $EndComp
 $Comp
-L Device:LED D10
+L Device:LED D6
 U 1 1 5F8B1FFB
 P 2550 2100
-F 0 "D10" H 2600 2000 50  0000 R CNN
+F 0 "D6" H 2600 2000 50  0000 R CNN
 F 1 "LED" H 2600 2200 50  0000 R CNN
 F 2 "LED_SMD:LED_0603_1608Metric_Pad1.05x0.95mm_HandSolder" H 2550 2100 50  0001 C CNN
@@
 $EndComp
 $Comp
-L Device:R R6
+L Device:R R4
 U 1 1 5F8B2001
 P 2100 2100
-F 0 "R6" V 2000 2150 50  0000 R CNN
+F 0 "R4" V 2000 2150 50  0000 R CNN
 F 1 "330" V 2100 2150 50  0000 R CNN
 F 2 "Resistor_SMD:R_0603_1608Metric_Pad1.05x0.95mm_HandSolder" V 2030 2100 50  0001 C CNN
@@
 $EndComp
 $Comp
-L Device:LED D11
+L Device:LED D7
 U 1 1 5F8B47D6
 P 2550 2550
-F 0 "D11" H 2600 2450 50  0000 R CNN
+F 0 "D7" H 2600 2450 50  0000 R CNN
 F 1 "LED" H 2600 2650 50  0000 R CNN
 F 2 "LED_SMD:LED_0603_1608Metric_Pad1.05x0.95mm_HandSolder" H 2550 2550 50  0001 C CNN
@@
 $EndComp
 $Comp
-L Device:R R7
+L Device:R R5
 U 1 1 5F8B47DC
 P 2100 2550
-F 0 "R7" V 2000 2600 50  0000 R CNN
+F 0 "R5" V 2000 2600 50  0000 R CNN
 F 1 "330" V 2100 2600 50  0000 R CNN
 F 2 "Resistor_SMD:R_0603_1608Metric_Pad1.05x0.95mm_HandSolder" V 2030 2550 50  0001 C CNN
@@
 $EndComp
 $Comp
-L Device:LED D12
+L Device:LED D8
 U 1 1 5F8B6360
 P 2550 3000
-F 0 "D12" H 2600 2900 50  0000 R CNN
+F 0 "D8" H 2600 2900 50  0000 R CNN
 F 1 "LED" H 2600 3100 50  0000 R CNN
 F 2 "LED_SMD:LED_0603_1608Metric_Pad1.05x0.95mm_HandSolder" H 2550 3000 50  0001 C CNN
@@
 $EndComp
 $Comp
-L Device:R R8
+L Device:R R6
 U 1 1 5F8B6366
 P 2100 3000
-F 0 "R8" V 2000 3050 50  0000 R CNN
+F 0 "R6" V 2000 3050 50  0000 R CNN
 F 1 "330" V 2100 3050 50  0000 R CNN
 F 2 "Resistor_SMD:R_0603_1608Metric_Pad1.05x0.95mm_HandSolder" V 2030 3000 50  0001 C CNN
@@
 $EndComp
 $Comp
-L Device:LED D13
+L Device:LED D9
 U 1 1 5F8C3019
 P 2550 3450
-F 0 "D13" H 2600 3350 50  0000 R CNN
+F 0 "D9" H 2600 3350 50  0000 R CNN
 F 1 "LED" H 2600 3550 50  0000 R CNN
 F 2 "LED_SMD:LED_0603_1608Metric_Pad1.05x0.95mm_HandSolder" H 2550 3450 50  0001 C CNN
@@
 $EndComp
 $Comp
-L Device:R R9
+L Device:R R7
 U 1 1 5F8C301F
 P 2100 3450
-F 0 "R9" V 2000 3500 50  0000 R CNN
+F 0 "R7" V 2000 3500 50  0000 R CNN
 F 1 "330" V 2100 3500 50  0000 R CNN
 F 2 "Resistor_SMD:R_0603_1608Metric_Pad1.05x0.95mm_HandSolder" V 2030 3450 50  0001 C CNN
@@
 $EndComp
 $Comp
-L Device:LED D14
+L Device:LED D10
 U 1 1 5F8C3034
 P 2550 3900
-F 0 "D14" H 2600 3800 50  0000 R CNN
+F 0 "D10" H 2600 3800 50  0000 R CNN
 F 1 "LED" H 2600 4000 50  0000 R CNN
 F 2 "LED_SMD:LED_0603_1608Metric_Pad1.05x0.95mm_HandSolder" H 2550 3900 50  0001 C CNN
@@
 $EndComp
 $Comp
-L Device:R R10
+L Device:R R8
 U 1 1 5F8C303A
 P 2100 3900
-F 0 "R10" V 2000 3950 50  0000 R CNN
+F 0 "R8" V 2000 3950 50  0000 R CNN
 F 1 "330" V 2100 3950 50  0000 R CNN
 F 2 "Resistor_SMD:R_0603_1608Metric_Pad1.05x0.95mm_HandSolder" V 2030 3900 50  0001 C CNN
@@
 $EndComp
 $Comp
-L Device:LED D15
+L Device:LED D11
 U 1 1 5F8C304F
 P 2550 4350
-F 0 "D15" H 2600 4250 50  0000 R CNN
+F 0 "D11" H 2600 4250 50  0000 R CNN
 F 1 "LED" H 2600 4450 50  0000 R CNN
 F 2 "LED_SMD:LED_0603_1608Metric_Pad1.05x0.95mm_HandSolder" H 2550 4350 50  0001 C CNN
@@
 $EndComp
 $Comp
-L Device:R R11
+L Device:R R9
 U 1 1 5F8C3055
 P 2100 4350
-F 0 "R11" V 2000 4400 50  0000 R CNN
+F 0 "R9" V 2000 4400 50  0000 R CNN
 F 1 "330" V 2100 4400 50  0000 R CNN
 F 2 "Resistor_SMD:R_0603_1608Metric_Pad1.05x0.95mm_HandSolder" V 2030 4350 50  0001 C CNN
@@
 $EndComp
 $Comp
-L Device:LED D16
+L Device:LED D12
 U 1 1 5F8C306A
 P 2550 4800
-F 0 "D16" H 2600 4700 50  0000 R CNN
+F 0 "D12" H 2600 4700 50  0000 R CNN
 F 1 "LED" H 2600 4900 50  0000 R CNN
 F 2 "LED_SMD:LED_0603_1608Metric_Pad1.05x0.95mm_HandSolder" H 2550 4800 50  0001 C CNN
@@
 $EndComp
 $Comp
-L Device:R R12
+L Device:R R10
 U 1 1 5F8C3070
 P 2100 4800
-F 0 "R12" V 2000 4850 50  0000 R CNN
+F 0 "R10" V 2000 4850 50  0000 R CNN
 F 1 "330" V 2100 4850 50  0000 R CNN
 F 2 "Resistor_SMD:R_0603_1608Metric_Pad1.05x0.95mm_HandSolder" V 2030 4800 50  0001 C CNN
@@
 	1100 1650 1100 2100
 $Comp
-L power:GND #PWR022
+L power:GND #PWR014
 U 1 1 5F8D7076
 P 3000 4950
-F 0 "#PWR022" H 3000 4700 50  0001 C CNN
+F 0 "#PWR014" H 3000 4700 50  0001 C CNN
 F 1 "GND" H 3005 4777 50  0000 C CNN
 F 2 "" H 3000 4950 50  0001 C CNN

Commit message: layout 11
Parts:
- renumbered D12 to D10, D13 to D11, D14 to D12, D5 to D3, D6 to D4, D7 to D5, D8 to D6, D9 to D7, D10 to D8, D11 to D9, R3 to R1, R12 to R10, R4 to R2, R5 to R3, R6 to R4, R7 to R5, R8 to R6, R9 to R7, R10 to R8, R11 to R9
Changed lines of the file:
@@
 EESchema Schematic File Version 4
-LIBS:gimble_board-cache
 EELAYER 30 0
 EELAYER END
@@
 Sheet 02: Buttons
 $Comp
-L Device:LED D5
+L Device:LED D3
 U 1 1 5FB32644
 P 2550 1650
-F 0 "D5" H 2600 1550 50  0000 R CNN
+F 0 "D3" H 2600 1550 50  0000 R CNN
 F 1 "LED" H 2600 1750 50  0000 R CNN
 F 2 "LED_SMD:LED_0603_1608Metric_Pad1.05x0.95mm_HandSolder" H 2550 1650 50  0001 C CNN
@@
 $EndComp
 $Comp
-L Device:R R3
+L Device:R R1
 U 1 1 5FB3264A
 P 2100 1650
-F 0 "R3" V 2000 1700 50  0000 R CNN
+F 0 "R1" V 2000 1700 50  0000 R CNN
 F 1 "330" V 2100 1700 50  0000 R CNN
 F 2 "Resistor_SMD:R_0603_1608Metric_Pad1.05x0.95mm_HandSolder" V 2030 1650 50  0001 C CNN
@@
 Servo_1_SW
 $Comp
-L power:+3.3V #PWR013
+L power:+3.3V #PWR011
 U 1 1 5FB3F7E5
 P 1100 1500
-F 0 "#PWR013" H 1100 1350 50  0001 C CNN
+F 0 "#PWR011" H 1100 1350 50  0001 C CNN
 F 1 "+3.3V" H 1115 1673 50  0000 C CNN
 F 2 "" H 1100 1500 50  0001 C CNN
@@
 $EndComp
 $Comp
-L power:+3.3V #PWR015
+L power:+3.3V #PWR013
 U 1 1 5FBFCB75
 P 3450 1750
-F 0 "#PWR015" H 3450 1600 50  0001 C CNN
+F 0 "#PWR013" H 3450 1600 50  0001 C CNN
 F 1 "+3.3V" H 3465 1923 50  0000 C CNN
 F 2 "" H 3450 1750 50  0001 C CNN
@@
 $EndComp
 $Comp
-L Device:R R11
+L Device:R R9
 U 1 1 5FC035C3
 P 4300 1800
-F 0 "R11" V 4400 1850 50  0000 R CNN
+F 0 "R9" V 4400 1850 50  0000 R CNN
 F 1 "330" V 4300 1900 50  0000 R CNN
 F 2 "Resistor_SMD:R_0603_1608Metric_Pad1.05x0.95mm_HandSolder" V 4230 1800 50  0001 C CNN
@@
 $EndComp
 $Comp
-L Device:R R12
+L Device:R R10
 U 1 1 5FC046BB
 P 4300 2000
-F 0 "R12" V 4400 2050 50  0000 R CNN
+F 0 "R10" V 4400 2050 50  0000 R CNN
 F 1 "330" V 4300 2100 50  0000 R CNN
 F 2 "Resistor_SMD:R_0603_1608Metric_Pad1.05x0.95mm_HandSolder" V 4230 2000 50  0001 C CNN
@@
 $EndComp
 $Comp
-L Device:LED D13
+L Device:LED D11
 U 1 1 5FC05378
 P 4900 1500
-F 0 "D13" H 4900 1400 50  0000 C CNN
+F 0 "D11" H 4900 1400 50  0000 C CNN
 F 1 "LED" H 4900 1600 50  0000 C CNN
 F 2 "LED_SMD:LED_0603_1608Metric_Pad1.05x0.95mm_HandSolder" H 4900 1500 50  0001 C CNN
@@
 $EndComp
 $Comp
-L Device:LED D14
+L Device:LED D12
 U 1 1 5FC0654D
 P 4900 2300
-F 0 "D14" H 4900 2200 50  0000 C CNN
+F 0 "D12" H 4900 2200 50  0000 C CNN
 F 1 "LED" H 4900 2400 50  0000 C CNN
 F 2 "LED_SMD:LED_0603_1608Metric_Pad1.05x0.95mm_HandSolder" H 4900 2300 50  0001 C CNN
@@
 $EndComp
 $Comp
-L power:GND #PWR016
+L power:GND #PWR014
 U 1 1 5FC0BD93
 P 5550 2450
-F 0 "#PWR016" H 5550 2200 50  0001 C CNN
+F 0 "#PWR014" H 5550 2200 50  0001 C CNN
 F 1 "GND" H 5555 2277 50  0000 C CNN
 F 2 "" H 5550 2450 50  0001 C CNN
@@
 $EndComp
 $Comp
-L Device:LED D6
+L Device:LED D4
 U 1 1 5F8B1FFB
 P 2550 2100
-F 0 "D6" H 2600 2000 50  0000 R CNN
+F 0 "D4" H 2600 2000 50  0000 R CNN
 F 1 "LED" H 2600 2200 50  0000 R CNN
 F 2 "LED_SMD:LED_0603_1608Metric_Pad1.05x0.95mm_HandSolder" H 2550 2100 50  0001 C CNN
@@
 $EndComp
 $Comp
-L Device:R R4
+L Device:R R2
 U 1 1 5F8B2001
 P 2100 2100
-F 0 "R4" V 2000 2150 50  0000 R CNN
+F 0 "R2" V 2000 2150 50  0000 R CNN
 F 1 "330" V 2100 2150 50  0000 R CNN
 F 2 "Resistor_SMD:R_0603_1608Metric_Pad1.05x0.95mm_HandSolder" V 2030 2100 50  0001 C CNN
@@
 $EndComp
 $Comp
-L Device:LED D7
+L Device:LED D5
 U 1 1 5F8B47D6
 P 2550 2550
-F 0 "D7" H 2600 2450 50  0000 R CNN
+F 0 "D5" H 2600 2450 50  0000 R CNN
 F 1 "LED" H 2600 2650 50  0000 R CNN
 F 2 "LED_SMD:LED_0603_1608Metric_Pad1.05x0.95mm_HandSolder" H 2550 2550 50  0001 C CNN
@@
 $EndComp
 $Comp
-L Device:R R5
+L Device:R R3
 U 1 1 5F8B47DC
 P 2100 2550
-F 0 "R5" V 2000 2600 50  0000 R CNN
+F 0 "R3" V 2000 2600 50  0000 R CNN
 F 1 "330" V 2100 2600 50  0000 R CNN
 F 2 "Resistor_SMD:R_0603_1608Metric_Pad1.05x0.95mm_HandSolder" V 2030 2550 50  0001 C CNN
@@
 $EndComp
 $Comp
-L Device:LED D8
+L Device:LED D6
 U 1 1 5F8B6360
 P 2550 3000
-F 0 "D8" H 2600 2900 50  0000 R CNN
+F 0 "D6" H 2600 2900 50  0000 R CNN
 F 1 "LED" H 2600 3100 50  0000 R CNN
 F 2 "LED_SMD:LED_0603_1608Metric_Pad1.05x0.95mm_HandSolder" H 2550 3000 50  0001 C CNN
@@
 $EndComp
 $Comp
-L Device:R R6
+L Device:R R4
 U 1 1 5F8B6366
 P 2100 3000
-F 0 "R6" V 2000 3050 50  0000 R CNN
+F 0 "R4" V 2000 3050 50  0000 R CNN
 F 1 "330" V 2100 3050 50  0000 R CNN
 F 2 "Resistor_SMD:R_0603_1608Metric_Pad1.05x0.95mm_HandSolder" V 2030 3000 50  0001 C CNN
@@
 $EndComp
 $Comp
-L Device:LED D9
+L Device:LED D7
 U 1 1 5F8C3019
 P 2550 3450
-F 0 "D9" H 2600 3350 50  0000 R CNN
+F 0 "D7" H 2600 3350 50  0000 R CNN
 F 1 "LED" H 2600 3550 50  0000 R CNN
 F 2 "LED_SMD:LED_0603_1608Metric_Pad1.05x0.95mm_HandSolder" H 2550 3450 50  0001 C CNN
@@
 $EndComp
 $Comp
-L Device:R R7
+L Device:R R5
 U 1 1 5F8C301F
 P 2100 3450
-F 0 "R7" V 2000 3500 50  0000 R CNN
+F 0 "R5" V 2000 3500 50  0000 R CNN
 F 1 "330" V 2100 3500 50  0000 R CNN
 F 2 "Resistor_SMD:R_0603_1608Metric_Pad1.05x0.95mm_HandSolder" V 2030 3450 50  0001 C CNN
@@
 $EndComp
 $Comp
-L Device:LED D10
+L Device:LED D8
 U 1 1 5F8C3034
 P 2550 3900
-F 0 "D10" H 2600 3800 50  0000 R CNN
+F 0 "D8" H 2600 3800 50  0000 R CNN
 F 1 "LED" H 2600 4000 50  0000 R CNN
 F 2 "LED_SMD:LED_0603_1608Metric_Pad1.05x0.95mm_HandSolder" H 2550 3900 50  0001 C CNN
@@
 $EndComp
 $Comp
-L Device:R R8
+L Device:R R6
 U 1 1 5F8C303A
 P 2100 3900
-F 0 "R8" V 2000 3950 50  0000 R CNN
+F 0 "R6" V 2000 3950 50  0000 R CNN
 F 1 "330" V 2100 3950 50  0000 R CNN
 F 2 "Resistor_SMD:R_0603_1608Metric_Pad1.05x0.95mm_HandSolder" V 2030 3900 50  0001 C CNN
@@
 $EndComp
 $Comp
-L Device:LED D11
+L Device:LED D9
 U 1 1 5F8C304F
 P 2550 4350
-F 0 "D11" H 2600 4250 50  0000 R CNN
+F 0 "D9" H 2600 4250 50  0000 R CNN
 F 1 "LED" H 2600 4450 50  0000 R CNN
 F 2 "LED_SMD:LED_0603_1608Metric_Pad1.05x0.95mm_HandSolder" H 2550 4350 50  0001 C CNN
@@
 $EndComp
 $Comp
-L Device:R R9
+L Device:R R7
 U 1 1 5F8C3055
 P 2100 4350
-F 0 "R9" V 2000 4400 50  0000 R CNN
+F 0 "R7" V 2000 4400 50  0000 R CNN
 F 1 "330" V 2100 4400 50  0000 R CNN
 F 2 "Resistor_SMD:R_0603_1608Metric_Pad1.05x0.95mm_HandSolder" V 2030 4350 50  0001 C CNN
@@
 $EndComp
 $Comp
-L Device:LED D12
+L Device:LED D10
 U 1 1 5F8C306A
 P 2550 4800
-F 0 "D12" H 2600 4700 50  0000 R CNN
+F 0 "D10" H 2600 4700 50  0000 R CNN
 F 1 "LED" H 2600 4900 50  0000 R CNN
 F 2 "LED_SMD:LED_0603_1608Metric_Pad1.05x0.95mm_HandSolder" H 2550 4800 50  0001 C CNN
@@
 $EndComp
 $Comp
-L Device:R R10
+L Device:R R8
 U 1 1 5F8C3070
 P 2100 4800
-F 0 "R10" V 2000 4850 50  0000 R CNN
+F 0 "R8" V 2000 4850 50  0000 R CNN
 F 1 "330" V 2100 4850 50  0000 R CNN
 F 2 "Resistor_SMD:R_0603_1608Metric_Pad1.05x0.95mm_HandSolder" V 2030 4800 50  0001 C CNN
@@
 	1100 1650 1100 2100
 $Comp
-L power:GND #PWR014
+L power:GND #PWR012
 U 1 1 5F8D7076
 P 3000 4950
-F 0 "#PWR014" H 3000 4700 50  0001 C CNN
+F 0 "#PWR012" H 3000 4700 50  0001 C CNN
 F 1 "GND" H 3005 4777 50  0000 C CNN
 F 2 "" H 3000 4950 50  0001 C CNN
