File: Hardware/gimble_board/GimbleBoard03.sch (KiCad schematic (older format))
At the start: 9 parts

Commit message: footprints
Parts:
- added unit 3 of Conn1
- Conn1: footprint (none) -> MRDT_Connectors:Anderson_3_Horizontal_Side_by_Side
- Conn2, Conn3, Conn4, Conn5, Conn6, Conn7, Conn8, Conn9: footprint (none) -> MRDT_Connectors:MOLEX_SL_03_Horizontal
Connections:
- net Power_Input renamed Power_Input_Log
- new net Power_Input_Act: Conn1.3 (V+Act)
Other:
- moved on the sheet: Conn1A
Changed lines of the file:
@@
 EESchema Schematic File Version 4
+LIBS:gimble_board-cache
 EELAYER 30 0
 EELAYER END
@@
 F 0 "Conn1" H 1558 1887 60  0000 C CNN
 F 1 "AndersonPP" H 1558 1781 60  0000 C CNN
-F 2 "" H 1200 950 60  0001 C CNN
+F 2 "MRDT_Connectors:Anderson_3_Horizontal_Side_by_Side" H 1200 950 60  0001 C CNN
 F 3 "" H 1200 950 60  0001 C CNN
 	2    1350 1500
@@
 L MRDT_Connectors:AndersonPP Conn1
 U 1 1 5F7E5011
-P 1350 2050
-F 0 "Conn1" H 1558 2437 60  0000 C CNN
-F 1 "AndersonPP" H 1558 2331 60  0000 C CNN
-F 2 "" H 1200 1500 60  0001 C CNN
-F 3 "" H 1200 1500 60  0001 C CNN
-	1    1350 2050
-	1    0    0    -1
-$EndComp
-$Comp
-L power:GND #PWR09
+P 1350 2650
+F 0 "Conn1" H 1558 3037 60  0000 C CNN
+F 1 "AndersonPP" H 1558 2931 60  0000 C CNN
+F 2 "MRDT_Connectors:Anderson_3_Horizontal_Side_by_Side" H 1200 2100 60  0001 C CNN
+F 3 "" H 1200 2100 60  0001 C CNN
+	1    1350 2650
+	1    0    0    -1
+$EndComp
+$Comp
+L power:GND #PWR025
 U 1 1 5F7E9270
-P 1900 2100
-F 0 "#PWR09" H 1900 1850 50  0001 C CNN
-F 1 "GND" H 1905 1927 50  0000 C CNN
-F 2 "" H 1900 2100 50  0001 C CNN
-F 3 "" H 1900 2100 50  0001 C CNN
-	1    1900 2100
-	1    0    0    -1
-$EndComp
-Text GLabel 1900 1400 2    39   Output ~ 0
-Power_Input
+P 1900 2700
+F 0 "#PWR025" H 1900 2450 50  0001 C CNN
+F 1 "GND" H 1905 2527 50  0000 C CNN
+F 2 "" H 1900 2700 50  0001 C CNN
+F 3 "" H 1900 2700 50  0001 C CNN
+	1    1900 2700
+	1    0    0    -1
+$EndComp
 $Comp
 L MRDT_Connectors:Molex_SL_03 Conn2
@@
 F 0 "Conn2" H 3292 1213 60  0000 C CNN
 F 1 "Molex_SL_03" H 3292 1319 60  0000 C CNN
-F 2 "" H 3350 1400 60  0001 C CNN
+F 2 "MRDT_Connectors:MOLEX_SL_03_Horizontal" H 3350 1400 60  0001 C CNN
 F 3 "" H 3350 1400 60  0001 C CNN
 	1    3350 1400
@@
 F 0 "Conn3" H 3292 1813 60  0000 C CNN
 F 1 "Molex_SL_03" H 3292 1919 60  0000 C CNN
-F 2 "" H 3350 2000 60  0001 C CNN
+F 2 "MRDT_Connectors:MOLEX_SL_03_Horizontal" H 3350 2000 60  0001 C CNN
 F 3 "" H 3350 2000 60  0001 C CNN
 	1    3350 2000
@@
 F 0 "Conn4" H 3292 2413 60  0000 C CNN
 F 1 "Molex_SL_03" H 3292 2519 60  0000 C CNN
-F 2 "" H 3350 2600 60  0001 C CNN
+F 2 "MRDT_Connectors:MOLEX_SL_03_Horizontal" H 3350 2600 60  0001 C CNN
 F 3 "" H 3350 2600 60  0001 C CNN
 	1    3350 2600
@@
 F 0 "Conn5" H 3292 3013 60  0000 C CNN
 F 1 "Molex_SL_03" H 3292 3119 60  0000 C CNN
-F 2 "" H 3350 3200 60  0001 C CNN
+F 2 "MRDT_Connectors:MOLEX_SL_03_Horizontal" H 3350 3200 60  0001 C CNN
 F 3 "" H 3350 3200 60  0001 C CNN
 	1    3350 3200
@@
 F 0 "Conn6" H 3292 3613 60  0000 C CNN
 F 1 "Molex_SL_03" H 3292 3719 60  0000 C CNN
-F 2 "" H 3350 3800 60  0001 C CNN
+F 2 "MRDT_Connectors:MOLEX_SL_03_Horizontal" H 3350 3800 60  0001 C CNN
 F 3 "" H 3350 3800 60  0001 C CNN
 	1    3350 3800
@@
 F 0 "Conn7" H 3292 4213 60  0000 C CNN
 F 1 "Molex_SL_03" H 3292 4319 60  0000 C CNN
-F 2 "" H 3350 4400 60  0001 C CNN
+F 2 "MRDT_Connectors:MOLEX_SL_03_Horizontal" H 3350 4400 60  0001 C CNN
 F 3 "" H 3350 4400 60  0001 C CNN
 	1    3350 4400
@@
 F 0 "Conn8" H 3292 4813 60  0000 C CNN
 F 1 "Molex_SL_03" H 3292 4919 60  0000 C CNN
-F 2 "" H 3350 5000 60  0001 C CNN
+F 2 "MRDT_Connectors:MOLEX_SL_03_Horizontal" H 3350 5000 60  0001 C CNN
 F 3 "" H 3350 5000 60  0001 C CNN
 	1    3350 5000
@@
 F 0 "Conn9" H 3292 5413 60  0000 C CNN
 F 1 "Molex_SL_03" H 3292 5519 60  0000 C CNN
-F 2 "" H 3350 5600 60  0001 C CNN
+F 2 "MRDT_Connectors:MOLEX_SL_03_Horizontal" H 3350 5600 60  0001 C CNN
 F 3 "" H 3350 5600 60  0001 C CNN
 	1    3350 5600
@@
 $EndComp
 $Comp
-L power:+5V #PWR047
+L power:+5V #PWR026
 U 1 1 5F854A29
 P 3800 1150
-F 0 "#PWR047" H 3800 1000 50  0001 C CNN
+F 0 "#PWR026" H 3800 1000 50  0001 C CNN
 F 1 "+5V" H 3815 1323 50  0000 C CNN
 F 2 "" H 3800 1150 50  0001 C CNN
@@
 $EndComp
 $Comp
-L power:GND #PWR048
+L power:GND #PWR027
 U 1 1 5F856854
 P 3900 6150
-F 0 "#PWR048" H 3900 5900 50  0001 C CNN
+F 0 "#PWR027" H 3900 5900 50  0001 C CNN
 F 1 "GND" H 3905 5977 50  0000 C CNN
 F 2 "" H 3900 6150 50  0001 C CNN
@@
 	1750 1400 1900 1400
 Wire Wire Line
-	1750 1950 1900 1950
-Wire Wire Line
-	1900 1950 1900 2100
+	1750 2550 1900 2550
+Wire Wire Line
+	1900 2550 1900 2700
 Text Notes 1300 900  0    79   ~ 0
 Anderson
 Text Notes 3550 800  0    79   ~ 0
 Molex
+Text GLabel 1900 1400 2    39   Output ~ 0
+Power_Input_Log
+Text GLabel 1950 1900 2    39   Output ~ 0
+Power_Input_Act
+$Comp
+L MRDT_Connectors:AndersonPP Conn1
+U 3 1 5FB2D4BE
+P 1350 2000
+F 0 "Conn1" H 1558 2387 60  0000 C CNN
+F 1 "AndersonPP" H 1558 2281 60  0000 C CNN
+F 2 "MRDT_Connectors:Anderson_3_Horizontal_Side_by_Side" H 1200 1450 60  0001 C CNN
+F 3 "" H 1200 1450 60  0001 C CNN
+	3    1350 2000
+	1    0    0    -1
+$EndComp
+Wire Wire Line
+	1750 1900 1950 1900
 $EndSCHEMATC

Commit message: layout 2
Connections:
- net Servo_5_AW renamed Servo_5_PWM
- net Servo_8_PWM renamed Servo_8_AW
Changed lines of the file:
@@
 Servo_4_PWM
 Text GLabel 4050 3850 2    39   Input ~ 0
-Servo_5_AW
+Servo_5_PWM
 Text GLabel 4050 4450 2    39   Input ~ 0
 Servo_6_PWM
@@
 Servo_7_PWM
 Text GLabel 4050 5650 2    39   Input ~ 0
-Servo_8_PWM
+Servo_8_AW
 Wire Wire Line
 	3550 5650 4050 5650

Commit message: layout 11
Other:
- moved on the sheet: Conn1A
Changed lines of the file:
@@
 EESchema Schematic File Version 4
-LIBS:gimble_board-cache
 EELAYER 30 0
 EELAYER END
@@
 L MRDT_Connectors:AndersonPP Conn1
 U 1 1 5F7E5011
-P 1350 2650
-F 0 "Conn1" H 1558 3037 60  0000 C CNN
-F 1 "AndersonPP" H 1558 2931 60  0000 C CNN
-F 2 "MRDT_Connectors:Anderson_3_Horizontal_Side_by_Side" H 1200 2100 60  0001 C CNN
-F 3 "" H 1200 2100 60  0001 C CNN
-	1    1350 2650
-	1    0    0    -1
-$EndComp
-$Comp
-L power:GND #PWR017
+P 1350 2500
+F 0 "Conn1" H 1558 2887 60  0000 C CNN
+F 1 "AndersonPP" H 1558 2781 60  0000 C CNN
+F 2 "MRDT_Connectors:Anderson_3_Horizontal_Side_by_Side" H 1200 1950 60  0001 C CNN
+F 3 "" H 1200 1950 60  0001 C CNN
+	1    1350 2500
+	1    0    0    -1
+$EndComp
+$Comp
+L power:GND #PWR015
 U 1 1 5F7E9270
-P 1900 2700
-F 0 "#PWR017" H 1900 2450 50  0001 C CNN
-F 1 "GND" H 1905 2527 50  0000 C CNN
-F 2 "" H 1900 2700 50  0001 C CNN
-F 3 "" H 1900 2700 50  0001 C CNN
-	1    1900 2700
+P 1900 2550
+F 0 "#PWR015" H 1900 2300 50  0001 C CNN
+F 1 "GND" H 1905 2377 50  0000 C CNN
+F 2 "" H 1900 2550 50  0001 C CNN
+F 3 "" H 1900 2550 50  0001 C CNN
+	1    1900 2550
 	1    0    0    -1
 $EndComp
@@
 $EndComp
 $Comp
-L power:+5V #PWR018
+L power:+5V #PWR016
 U 1 1 5F854A29
 P 3800 1150
-F 0 "#PWR018" H 3800 1000 50  0001 C CNN
+F 0 "#PWR016" H 3800 1000 50  0001 C CNN
 F 1 "+5V" H 3815 1323 50  0000 C CNN
 F 2 "" H 3800 1150 50  0001 C CNN
@@
 $EndComp
 $Comp
-L power:GND #PWR019
+L power:GND #PWR017
 U 1 1 5F856854
 P 3900 6150
-F 0 "#PWR019" H 3900 5900 50  0001 C CNN
+F 0 "#PWR017" H 3900 5900 50  0001 C CNN
 F 1 "GND" H 3905 5977 50  0000 C CNN
 F 2 "" H 3900 6150 50  0001 C CNN
@@
 	1750 1400 1900 1400
 Wire Wire Line
-	1750 2550 1900 2550
-Wire Wire Line
-	1900 2550 1900 2700
+	1750 2400 1900 2400
+Wire Wire Line
+	1900 2400 1900 2550
 Text Notes 1300 900  0    79   ~ 0
 Anderson
 Text Notes 3550 800  0    79   ~ 0
 Molex
-Text GLabel 1900 1400 2    39   Output ~ 0
-Power_Input_Log
-Text GLabel 1950 1900 2    39   Output ~ 0
-Power_Input_Act
 $Comp
 L MRDT_Connectors:AndersonPP Conn1
@@
 $EndComp
 Wire Wire Line
-	1750 1900 1950 1900
+	1900 1900 1750 1900
+Text GLabel 1900 1400 2    50   Input ~ 0
+Power_Input_Log
+Text GLabel 1900 1900 2    50   Input ~ 0
+Power_Input_Act
 $EndSCHEMATC
