File: Hardware/gimble_board/gimble_board.kicad_pcb (KiCad board)
At the start: 2 copper layers, 101 parts, among them J1 Test_Point, J2 Test_Point, J3 Test_Point, J4 Test_Point, Q1 Q_NMOS_GDS, Q2 Q_NMOS_GDS, Q3 Q_NMOS_GDS, Q4 Q_NMOS_GDS, Q5 Q_NMOS_GDS, Q6 Q_NMOS_GDS, Q7 Q_NMOS_GDS, Q8 Q_NMOS_GDS, SW1 SW_Push, SW2 SW_Push, SW3 SW_Push, SW4 SW_Push, SW5 SW_Push, SW6 SW_Push, SW7 SW_Push, SW8 SW_Push, SW9 SW_SPDT, U1 LM2576SX-3.3, U2 LM2576SX-5.0, U3 TM4C129E_Launchpad

Commit message: layout 2
Parts:
- moved R31 224.5 mm to (42.4, 151.5)
- moved R29 219.3 mm to (36.4, 105.5)
- moved R30 219.3 mm to (33.5, 131.6)
- moved R20 219.0 mm to (33.1, 80.5)
- moved R27 215.8 mm to (34.4, 66.4)
- moved Q6 215.2 mm to (36.7, 149.7)
- moved D22 215.1 mm to (36.7, 29.7)
- moved D27 214.9 mm to (42.0, 147.8)
- moved R28 214.7 mm to (33.0, 84.3)
- moved R26 213.7 mm to (37.0, 33.3)
- moved R22 212.3 mm to (38.7, 125.3)
- moved R18 208.6 mm to (37.1, 36.3)
- moved R23 207.1 mm to (35.6, 145.5)
- moved R19 207.1 mm to (33.9, 58.8)
- moved R21 206.7 mm to (36.2, 109.5)
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Connections:
- Conn6 pad 3: Servo_5_AW -> Servo_5_PWM
- Conn9 pad 3: Servo_8_PWM -> Servo_8_AW
- R22 pad 1: Servo_5_AW -> Servo_5_PWM
- R25 pad 1: Servo_8_PWM -> Servo_8_AW
- U3 pad PA4: Net-(U3-PadPA4) -> Servo_Digital_Control
- U3 pad PA5: Net-(U3-PadPA5) -> Servo_Manual_Control
- U3 pad PA6: Net-(U3-PadPA6) -> Servo_6_SW
- U3 pad PB2: Servo_8_SW -> Net-(U3-PadPB2)
- U3 pad PC4: Servo_2_SW -> Net-(U3-PadPC4)
- U3 pad PC5: Servo_3_SW -> Net-(U3-PadPC5)
- U3 pad PC6: Servo_4_SW -> Net-(U3-PadPC6)
- U3 pad PC7: Servo_7_SW -> Net-(U3-PadPC7)
- U3 pad PD2: Servo_Manual_Control -> Net-(U3-PadPD2)
- U3 pad PD3: Servo_6_SW -> Net-(U3-PadPD3)
- U3 pad PD7: Net-(U3-PadPD7) -> Servo_5_SW
- U3 pad PE0: Net-(U3-PadPE0) -> Servo_1_SW
- U3 pad PE1: Net-(U3-PadPE1) -> Servo_2_SW
- U3 pad PE2: Net-(U3-PadPE2) -> Servo_3_SW
- U3 pad PE3: Net-(U3-PadPE3) -> Servo_4_SW
- U3 pad PE4: Servo_1_SW -> Net-(U3-PadPE4)
- U3 pad PE5: Servo_5_SW -> Net-(U3-PadPE5)
- U3 pad PG1: Servo_6_PWM -> Servo_5_PWM
- U3 pad PK4: Servo_7_PWM -> Servo_6_PWM
- U3 pad PK5: Servo_8_PWM -> Servo_7_PWM
- U3 pad PL4: Servo_5_AW -> Net-(U3-PadPL4)
- U3 pad PM0: Net-(U3-PadPM0) -> Servo_8_AW
- U3 pad PM4: Net-(U3-PadPM4) -> Servo_7_SW
- U3 pad PM5: Net-(U3-PadPM5) -> Servo_8_SW
- U3 pad PP0: Servo_Digital_Control -> Net-(U3-PadPP0)
Routing:
- added copper zone on F.Cu, net GND

Commit message: layout 3
Parts:
- U3: footprint MRDT_Shields:TM4C129E_Launchpad_FULL_THT_TOP -> MRDT_Shields:TM4C129E_Launchpad_FULL_THT_BOTTOM

Commit message: layout 4
Parts:
- removed D19, D20, D21: LED, LED_SMD:LED_0603_1608Metric_Pad1.05x0.95mm_HandSolder
- removed R15: 1k, Resistor_SMD:R_0603_1608Metric_Pad1.05x0.95mm_HandSolder
- removed R16: 500, Resistor_SMD:R_0603_1608Metric_Pad1.05x0.95mm_HandSolder
- removed R17: 330, Resistor_SMD:R_0603_1608Metric_Pad1.05x0.95mm_HandSolder
- moved D16 166.2 mm to (110.0, 75.1), turned to 270 degrees
- moved D18 166.0 mm to (80.5, 60.8), turned to 90 degrees
- moved R12 165.6 mm to (110.0, 78.7), turned to 270 degrees
- moved R14 164.5 mm to (78.6, 60.8), turned to 90 degrees
- moved D17 158.4 mm to (80.5, 66.7), turned to 270 degrees
- moved R13 157.5 mm to (78.6, 66.7), turned to 270 degrees
- moved SW8 156.7 mm to (108.5, 85.5), turned to 90 degrees
- moved SW9 156.5 mm to (70.7, 65.8), turned to 90 degrees
- moved R31 147.9 mm to (144.4, 44.3), turned to 270 degrees
- moved D15 147.2 mm to (104.1, 75.1), turned to 270 degrees
- moved R11 146.5 mm to (104.1, 78.7), turned to 270 degrees
- moved R23 145.3 mm to (141.0, 45.5), turned to 270 degrees
- moved Q6 144.6 mm to (138.1, 46.6), turned to 90 degrees
- moved D27 141.0 mm to (142.0, 48.5)
- moved J4 138.1 mm to (130.0, 89.7)
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
Commit message: layout 6
Parts:
- moved R4 18.5 mm to (135.2, 80.4), turned to 0 degrees
- moved D8 17.3 mm to (135.2, 78.6), turned to 180 degrees
- moved D7 15.2 mm to (157.1, 78.5), turned to 180 degrees
- moved C3 14.1 mm to (157.2, 88.3), turned to 180 degrees
- moved D18 12.4 mm to (70.0, 67.4), turned to 180 degrees
- moved R3 12.3 mm to (157.1, 80.3)
- moved D17 11.8 mm to (70.0, 61.5), turned to 180 degrees
- moved D1 10.3 mm to (157.1, 74.7), turned to 0 degrees
- moved R14 9.75 mm to (70.0, 65.4), turned to 180 degrees
- moved C2 9.25 mm to (162.2, 56.4)
- moved R13 9.23 mm to (70.0, 63.4), turned to 180 degrees
- moved SW9 8.84 mm to (78.8, 62.2), turned to 270 degrees
- moved D2 8.74 mm to (135.2, 74.7), turned to 0 degrees
- moved R2 8.11 mm to (162.2, 52.1)
- moved J3 7.66 mm to (157.2, 85.2)
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Connections:
- U3 pad PA4: Servo_Digital_Control -> Net-(U3-PadPA4)
- U3 pad PA5: Servo_Manual_Control -> Net-(U3-PadPA5)
- U3 pad PC4: Net-(U3-PadPC4) -> Servo_Manual_Control
- U3 pad PE4: Net-(U3-PadPE4) -> Servo_Digital_Control
Routing:
- net +3V3: track 0.00 -> 449.7 mm, vias 0 -> 13
- net +5V: track 0.00 -> 86.1 mm
- net Power_Input_Act: track 0.00 -> 67.0 mm, vias 0 -> 2
- net Net-(D5-Pad1): track 0.00 -> 55.0 mm, vias 0 -> 1
- net Servo_4_PWM: track 0.00 -> 50.9 mm, vias 0 -> 1
- net Power_Input_Log: track 0.00 -> 43.5 mm, vias 0 -> 2
- net Servo_3_PWM: track 0.00 -> 41.0 mm, vias 0 -> 1
- net Servo_8_AW: track 0.00 -> 39.4 mm, vias 0 -> 1
- net Servo_8_SW: track 0.00 -> 38.6 mm
- net Servo_Digital_Control: track 0.00 -> 38.0 mm
- net GND: track 0.00 -> 37.1 mm, vias 0 -> 11
- net Servo_7_SW: track 0.00 -> 34.0 mm
- net Servo_Manual_Control: track 0.00 -> 33.0 mm
- net Servo_2_PWM: track 0.00 -> 32.7 mm, vias 0 -> 1
- net Servo_6_SW: track 0.00 -> 30.8 mm
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- added copper zone on B.Cu, net +5V
Other:
- board outline added: 124.5 x 95.9 mm
- board text added: "3.3V"
- board text added: "5V"
- board text added: "Actuation"
- board text added: "Buck Converters"
- board text added: "Digital/Manual Control"
- board text added: "Logic"
- board text added: "Manual Servo Control"
- board text added: "Schott-kys"
- board text added: "Servo Connectors"
- board text added: "Servo Indicators"

Commit message: layout 7
Parts:
- added G***: LOGO, MRDT_Silkscreens:0_MRDT_Logo_20mm, F.Cu at (90.4, 110.7)
- added G***: LOGO, MRDT_Silkscreens:2_Dahlbot_2.0, F.Cu at (179.8, 35.9)

Commit message: layout 9
Parts:
- removed C1, C2: 100uF, Capacitor_SMD:C_0603_1608Metric_Pad1.05x0.95mm_HandSolder
- removed C3, C4: 1000uF, Capacitor_SMD:C_0603_1608Metric_Pad1.05x0.95mm_HandSolder
- removed Conn1: AndersonPP, MRDT_Connectors:Anderson_3_Horizontal_Side_by_Side
- removed Conn2, Conn3, Conn4, Conn5, Conn6, Conn7, Conn8, Conn9: Molex_SL_03, MRDT_Connectors:MOLEX_SL_03_Horizontal
- removed D23, D24, D25, D26, D27, D28, D29: LED, LED_SMD:LED_0603_1608Metric_Pad1.05x0.95mm_HandSolder
- removed G***: LOGO, MRDT_Silkscreens:0_MRDT_Logo_20mm
- removed G***: LOGO, MRDT_Silkscreens:2_Dahlbot_2.0
- removed J3, J4: Test_Point, TestPoint:TestPoint_Pad_2.0x2.0mm
- removed L1, L2: 100uH, Inductor_SMD:L_0603_1608Metric_Pad1.05x0.95mm_HandSolder
- removed R1, R2: 1k, Resistor_SMD:R_0603_1608Metric_Pad1.05x0.95mm_HandSolder
- removed R10, R11, R12, R13, R14, R26, R27, R28, R29, R3, R30, R31, R32, R33, R5, R6, R7, R8, R9: 330, Resistor_SMD:R_0603_1608Metric_Pad1.05x0.95mm_HandSolder
- removed R18, R19, R20, R21, R22, R23, R24, R25, R4: 500, Resistor_SMD:R_0603_1608Metric_Pad1.05x0.95mm_HandSolder
- removed U1: LM2576SX-3.3, Package_TO_SOT_SMD:TO-263-6
- removed U2: LM2576SX-5.0, Package_TO_SOT_SMD:TO-263-6
- removed U3: TM4C129E_Launchpad, MRDT_Shields:TM4C129E_Launchpad_FULL_THT_BOTTOM
- added D19: LED, LED_SMD:LED_0603_1608Metric_Pad1.05x0.95mm_HandSolder, F.Cu at (151.1, 52.8)
- added D20: LED, LED_SMD:LED_0603_1608Metric_Pad1.05x0.95mm_HandSolder, F.Cu at (153.2, 48.9)
- added D21: LED, LED_SMD:LED_0603_1608Metric_Pad1.05x0.95mm_HandSolder, F.Cu at (146.7, 55.4)
- D5, D6: value D_Schottky -> LED; footprint Diode_THT:D_DO-201AD_P15.24mm_Horizontal -> LED_SMD:LED_0603_1608Metric_Pad1.05x0.95mm_HandSolder
- moved D17 86.1 mm to (155.5, 51.5), turned to 0 degrees
- moved D18 82.0 mm to (151.1, 55.4), turned to 0 degrees
- moved D22 77.1 mm to (153.2, 46.3)
- moved Q1 75.5 mm to (147.7, 49.3), turned to 0 degrees
- moved D3 75.4 mm to (86.8, 74.1)
- moved D4 73.1 mm to (91.2, 71.5)
- moved J2 72.7 mm to (91.0, 74.8)
- moved D1 70.3 mm to (86.8, 76.7)
- moved J1 67.3 mm to (95.4, 72.2)
- moved SW1 65.4 mm to (122.9, 45.5), turned to 0 degrees
- moved Q2 56.4 mm to (141.3, 53.8), turned to 0 degrees
- moved D16 51.0 mm to (153.2, 43.7), turned to 0 degrees
- moved Q3 49.4 mm to (147.7, 44.7), turned to 0 degrees
- moved D2 48.5 mm to (86.8, 71.5)
- moved D7 48.5 mm to (111.9, 61.0), turned to 0 degrees
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Connections:
- D13 pad 2: Net-(D13-Pad2) -> Servo_Digital_Control
- D14 pad 2: Net-(D14-Pad2) -> Servo_Manual_Control
- D15 pad 1: GND -> Net-(D15-Pad1)
- D16 pad 1: GND -> Net-(D16-Pad1)
- D17 pad 1: GND -> Net-(D17-Pad1)
- D17 pad 2: Servo_Digital_Control -> Net-(D17-Pad2)
- D18 pad 1: GND -> Net-(D18-Pad1)
- D18 pad 2: Servo_Manual_Control -> Net-(D18-Pad2)
- D5 pad 1: Net-(D5-Pad1) -> GND
- D5 pad 2: GND -> Net-(D5-Pad2)
- D6 pad 1: Net-(D6-Pad1) -> GND
- D6 pad 2: GND -> Net-(D6-Pad2)
- D7 pad 1: Net-(D7-Pad1) -> GND
- D7 pad 2: +3V3 -> Net-(D7-Pad2)
- D8 pad 1: Net-(D8-Pad1) -> GND
- D8 pad 2: +5V -> Net-(D8-Pad2)
- Q1 pad 2: Net-(D22-Pad1) -> Net-(D15-Pad1)
- Q2 pad 2: Net-(D23-Pad1) -> Net-(D16-Pad1)
- Q3 pad 2: Net-(D24-Pad1) -> Net-(D17-Pad1)
- Q4 pad 2: Net-(D25-Pad1) -> Net-(D18-Pad1)
- Q8 pad 2: Net-(D29-Pad1) -> Net-(D22-Pad1)
Routing:
- net +3V3: track 449.7 -> 0.00 mm, vias 13 -> 0
- net +5V: track 86.1 -> 0.00 mm
- net Power_Input_Act: track 67.0 -> 0.00 mm, vias 2 -> 0
- net Net-(D5-Pad1): track 55.0 -> 0.00 mm, vias 1 -> 0
- net Servo_4_PWM: track 50.9 -> 0.00 mm, vias 1 -> 0
- net Power_Input_Log: track 43.5 -> 0.00 mm, vias 2 -> 0
- net Servo_3_PWM: track 41.0 -> 0.00 mm, vias 1 -> 0
- net Servo_8_AW: track 39.4 -> 0.00 mm, vias 1 -> 0
- net Servo_8_SW: track 38.6 -> 0.00 mm
- net Servo_Digital_Control: track 38.0 -> 0.00 mm
- net GND: track 37.1 -> 0.00 mm, vias 11 -> 0
- net Servo_7_SW: track 34.0 -> 0.00 mm
- net Servo_Manual_Control: track 33.0 -> 0.00 mm
- net Servo_2_PWM: track 32.7 -> 0.00 mm, vias 1 -> 0
- net Servo_6_SW: track 30.8 -> 0.00 mm
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- removed copper zone on B.Cu, net +5V
- removed copper zone on F.Cu, net GND
Other:
- board outline removed
- board text removed: "3.3V"
- board text removed: "5V"
- board text removed: "Actuation"
- board text removed: "Buck Converters"
- board text removed: "Digital/Manual Control"
- board text removed: "Logic"
- board text removed: "Manual Servo Control"
- board text removed: "Schott-kys"
- board text removed: "Servo Connectors"
- board text removed: "Servo Indicators"

Commit message: layout 10
Parts:
- added C1: 10uF, Capacitor_SMD:C_0603_1608Metric_Pad1.05x0.95mm_HandSolder, F.Cu at (209.3, 43.3)
- added C2: 10uF, Capacitor_SMD:C_0603_1608Metric_Pad1.05x0.95mm_HandSolder, F.Cu at (213.6, 43.3)
- added C3: 10uF, Capacitor_SMD:C_0603_1608Metric_Pad1.05x0.95mm_HandSolder, F.Cu at (209.3, 45.8)
- added C4: 10uF, Capacitor_SMD:C_0603_1608Metric_Pad1.05x0.95mm_HandSolder, F.Cu at (209.3, 48.3)
- added Conn1: AndersonPP, MRDT_Connectors:Anderson_3_Horizontal_Side_by_Side, F.Cu at (91.3, 205.3)
- added Conn2: Molex_SL_03, MRDT_Connectors:MOLEX_SL_03_Horizontal, F.Cu at (72.3, 219.8)
- added Conn3: Molex_SL_03, MRDT_Connectors:MOLEX_SL_03_Horizontal, F.Cu at (129.3, 210.5)
- added Conn4: Molex_SL_03, MRDT_Connectors:MOLEX_SL_03_Horizontal, F.Cu at (116.7, 210.5)
- added Conn5: Molex_SL_03, MRDT_Connectors:MOLEX_SL_03_Horizontal, F.Cu at (129.3, 194.8)
- added Conn6: Molex_SL_03, MRDT_Connectors:MOLEX_SL_03_Horizontal, F.Cu at (116.7, 194.8)
- added Conn7: Molex_SL_03, MRDT_Connectors:MOLEX_SL_03_Horizontal, F.Cu at (104.1, 210.5)
- added Conn8: Molex_SL_03, MRDT_Connectors:MOLEX_SL_03_Horizontal, F.Cu at (84.9, 219.8)
- added Conn9: Molex_SL_03, MRDT_Connectors:MOLEX_SL_03_Horizontal, F.Cu at (104.1, 194.8)
- added R1: 1k, Resistor_SMD:R_0603_1608Metric_Pad1.05x0.95mm_HandSolder, F.Cu at (263.0, 95.1)
- added R10: 330, Resistor_SMD:R_0603_1608Metric_Pad1.05x0.95mm_HandSolder, F.Cu at (225.2, 129.9)
- added R11: 330, Resistor_SMD:R_0603_1608Metric_Pad1.05x0.95mm_HandSolder, F.Cu at (229.6, 127.4)
- added R12: 330, Resistor_SMD:R_0603_1608Metric_Pad1.05x0.95mm_HandSolder, F.Cu at (233.9, 124.9)
- added R13: 500, Resistor_SMD:R_0603_1608Metric_Pad1.05x0.95mm_HandSolder, F.Cu at (154.1, 187.5)
- added R14: 500, Resistor_SMD:R_0603_1608Metric_Pad1.05x0.95mm_HandSolder, F.Cu at (158.5, 184.9)
- added R15: 500, Resistor_SMD:R_0603_1608Metric_Pad1.05x0.95mm_HandSolder, F.Cu at (149.7, 192.5)
- added R16: 500, Resistor_SMD:R_0603_1608Metric_Pad1.05x0.95mm_HandSolder, F.Cu at (154.1, 190.0)
- added R17: 500, Resistor_SMD:R_0603_1608Metric_Pad1.05x0.95mm_HandSolder, F.Cu at (162.8, 182.3)
- added R18: 500, Resistor_SMD:R_0603_1608Metric_Pad1.05x0.95mm_HandSolder, F.Cu at (149.7, 187.5)
- added R19: 500, Resistor_SMD:R_0603_1608Metric_Pad1.05x0.95mm_HandSolder, F.Cu at (158.4, 187.4)
- added R2: 1k, Resistor_SMD:R_0603_1608Metric_Pad1.05x0.95mm_HandSolder, F.Cu at (242.9, 112.6)
- added R20: 500, Resistor_SMD:R_0603_1608Metric_Pad1.05x0.95mm_HandSolder, F.Cu at (162.8, 184.8)
- added R21: 330, Resistor_SMD:R_0603_1608Metric_Pad1.05x0.95mm_HandSolder, F.Cu at (154.1, 192.5)
- added R22: 330, Resistor_SMD:R_0603_1608Metric_Pad1.05x0.95mm_HandSolder, F.Cu at (167.2, 182.3)
- added R23: 330, Resistor_SMD:R_0603_1608Metric_Pad1.05x0.95mm_HandSolder, F.Cu at (158.4, 189.9)
- added R24: 330, Resistor_SMD:R_0603_1608Metric_Pad1.05x0.95mm_HandSolder, F.Cu at (162.8, 187.4)
- added R25: 330, Resistor_SMD:R_0603_1608Metric_Pad1.05x0.95mm_HandSolder, F.Cu at (167.2, 184.8)
- added R26: 330, Resistor_SMD:R_0603_1608Metric_Pad1.05x0.95mm_HandSolder, F.Cu at (158.4, 192.4)
- added R27: 330, Resistor_SMD:R_0603_1608Metric_Pad1.05x0.95mm_HandSolder, F.Cu at (162.8, 189.9)
- added R28: 330, Resistor_SMD:R_0603_1608Metric_Pad1.05x0.95mm_HandSolder, F.Cu at (167.1, 187.3)
- added R3: 330, Resistor_SMD:R_0603_1608Metric_Pad1.05x0.95mm_HandSolder, F.Cu at (220.9, 132.4)
- added R4: 330, Resistor_SMD:R_0603_1608Metric_Pad1.05x0.95mm_HandSolder, F.Cu at (229.6, 124.9)
- added R5: 330, Resistor_SMD:R_0603_1608Metric_Pad1.05x0.95mm_HandSolder, F.Cu at (220.9, 127.4)
- added R6: 330, Resistor_SMD:R_0603_1608Metric_Pad1.05x0.95mm_HandSolder, F.Cu at (220.9, 124.9)
- added R7: 330, Resistor_SMD:R_0603_1608Metric_Pad1.05x0.95mm_HandSolder, F.Cu at (225.2, 124.9)
- added R8: 330, Resistor_SMD:R_0603_1608Metric_Pad1.05x0.95mm_HandSolder, F.Cu at (220.9, 129.9)
- added R9: 330, Resistor_SMD:R_0603_1608Metric_Pad1.05x0.95mm_HandSolder, F.Cu at (225.2, 127.4)
- added U1: OKI, MRDT_Devices:OKI_Horizontal, F.Cu at (184.9, 42.8)
- added U2: OKI, MRDT_Devices:OKI_Horizontal, F.Cu at (196.4, 42.8)
- added U3: TM4C129E_Launchpad, MRDT_Shields:TM4C129E_Launchpad_FULL_THT_BOTTOM, F.Cu at (66.8, 150.3)

Commit message: layout 11
Parts:
- removed the D10 at (117.9, 49.8)
- removed the D3 at (86.8, 74.1)
- removed the D4 at (91.2, 71.5)
- removed the R1 at (263.0, 95.1)
- removed the R19 at (158.4, 187.4)
- removed the R2 at (242.9, 112.6)
- removed the R20 at (162.8, 184.8)
- removed R28: 330, Resistor_SMD:R_0603_1608Metric_Pad1.05x0.95mm_HandSolder
- added D20: LED, LED_SMD:LED_0603_1608Metric_Pad1.05x0.95mm_HandSolder, F.Cu at (177.7, 95.0)
- added D21: LED, LED_SMD:LED_0603_1608Metric_Pad1.05x0.95mm_HandSolder, F.Cu at (195.2, 136.1)
- added D23: LED, LED_SMD:LED_0603_1608Metric_Pad1.05x0.95mm_HandSolder, F.Cu at (195.7, 145.8)
- added D24: LED, LED_SMD:LED_0603_1608Metric_Pad1.05x0.95mm_HandSolder, F.Cu at (195.9, 150.4)
- added D8: LED, LED_SMD:LED_0603_1608Metric_Pad1.05x0.95mm_HandSolder, F.Cu at (107.6, 128.5)
- added R15: 500, Resistor_SMD:R_0603_1608Metric_Pad1.05x0.95mm_HandSolder, F.Cu at (142.0, 94.1)
- added R18: 500, Resistor_SMD:R_0603_1608Metric_Pad1.05x0.95mm_HandSolder, F.Cu at (187.7, 94.1)
- added R26: 330, Resistor_SMD:R_0603_1608Metric_Pad1.05x0.95mm_HandSolder, F.Cu at (177.7, 97.0)
- moved R10 157.2 mm to (77.2, 112.4), turned to 90 degrees
- moved R9 152.5 mm to (77.2, 120.3), turned to 270 degrees
- moved Conn8 151.8 mm to (166.9, 91.9)
- moved R2 147.4 mm to (82.2, 126.5)
- moved R1 145.0 mm to (76.1, 126.5)
- moved R3 132.4 mm to (88.5, 126.5)
- moved Conn1 131.4 mm to (175.3, 104.1), turned to 180 degrees
- moved Conn9 129.1 mm to (182.1, 91.9)
- moved Conn2 127.9 mm to (75.4, 91.9)
- moved Conn7 127.7 mm to (151.6, 91.9)
- moved R19 126.5 mm to (71.0, 97.0), turned to 180 degrees
- moved R4 126.0 mm to (94.9, 126.5)
- moved Conn3 124.6 mm to (90.7, 91.9)
- moved R5 124.0 mm to (101.2, 126.5)
- moved Conn4 119.0 mm to (105.9, 91.9)
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- renumbered D12 to D10, D13 to D11, D14 to D12, D15 to D13, D16 to D14, D17 to D15, D18 to D16, D19 to D17, D20 to D18, D21 to D19, D5 to D3, D6 to D4, D7 to D5, D8 to D6, D9 to D7, D11 to D9, R3 to R1, R12 to R10, R13 to R11, R14 to R12, R15 to R13, R16 to R14, R18 to R16, R21 to R19, R4 to R2, R22 to R20, R23 to R21, R24 to R22, R25 to R23, R26 to R24, R27 to R25, R5 to R3, R6 to R4, R7 to R5, R8 to R6, R9 to R7, R10 to R8, R11 to R9
Connections:
- D22 pad 1: Net-(D22-Pad1) -> GND
- Q8 pad 2: Net-(D22-Pad1) -> Net-(D20-Pad1)
- R17 pad 1: Servo_5_PWM -> Servo_7_PWM
- R17 pad 2: Net-(Q5-Pad1) -> Net-(Q7-Pad1)
