File: Hardware/gimble_board/gimble_board.kicad_pcb (KiCad board)
At the start: 2 copper layers, 85 parts, among them J1 Test_Point, J2 Test_Point, Q1 Q_NMOS_GDS, Q2 Q_NMOS_GDS, Q3 Q_NMOS_GDS, Q4 Q_NMOS_GDS, Q5 Q_NMOS_GDS, Q6 Q_NMOS_GDS, Q7 Q_NMOS_GDS, Q8 Q_NMOS_GDS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

Commit message: layout 12
Parts:
- added R27: 1000, Resistor_SMD:R_0603_1608Metric_Pad1.05x0.95mm_HandSolder, F.Cu at (206.7, 114.9)
- added R28: 1000, Resistor_SMD:R_0603_1608Metric_Pad1.05x0.95mm_HandSolder, F.Cu at (206.7, 117.4)
- added R29: 330, Resistor_SMD:R_0603_1608Metric_Pad1.05x0.95mm_HandSolder, F.Cu at (211.0, 114.9)
- added R30: 330, Resistor_SMD:R_0603_1608Metric_Pad1.05x0.95mm_HandSolder, F.Cu at (211.0, 117.4)
Changed lines of the file:
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@@
-(kicad_pcb (version 20171130) (host pcbnew "(5.1.7)-1")
+(kicad_pcb (version 20171130) (host pcbnew "(5.1.4)-1")
   (general
     (thickness 1.6)
@@
     (tracks 0)
     (zones 0)
-    (modules 85)
+    (modules 89)
     (nets 116)
   )
@@
   )
   (setup
-    (last_trace_width 0.381)
+    (last_trace_width 0.25)
     (user_trace_width 0.381)
     (user_trace_width 0.762)
@@
       (at (xyz 0 0 0))
       (scale (xyz 1 1 1))
+      (rotate (xyz 0 0 0))
+    )
+  )
+  (module Resistor_SMD:R_0603_1608Metric_Pad1.05x0.95mm_HandSolder (layer F.Cu)
+    (at 206.653001 114.928001)
+    (descr "Resistor SMD 0603 (1608 Metric), square (rectangular) end terminal, IPC_7351 nominal with elongated pad for handsoldering. (Body size source: http://www.tortai-tech.com/upload/download/2011102023233369053.pdf), generated with kicad-footprint-generator")
+    (tags "resistor handsolder")
+    (attr smd)
+    (fp_text reference R27 (at 0 -1.43) (layer F.SilkS)
+      (effects (font (size 1 1) (thickness 0.15)))
+    )
+    (fp_text value 1000 (at 0 1.43) (layer F.Fab)
+      (effects (font (size 1 1) (thickness 0.15)))
+    )
+    (fp_line (start -0.8 0.4) (end -0.8 -0.4) (layer F.Fab) (width 0.1))
+    (fp_line (start -0.8 -0.4) (end 0.8 -0.4) (layer F.Fab) (width 0.1))
+    (fp_line (start 0.8 -0.4) (end 0.8 0.4) (layer F.Fab) (width 0.1))
+    (fp_line (start 0.8 0.4) (end -0.8 0.4) (layer F.Fab) (width 0.1))
+    (fp_line (start -0.171267 -0.51) (end 0.171267 -0.51) (layer F.SilkS) (width 0.12))
+    (fp_line (start -0.171267 0.51) (end 0.171267 0.51) (layer F.SilkS) (width 0.12))
+    (fp_line (start -1.65 0.73) (end -1.65 -0.73) (layer F.CrtYd) (width 0.05))
+    (fp_line (start -1.65 -0.73) (end 1.65 -0.73) (layer F.CrtYd) (width 0.05))
+    (fp_line (start 1.65 -0.73) (end 1.65 0.73) (layer F.CrtYd) (width 0.05))
+    (fp_line (start 1.65 0.73) (end -1.65 0.73) (layer F.CrtYd) (width 0.05))
+    (fp_text user %R (at 0 0) (layer F.Fab)
+      (effects (font (size 0.4 0.4) (thickness 0.06)))
+    )
+    (pad 1 smd roundrect (at -0.875 0) (size 1.05 0.95) (layers F.Cu F.Paste F.Mask) (roundrect_rratio 0.25)
+      (net 42 "Net-(D21-Pad2)"))
+    (pad 2 smd roundrect (at 0.875 0) (size 1.05 0.95) (layers F.Cu F.Paste F.Mask) (roundrect_rratio 0.25)
+      (net 2 Power_Input_Log))
+    (model ${KISYS3DMOD}/Resistor_SMD.3dshapes/R_0603_1608Metric.wrl
+      (at (xyz 0 0 0))
+      (scale (xyz 1 1 1))
+      (rotate (xyz 0 0 0))
+    )
+  )
+  (module Resistor_SMD:R_0603_1608Metric_Pad1.05x0.95mm_HandSolder (layer F.Cu)
+    (at 206.653001 117.438001)
+    (descr "Resistor SMD 0603 (1608 Metric), square (rectangular) end terminal, IPC_7351 nominal with elongated pad for handsoldering. (Body size source: http://www.tortai-tech.com/upload/download/2011102023233369053.pdf), generated with kicad-footprint-generator")
+    (tags "resistor handsolder")
+    (attr smd)
+    (fp_text reference R28 (at 0 -1.43) (layer F.SilkS)
+      (effects (font (size 1 1) (thickness 0.15)))
+    )
+    (fp_text value 1000 (at 0 1.43) (layer F.Fab)
+      (effects (font (size 1 1) (thickness 0.15)))
+    )
+    (fp_text user %R (at 0 0) (layer F.Fab)
+      (effects (font (size 0.4 0.4) (thickness 0.06)))
+    )
+    (fp_line (start 1.65 0.73) (end -1.65 0.73) (layer F.CrtYd) (width 0.05))
+    (fp_line (start 1.65 -0.73) (end 1.65 0.73) (layer F.CrtYd) (width 0.05))
+    (fp_line (start -1.65 -0.73) (end 1.65 -0.73) (layer F.CrtYd) (width 0.05))
+    (fp_line (start -1.65 0.73) (end -1.65 -0.73) (layer F.CrtYd) (width 0.05))
+    (fp_line (start -0.171267 0.51) (end 0.171267 0.51) (layer F.SilkS) (width 0.12))
+    (fp_line (start -0.171267 -0.51) (end 0.171267 -0.51) (layer F.SilkS) (width 0.12))
+    (fp_line (start 0.8 0.4) (end -0.8 0.4) (layer F.Fab) (width 0.1))
+    (fp_line (start 0.8 -0.4) (end 0.8 0.4) (layer F.Fab) (width 0.1))
+    (fp_line (start -0.8 -0.4) (end 0.8 -0.4) (layer F.Fab) (width 0.1))
+    (fp_line (start -0.8 0.4) (end -0.8 -0.4) (layer F.Fab) (width 0.1))
+    (pad 2 smd roundrect (at 0.875 0) (size 1.05 0.95) (layers F.Cu F.Paste F.Mask) (roundrect_rratio 0.25)
+      (net 3 Power_Input_Act))
+    (pad 1 smd roundrect (at -0.875 0) (size 1.05 0.95) (layers F.Cu F.Paste F.Mask) (roundrect_rratio 0.25)
+      (net 11 "Net-(D22-Pad2)"))
+    (model ${KISYS3DMOD}/Resistor_SMD.3dshapes/R_0603_1608Metric.wrl
+      (at (xyz 0 0 0))
+      (scale (xyz 1 1 1))
+      (rotate (xyz 0 0 0))
+    )
+  )
+  (module Resistor_SMD:R_0603_1608Metric_Pad1.05x0.95mm_HandSolder (layer F.Cu)
+    (at 211.003001 114.928001)
+    (descr "Resistor SMD 0603 (1608 Metric), square (rectangular) end terminal, IPC_7351 nominal with elongated pad for handsoldering. (Body size source: http://www.tortai-tech.com/upload/download/2011102023233369053.pdf), generated with kicad-footprint-generator")
+    (tags "resistor handsolder")
+    (attr smd)
+    (fp_text reference R29 (at 0 -1.43) (layer F.SilkS)
+      (effects (font (size 1 1) (thickness 0.15)))
+    )
+    (fp_text value 330 (at 0 1.43) (layer F.Fab)
+      (effects (font (size 1 1) (thickness 0.15)))
+    )
+    (fp_text user %R (at 0 0) (layer F.Fab)
+      (effects (font (size 0.4 0.4) (thickness 0.06)))
+    )
+    (fp_line (start 1.65 0.73) (end -1.65 0.73) (layer F.CrtYd) (width 0.05))
+    (fp_line (start 1.65 -0.73) (end 1.65 0.73) (layer F.CrtYd) (width 0.05))
+    (fp_line (start -1.65 -0.73) (end 1.65 -0.73) (layer F.CrtYd) (width 0.05))
+    (fp_line (start -1.65 0.73) (end -1.65 -0.73) (layer F.CrtYd) (width 0.05))
+    (fp_line (start -0.171267 0.51) (end 0.171267 0.51) (layer F.SilkS) (width 0.12))
+    (fp_line (start -0.171267 -0.51) (end 0.171267 -0.51) (layer F.SilkS) (width 0.12))
+    (fp_line (start 0.8 0.4) (end -0.8 0.4) (layer F.Fab) (width 0.1))
+    (fp_line (start 0.8 -0.4) (end 0.8 0.4) (layer F.Fab) (width 0.1))
+    (fp_line (start -0.8 -0.4) (end 0.8 -0.4) (layer F.Fab) (width 0.1))
+    (fp_line (start -0.8 0.4) (end -0.8 -0.4) (layer F.Fab) (width 0.1))
+    (pad 2 smd roundrect (at 0.875 0) (size 1.05 0.95) (layers F.Cu F.Paste F.Mask) (roundrect_rratio 0.25)
+      (net 4 +3V3))
+    (pad 1 smd roundrect (at -0.875 0) (size 1.05 0.95) (layers F.Cu F.Paste F.Mask) (roundrect_rratio 0.25)
+      (net 112 "Net-(D23-Pad2)"))
+    (model ${KISYS3DMOD}/Resistor_SMD.3dshapes/R_0603_1608Metric.wrl
+      (at (xyz 0 0 0))
+      (scale (xyz 1 1 1))
+      (rotate (xyz 0 0 0))
+    )
+  )
+  (module Resistor_SMD:R_0603_1608Metric_Pad1.05x0.95mm_HandSolder (layer F.Cu)
+    (at 211.003001 117.438001)
+    (descr "Resistor SMD 0603 (1608 Metric), square (rectangular) end terminal, IPC_7351 nominal with elongated pad for handsoldering. (Body size source: http://www.tortai-tech.com/upload/download/2011102023233369053.pdf), generated with kicad-footprint-generator")
+    (tags "resistor handsolder")
+    (attr smd)
+    (fp_text reference R30 (at 0 -1.43) (layer F.SilkS)
+      (effects (font (size 1 1) (thickness 0.15)))
+    )
+    (fp_text value 330 (at 0 1.43) (layer F.Fab)
+      (effects (font (size 1 1) (thickness 0.15)))
+    )
+    (fp_line (start -0.8 0.4) (end -0.8 -0.4) (layer F.Fab) (width 0.1))
+    (fp_line (start -0.8 -0.4) (end 0.8 -0.4) (layer F.Fab) (width 0.1))
+    (fp_line (start 0.8 -0.4) (end 0.8 0.4) (layer F.Fab) (width 0.1))
+    (fp_line (start 0.8 0.4) (end -0.8 0.4) (layer F.Fab) (width 0.1))
+    (fp_line (start -0.171267 -0.51) (end 0.171267 -0.51) (layer F.SilkS) (width 0.12))
+    (fp_line (start -0.171267 0.51) (end 0.171267 0.51) (layer F.SilkS) (width 0.12))
+    (fp_line (start -1.65 0.73) (end -1.65 -0.73) (layer F.CrtYd) (width 0.05))
+    (fp_line (start -1.65 -0.73) (end 1.65 -0.73) (layer F.CrtYd) (width 0.05))
+    (fp_line (start 1.65 -0.73) (end 1.65 0.73) (layer F.CrtYd) (width 0.05))
+    (fp_line (start 1.65 0.73) (end -1.65 0.73) (layer F.CrtYd) (width 0.05))
+    (fp_text user %R (at 0 0) (layer F.Fab)
+      (effects (font (size 0.4 0.4) (thickness 0.06)))
+    )
+    (pad 1 smd roundrect (at -0.875 0) (size 1.05 0.95) (layers F.Cu F.Paste F.Mask) (roundrect_rratio 0.25)
+      (net 113 "Net-(D24-Pad2)"))
+    (pad 2 smd roundrect (at 0.875 0) (size 1.05 0.95) (layers F.Cu F.Paste F.Mask) (roundrect_rratio 0.25)
+      (net 43 +5V))
+    (model ${KISYS3DMOD}/Resistor_SMD.3dshapes/R_0603_1608Metric.wrl
+      (at (xyz 0 0 0))
+      (scale (xyz 1 1 1))

Commit message: layout 13
Parts:
- moved D24 103.2 mm to (114.9, 86.5), turned to 180 degrees
- moved R30 100.0 mm to (114.9, 89.7)
- moved D22 92.3 mm to (121.4, 86.5), turned to 180 degrees
- moved R28 89.7 mm to (121.4, 89.7)
- moved D23 88.8 mm to (129.7, 86.5), turned to 180 degrees
- moved R29 85.2 mm to (129.7, 89.7)
- moved D21 77.2 mm to (136.1, 86.5), turned to 180 degrees
- moved R27 74.9 mm to (136.1, 89.7)
- moved U2 56.0 mm to (106.7, 106.6)
- moved J1 47.4 mm to (142.9, 88.3)
- moved J2 42.6 mm to (142.9, 80.0)
- moved C3 40.3 mm to (113.9, 108.1), turned to 180 degrees
- moved C4 38.6 mm to (119.5, 108.1), turned to 180 degrees
- moved D6 38.5 mm to (70.7, 98.6)
- moved D7 38.5 mm to (77.1, 98.6)
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Connections:
- U3 pad PC4: Servo_Manual_Control -> Net-(U3-PadPC4)
- U3 pad PE4: Servo_Digital_Control -> Net-(U3-PadPE4)
- U3 pad PL0: Net-(U3-PadPL0) -> Servo_Digital_Control
- U3 pad PL1: Net-(U3-PadPL1) -> Servo_Manual_Control
Routing:
- net +3V3: track 0.00 -> 361.3 mm, vias 0 -> 1
- net Power_Input_Act: track 0.00 -> 77.8 mm, vias 0 -> 1
- net +5V: track 0.00 -> 72.8 mm, vias 0 -> 1
- net Servo_4_PWM: track 0.00 -> 57.9 mm
- net Servo_8_AW: track 0.00 -> 55.4 mm
- net Power_Input_Log: track 0.00 -> 45.4 mm, vias 0 -> 1
- net Servo_3_PWM: track 0.00 -> 45.2 mm
- net Servo_7_PWM: track 0.00 -> 42.7 mm
- net Servo_8_SW: track 0.00 -> 40.3 mm, vias 0 -> 1
- net Servo_7_SW: track 0.00 -> 36.7 mm, vias 0 -> 1
- net Servo_6_SW: track 0.00 -> 32.9 mm, vias 0 -> 1
- net Servo_2_PWM: track 0.00 -> 32.5 mm
- net Servo_6_PWM: track 0.00 -> 30.0 mm
- net Servo_5_SW: track 0.00 -> 29.1 mm, vias 0 -> 1
- net Servo_4_SW: track 0.00 -> 25.3 mm, vias 0 -> 1
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- added copper zone on B.Cu, net +5V
- added copper zone on F.Cu, net GND
Other:
- board outline added: 124.5 x 95.5 mm
- board text added: "12V Actuation"
- board text added: "12V Logic"
- board text added: "3.3V"
- board text added: "5V"
- board text added: "Actuation"
- board text added: "Digital/Manual Switch"
- board text added: "GND"
- board text added: "Logic"
- board text added: "Manual Servo Control Buttons"
- board text added: "Test Points"

Commit message: layout 14
Parts:
- added G***: LOGO, Signature:z_sig_Jack_Schott_15.2mmx27mm, F.Cu at (97.0, 132.6)
- added G***: LOGO, MRDT_Silkscreens:2_Dahlbot_2.0, F.Cu at (53.1, 86.9)
- added G***: LOGO, MRDT_Silkscreens:0_MRDT_Logo_20mm, F.Cu at (137.9, 131.8)
- moved SW9 1.80 mm to (71.6, 89.2)
- moved D11 1.80 mm to (64.5, 91.0)
- moved D12 1.80 mm to (64.5, 83.2)
- moved R10 1.80 mm to (67.1, 83.2)
- moved R9 1.80 mm to (67.1, 91.0)
- moved D10 1.02 mm to (96.1, 97.5)
- moved D3 1.02 mm to (51.7, 97.5)
- moved D4 1.02 mm to (58.0, 97.5)
- moved D5 1.02 mm to (64.4, 97.5)
- moved D6 1.02 mm to (70.7, 97.5)
- moved D7 1.02 mm to (77.1, 97.5)
- moved D8 1.02 mm to (83.4, 97.5)
- moved D9 1.02 mm to (89.8, 97.5)
- moved R1 1.02 mm to (51.7, 99.6)
- moved R2 1.02 mm to (58.0, 99.6)
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Routing:
- net +5V: track 72.8 -> 36.8 mm, vias 1 -> 0
- net +3V3: track 361.3 -> 364.3 mm
- net Servo_Digital_Control: track 21.0 -> 19.2 mm
- net Servo_Manual_Control: track 10.4 -> 8.77 mm
- net Servo_8_SW: track 40.3 -> 41.3 mm
- net Servo_7_SW: track 36.7 -> 37.8 mm
- net Servo_5_SW: track 29.1 -> 30.1 mm
- net Servo_3_SW: track 21.5 -> 22.5 mm
- net Servo_1_SW: track 17.1 -> 18.1 mm
- net Servo_4_SW: track 25.3 -> 26.3 mm
- net Servo_2_SW: track 18.7 -> 19.7 mm
- net Servo_6_SW: track 32.9 -> 34.0 mm
Other:
- board text added: "+5V GND PWM"
- board text added: "12V Act."
- board text added: "Gimbal Board Mars Rover Design Team Missouri S&T, 2021 Jack Schott"
- board text added: "Ground"
- board text added: "Servo 1"
- board text added: "Servo 2"
- board text added: "Servo 3"
- board text added: "Servo 4"
- board text added: "Servo 5"
- board text added: "Servo 6"
- board text added: "Servo 7"
- board text added: "Servo 8"
- board text added: "Time-out Zone"
- board text removed: "12V Actuation"
- board text removed: "GND"

Commit message: layout 15
Parts:
- moved G*** 6.10 mm to (103.1, 132.8)
Changed lines of the file:
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@@
   )
   (setup
-    (last_trace_width 0.381)
+    (last_trace_width 0.25)
     (user_trace_width 0.381)
     (user_trace_width 0.762)
@@
   )
   (module Signature:z_sig_Jack_Schott_15.2mmx27mm (layer F.Cu)
-    (at 97.028 132.588 90)
+    (at 103.124 132.842 90)
     (fp_text reference G*** (at 0 0 90) (layer F.SilkS) hide
       (effects (font (size 1.524 1.524) (thickness 0.3)))

Commit message: layout 16
Other:
- board text added: "Gimbal Board Rev1 Mars Rover Design Team Missouri S&T, 2021 Jack Schott"
- board text removed: "Gimbal Board Mars Rover Design Team Missouri S&T, 2021 Jack Schott"

Commit message: layout 17
Parts:
- removed G***: LOGO, Signature:z_sig_Jack_Schott_15.2mmx27mm
- removed G***: LOGO, MRDT_Silkscreens:2_Dahlbot_2.0
- removed G***: LOGO, MRDT_Silkscreens:0_MRDT_Logo_20mm
- added C5: 10uF, Capacitor_SMD:C_0603_1608Metric_Pad1.05x0.95mm_HandSolder, F.Cu at (161.7, 26.9)
- added C6: 10uF, Capacitor_SMD:C_0603_1608Metric_Pad1.05x0.95mm_HandSolder, F.Cu at (166.1, 26.9)
- added U4: OKI, MRDT_Devices:OKI_Horizontal, F.Cu at (148.8, 26.4)

Commit message: layout 18
Parts:
- removed C5, C6: 10uF, Capacitor_SMD:C_0603_1608Metric_Pad1.05x0.95mm_HandSolder
- moved U4 81.8 mm to (84.3, 76.7)
- moved C3 41.3 mm to (83.3, 80.4), turned to 270 degrees
- moved C4 39.8 mm to (83.3, 91.6), turned to 90 degrees
- moved D2 33.4 mm to (83.3, 86.0), turned to 270 degrees
- moved U2 32.1 mm to (95.0, 76.7), turned to 0 degrees
- moved C1 20.5 mm to (114.2, 110.6)
- moved D1 20.5 mm to (108.8, 110.6)
- moved C2 20.5 mm to (119.5, 110.6)
- moved U1 20.5 mm to (107.2, 109.1)
Routing:
- net Power_Input_Log: track 45.4 -> 62.2 mm, vias 1 -> 0
- net +3V3: track 364.3 -> 347.8 mm, vias 1 -> 3
- net +5V: track 36.8 -> 49.2 mm, vias 0 -> 1
- net Power_Input_Act: track 77.8 -> 86.6 mm, vias 1 -> 0

Commit message: layout 19
Parts:
- added G***: LOGO, MRDT_Silkscreens:2_Dahlbot_2.0, F.Cu at (53.1, 86.6)
- added G***: LOGO, MRDT_Silkscreens:0_MRDT_Logo_20mm, F.Cu at (126.2, 131.6)
- added G***: LOGO, Signature:z_sig_Jack_Schott_15.2mmx27mm, F.Cu at (97.8, 132.6)
