File: Hardware/gimble_board/gimble_board.kicad_pcb (KiCad board)
At the start: 2 copper layers, 124.5 x 95.5 mm, 93 parts, among them J1 Test_Point, J2 Test_Point, Q1 Q_NMOS_GDS, Q2 Q_NMOS_GDS, Q3 Q_NMOS_GDS, Q4 Q_NMOS_GDS, Q5 Q_NMOS_GDS, Q6 Q_NMOS_GDS, Q7 Q_NMOS_GDS, Q8 Q_NMOS_GDS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

Commit message: checklist
Other:
- board text added: "5V OKIs"
Changed lines of the file:
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@@
   (general
     (thickness 1.6)
-    (drawings 86)
+    (drawings 91)
     (tracks 270)
     (zones 0)
@@
       (outputformat 1)
       (mirror false)
-      (drillshape 1)
+      (drillshape 0)
       (scaleselection 1)
-      (outputdirectory ""))
+      (outputdirectory "../../Documentation/Gerbs/"))
   )
   (net 0 "")
@@
     (at 94.996 76.708)
     (tags OKI)
-    (fp_text reference U2 (at 2.54 -1.27) (layer F.SilkS) hide
+    (fp_text reference U2 (at 1.016 -0.762) (layer F.SilkS) hide
       (effects (font (size 1 1) (thickness 0.15)))
     )
-    (fp_text value OKI (at 11.557 9.144 270) (layer F.SilkS)
+    (fp_text value OKI (at 4.826 -0.762) (layer F.SilkS) hide
       (effects (font (size 1 1) (thickness 0.15)))
     )
@@
     (at 84.328 76.708)
     (tags OKI)
-    (fp_text reference U4 (at 2.54 -1.27) (layer F.SilkS) hide
+    (fp_text reference U4 (at 1.778 -0.762) (layer F.SilkS) hide
       (effects (font (size 1 1) (thickness 0.15)))
     )
-    (fp_text value OKI (at 5.08 -1.27) (layer F.SilkS)
+    (fp_text value OKI (at -0.508 -1.524) (layer F.SilkS) hide
       (effects (font (size 1 1) (thickness 0.15)))
     )
@@
     )
   )
+  (gr_line (start 105.664 75.946) (end 105.664 93.726) (layer F.SilkS) (width 0.12))
+  (gr_line (start 105.41 75.946) (end 105.664 75.946) (layer F.SilkS) (width 0.12))
+  (gr_line (start 82.042 75.946) (end 105.41 75.946) (layer F.SilkS) (width 0.12))
+  (gr_line (start 82.042 93.726) (end 82.042 75.946) (layer F.SilkS) (width 0.12))
+  (gr_line (start 105.664 93.726) (end 82.042 93.726) (layer F.SilkS) (width 0.12))
   (gr_line (start 47.752 97.536) (end 47.752 96.012) (layer F.SilkS) (width 0.12))
   (gr_line (start 99.06 111.506) (end 98.806 111.506) (layer F.SilkS) (width 0.12))
@@
   (gr_line (start 106.68 98.552) (end 124.46 98.552) (layer F.SilkS) (width 0.12))
   (gr_line (start 106.68 111.76) (end 106.68 98.552) (layer F.SilkS) (width 0.12))
-  (gr_text 5V (at 93.98 73.152) (layer F.SilkS)
+  (gr_text "5V OKIs" (at 94.996 75.184) (layer F.SilkS)
     (effects (font (size 1 1) (thickness 0.15)))
   )
