File: Hardware/gimble_board/GimbleBoard01.sch (KiCad schematic (older format))
At the start: 21 parts, among them J1 Test_Point, J2 Test_Point, J3 Test_Point, U1 LM2576D2TR4, U2 LM2576D2TR4

Commit message: Replaced zener with schottky
Parts:
- removed D3, D4: D_Zener, symbol Device:D_Zener
- added D3, D4: D_Schottky, symbol Device:D_Schottky
Changed lines of the file:
@@
-$EndComp
-$Comp
-L Device:D_Zener D3
-U 1 1 5F7FDDFC
-P 5550 1750
-F 0 "D3" V 5504 1830 50  0000 L CNN
-F 1 "D_Zener" V 5595 1830 50  0000 L CNN
-F 2 "" H 5550 1750 50  0001 C CNN
-F 3 "~" H 5550 1750 50  0001 C CNN
-	1    5550 1750
-	0    1    1    0
 $EndComp
 $Comp
@@
 	7350 1600 7200 1600
 Wire Wire Line
-	5550 1600 5700 1600
-Wire Wire Line
 	5550 1900 5550 2050
 Wire Wire Line
 	6000 1600 6150 1600
-Wire Wire Line
-	5550 1600 5400 1600
-Connection ~ 5550 1600
 Wire Wire Line
 	5400 1750 5400 2350
@@
 $EndComp
 $Comp
-L Device:D_Zener D4
-U 1 1 5F98D276
-P 5550 3450
-F 0 "D4" V 5504 3530 50  0000 L CNN
-F 1 "D_Zener" V 5595 3530 50  0000 L CNN
-F 2 "" H 5550 3450 50  0001 C CNN
-F 3 "~" H 5550 3450 50  0001 C CNN
-	1    5550 3450
-	0    1    1    0
-$EndComp
-$Comp
 L power:GND #PWR012
 U 1 1 5F98D27C
@@
 	7350 3300 7200 3300
 Wire Wire Line
-	5550 3300 5700 3300
-Wire Wire Line
 	5550 3600 5550 3750
 Wire Wire Line
 	6000 3300 6150 3300
-Wire Wire Line
-	5550 3300 5400 3300
-Connection ~ 5550 3300
 Wire Wire Line
 	5400 3450 5400 4050
@@
 Wire Wire Line
 	3300 1500 3300 1650
+Wire Wire Line
+	5400 3300 5550 3300
+$Comp
+L Device:D_Schottky D4
+U 1 1 5F8005E7
+P 5550 3450
+F 0 "D4" V 5504 3530 50  0000 L CNN
+F 1 "D_Schottky" V 5595 3530 50  0000 L CNN
+F 2 "" H 5550 3450 50  0001 C CNN
+F 3 "~" H 5550 3450 50  0001 C CNN
+	1    5550 3450
+	0    1    1    0
+$EndComp
+Connection ~ 5550 3300
+Wire Wire Line
+	5550 3300 5700 3300
+Wire Wire Line
+	5400 1600 5550 1600
+$Comp
+L Device:D_Schottky D3
+U 1 1 5F80152B
+P 5550 1750
+F 0 "D3" V 5504 1830 50  0000 L CNN
+F 1 "D_Schottky" V 5595 1830 50  0000 L CNN
+F 2 "" H 5550 1750 50  0001 C CNN
+F 3 "~" H 5550 1750 50  0001 C CNN
+	1    5550 1750
+	0    1    1    0
+$EndComp
+Connection ~ 5550 1600
+Wire Wire Line
+	5550 1600 5700 1600
 $EndSCHEMATC

Commit message: fixed bucks
Parts:
- U1: value LM2576D2TR4 -> LM2576SX-3.3
- U2: value LM2576D2TR4 -> LM2576SX-5.0
Changed lines of the file:
@@
 P 4900 1650
 F 0 "U1" H 4900 2075 50  0000 C CNN
-F 1 "LM2576D2TR4" H 4900 1984 50  0000 C CNN
+F 1 "LM2576SX-3.3" H 4900 1984 50  0000 C CNN
 F 2 "" H 4900 2100 50  0001 C CNN
 F 3 "https://www.mouser.com/datasheet/2/308/LM2576_D-1810688.pdf" H 4900 2100 50  0001 C CNN
@@
 P 4900 3350
 F 0 "U2" H 4900 3775 50  0000 C CNN
-F 1 "LM2576D2TR4" H 4900 3684 50  0000 C CNN
+F 1 "LM2576SX-5.0" H 4900 3684 50  0000 C CNN
 F 2 "" H 4900 3800 50  0001 C CNN
 F 3 "https://www.mouser.com/datasheet/2/308/LM2576_D-1810688.pdf" H 4900 3800 50  0001 C CNN

Commit message: footprints
Parts:
- removed FB1: Ferrite_Bead, symbol Device:Ferrite_Bead
- added D2: D_Zener, LED_SMD:LED_0603_1608Metric_Pad1.05x0.95mm_HandSolder, symbol Device:D_Zener
- added D4: LED, LED_SMD:LED_0603_1608Metric_Pad1.05x0.95mm_HandSolder, symbol Device:LED
- added J2: Test_Point, TestPoint:TestPoint_Pad_2.0x2.0mm, symbol MRDT_Connectors:Test_Point
- added R2: 1k, Resistor_SMD:R_0603_1608Metric_Pad1.05x0.95mm_HandSolder, symbol Device:R
- C1, C4: footprint (none) -> Capacitor_SMD:C_0603_1608Metric_Pad1.05x0.95mm_HandSolder
- C2: renamed from C3; footprint (none) -> Capacitor_SMD:C_0603_1608Metric_Pad1.05x0.95mm_HandSolder
- C3: renamed from C2; footprint (none) -> Capacitor_SMD:C_0603_1608Metric_Pad1.05x0.95mm_HandSolder
- D1: footprint (none) -> LED_SMD:LED_0603_1608Metric_Pad1.05x0.95mm_HandSolder
- D3: renamed from D2; footprint (none) -> LED_SMD:LED_0603_1608Metric_Pad1.05x0.95mm_HandSolder
- D5: renamed from D3; footprint (none) -> Diode_THT:D_DO-201AD_P15.24mm_Horizontal
- D6: renamed from D4; footprint (none) -> Diode_THT:D_DO-201AD_P15.24mm_Horizontal
- D7: renamed from D5; footprint (none) -> LED_SMD:LED_0603_1608Metric_Pad1.05x0.95mm_HandSolder
- D8: renamed from D6; footprint (none) -> LED_SMD:LED_0603_1608Metric_Pad1.05x0.95mm_HandSolder
- J1: footprint (none) -> TestPoint:TestPoint_Pad_2.0x2.0mm
- J3: renamed from J2; footprint (none) -> TestPoint:TestPoint_Pad_2.0x2.0mm
- J4: renamed from J3; footprint (none) -> TestPoint:TestPoint_Pad_2.0x2.0mm
- L1, L2: footprint (none) -> Inductor_SMD:L_0603_1608Metric_Pad1.05x0.95mm_HandSolder
- R1: footprint (none) -> Resistor_SMD:R_0603_1608Metric_Pad1.05x0.95mm_HandSolder
- R3: renamed from R2; footprint (none) -> Resistor_SMD:R_0603_1608Metric_Pad1.05x0.95mm_HandSolder
- R4: renamed from R3; footprint (none) -> Resistor_SMD:R_0603_1608Metric_Pad1.05x0.95mm_HandSolder
- U1, U2: footprint (none) -> Package_TO_SOT_SMD:TO-263-6
Connections:
- net labels added: +12VA, Power_Input_Act, Power_Input_Log
- net labels removed: Power_Input
- wire segments 68 -> 78
Other:
- moved on the sheet: D1

Commit message: layout 9
Parts:
- removed D5, D6: D_Schottky, Diode_THT:D_DO-201AD_P15.24mm_Horizontal, symbol Device:D_Schottky
- removed D7, D8: LED, LED_SMD:LED_0603_1608Metric_Pad1.05x0.95mm_HandSolder, symbol Device:LED
- removed J3, J4: Test_Point, TestPoint:TestPoint_Pad_2.0x2.0mm, symbol MRDT_Connectors:Test_Point
- removed L1, L2: 100uH, Inductor_SMD:L_0603_1608Metric_Pad1.05x0.95mm_HandSolder, symbol Device:L
- removed R3: 330, Resistor_SMD:R_0603_1608Metric_Pad1.05x0.95mm_HandSolder, symbol Device:R
- removed R4: 500, Resistor_SMD:R_0603_1608Metric_Pad1.05x0.95mm_HandSolder, symbol Device:R
- removed U1: LM2576SX-3.3, Package_TO_SOT_SMD:TO-263-6, symbol MRDT_Devices:LM2576D2TR4
- removed U2: LM2576SX-5.0, Package_TO_SOT_SMD:TO-263-6, symbol MRDT_Devices:LM2576D2TR4
- added U1, U2: OKI, symbol MRDT_Devices:OKI
- C1, C2: value 100uF -> 10uF
- C3, C4: value 1000uF -> 10uF
Connections:
- net +12V: now also U1.1 (Vi)
- net +12VA: now also C3.2, U2.1 (Vi); no longer C2.2
- net +3V3: now also C2.2, U1.3 (Vo); no longer C3.2
- net +5V: now also U2.3 (Vo)
- net GND: now also U1.2 (GND), U2.2 (GND)

Commit message: layout 10
Parts:
- U1, U2: footprint (none) -> MRDT_Devices:OKI_Horizontal
Changed lines of the file:
@@
 EESchema Schematic File Version 4
+LIBS:gimble_board-cache
 EELAYER 30 0
 EELAYER END
@@
 F 0 "U1" H 5300 1400 60  0001 C CNN
 F 1 "OKI" H 5450 1731 60  0000 C CNN
-F 2 "" H 5050 1350 60  0001 C CNN
+F 2 "MRDT_Devices:OKI_Horizontal" H 5050 1350 60  0001 C CNN
 F 3 "" H 5050 1350 60  0001 C CNN
 	1    5250 1450
@@
 F 0 "U2" H 7600 1500 60  0001 C CNN
 F 1 "OKI" H 7750 1831 60  0000 C CNN
-F 2 "" H 7350 1450 60  0001 C CNN
+F 2 "MRDT_Devices:OKI_Horizontal" H 7350 1450 60  0001 C CNN
 F 3 "" H 7350 1450 60  0001 C CNN
 	1    7550 1550

Commit message: layout 11
Parts:
- removed D3, D4: LED, LED_SMD:LED_0603_1608Metric_Pad1.05x0.95mm_HandSolder, symbol Device:LED
- removed R1, R2: 1k, Resistor_SMD:R_0603_1608Metric_Pad1.05x0.95mm_HandSolder, symbol Device:R
- D1, D2: footprint LED_SMD:LED_0603_1608Metric_Pad1.05x0.95mm_HandSolder -> Diode_SMD:D_0201_0603Metric_Pad0.64x0.40mm_HandSolder
Connections:
- net +12V renamed +12L
Other:
- note removed: "Green"
- moved on the sheet: D2, J2
Changed lines of the file:
@@
 EESchema Schematic File Version 4
-LIBS:gimble_board-cache
 EELAYER 30 0
 EELAYER END
@@
 F 0 "D1" V 1900 1600 50  0000 L CNN
 F 1 "D_Zener" V 2000 1400 50  0000 L CNN
-F 2 "LED_SMD:LED_0603_1608Metric_Pad1.05x0.95mm_HandSolder" H 1950 1800 50  0001 C CNN
+F 2 "Diode_SMD:D_0201_0603Metric_Pad0.64x0.40mm_HandSolder" H 1950 1800 50  0001 C CNN
 F 3 "~" H 1950 1800 50  0001 C CNN
 	1    1950 1800
@@
 $EndComp
 $Comp
-L power:+12V #PWR03
-U 1 1 5F7F20BE
-P 2250 1350
-F 0 "#PWR03" H 2250 1200 50  0001 C CNN
-F 1 "+12V" H 2265 1523 50  0000 C CNN
-F 2 "" H 2250 1350 50  0001 C CNN
-F 3 "" H 2250 1350 50  0001 C CNN
-	1    2250 1350
-	1    0    0    -1
-$EndComp
-$Comp
-L Device:LED D3
-U 1 1 5F7F3188
-P 2550 1500
-F 0 "D3" H 2550 1300 50  0000 C CNN
-F 1 "LED" H 2550 1400 50  0000 C CNN
-F 2 "LED_SMD:LED_0603_1608Metric_Pad1.05x0.95mm_HandSolder" H 2550 1500 50  0001 C CNN
-F 3 "~" H 2550 1500 50  0001 C CNN
-	1    2550 1500
-	-1   0    0    1
-$EndComp
-$Comp
-L Device:R R1
-U 1 1 5F7F43C6
-P 3000 1500
-F 0 "R1" V 2793 1500 50  0000 C CNN
-F 1 "1k" V 2884 1500 50  0000 C CNN
-F 2 "Resistor_SMD:R_0603_1608Metric_Pad1.05x0.95mm_HandSolder" V 2930 1500 50  0001 C CNN
-F 3 "~" H 3000 1500 50  0001 C CNN
-	1    3000 1500
-	0    1    1    0
-$EndComp
-$Comp
-L power:GND #PWR05
-U 1 1 5F7F5224
-P 3300 1650
-F 0 "#PWR05" H 3300 1400 50  0001 C CNN
-F 1 "GND" H 3305 1477 50  0000 C CNN
-F 2 "" H 3300 1650 50  0001 C CNN
-F 3 "" H 3300 1650 50  0001 C CNN
-	1    3300 1650
-	1    0    0    -1
-$EndComp
-Text Notes 2500 1650 0    39   ~ 0
-Green
-$Comp
-L power:+12V #PWR07
-U 1 1 5F7F8ABA
-P 4900 1200
-F 0 "#PWR07" H 4900 1050 50  0001 C CNN
-F 1 "+12V" H 4915 1373 50  0000 C CNN
-F 2 "" H 4900 1200 50  0001 C CNN
-F 3 "" H 4900 1200 50  0001 C CNN
-	1    4900 1200
-	1    0    0    -1
-$EndComp
-$Comp
-L power:GND #PWR09
+L power:GND #PWR07
 U 1 1 5F80F9CA
 P 6150 2100
-F 0 "#PWR09" H 6150 1850 50  0001 C CNN
+F 0 "#PWR07" H 6150 1850 50  0001 C CNN
 F 1 "GND" H 6155 1927 50  0000 C CNN
 F 2 "" H 6150 2100 50  0001 C CNN
@@
 3.3v Converter
 $Comp
-L power:+5V #PWR011
+L power:+5V #PWR09
 U 1 1 5F98E7A2
 P 8300 1300
-F 0 "#PWR011" H 8300 1150 50  0001 C CNN
+F 0 "#PWR09" H 8300 1150 50  0001 C CNN
 F 1 "+5V" H 8315 1473 50  0000 C CNN
 F 2 "" H 8300 1300 50  0001 C CNN
@@
 Wire Wire Line
 	2250 1500 2250 1350
-Wire Wire Line
-	2250 1500 2400 1500
-Connection ~ 2250 1500
-Wire Wire Line
-	2700 1500 2850 1500
-Wire Wire Line
-	3150 1500 3300 1500
-Wire Wire Line
-	3300 1500 3300 1650
-Text GLabel 1800 3200 0    39   Input ~ 0
+Text GLabel 1800 2700 0    39   Input ~ 0
 Power_Input_Act
 $Comp
 L Device:D_Zener D2
 U 1 1 5FB1E563
-P 1950 3500
-F 0 "D2" V 1900 3300 50  0000 L CNN
-F 1 "D_Zener" V 2000 3100 50  0000 L CNN
-F 2 "LED_SMD:LED_0603_1608Metric_Pad1.05x0.95mm_HandSolder" H 1950 3500 50  0001 C CNN
-F 3 "~" H 1950 3500 50  0001 C CNN
-	1    1950 3500
+P 1950 3000
+F 0 "D2" V 1900 2800 50  0000 L CNN
+F 1 "D_Zener" V 2000 2600 50  0000 L CNN
+F 2 "Diode_SMD:D_0201_0603Metric_Pad0.64x0.40mm_HandSolder" H 1950 3000 50  0001 C CNN
+F 3 "~" H 1950 3000 50  0001 C CNN
+	1    1950 3000
 	0    1    1    0
 $EndComp
@@
 L power:GND #PWR02
 U 1 1 5FB1E569
-P 1950 3800
-F 0 "#PWR02" H 1950 3550 50  0001 C CNN
-F 1 "GND" H 1955 3627 50  0000 C CNN
-F 2 "" H 1950 3800 50  0001 C CNN
-F 3 "" H 1950 3800 50  0001 C CNN
-	1    1950 3800
-	1    0    0    -1
-$EndComp
-$Comp
-L Device:LED D4
-U 1 1 5FB1E575
-P 2550 3200
-F 0 "D4" H 2550 3000 50  0000 C CNN
-F 1 "LED" H 2550 3100 50  0000 C CNN
-F 2 "LED_SMD:LED_0603_1608Metric_Pad1.05x0.95mm_HandSolder" H 2550 3200 50  0001 C CNN
-F 3 "~" H 2550 3200 50  0001 C CNN
-	1    2550 3200
-	-1   0    0    1
-$EndComp
-$Comp
-L Device:R R2
-U 1 1 5FB1E57B
-P 3000 3200
-F 0 "R2" V 2793 3200 50  0000 C CNN
-F 1 "1k" V 2884 3200 50  0000 C CNN
-F 2 "Resistor_SMD:R_0603_1608Metric_Pad1.05x0.95mm_HandSolder" V 2930 3200 50  0001 C CNN
-F 3 "~" H 3000 3200 50  0001 C CNN
-	1    3000 3200
-	0    1    1    0
-$EndComp
-$Comp
-L power:GND #PWR06
-U 1 1 5FB1E581
-P 3300 3350
-F 0 "#PWR06" H 3300 3100 50  0001 C CNN
-F 1 "GND" H 3305 3177 50  0000 C CNN
-F 2 "" H 3300 3350 50  0001 C CNN
-F 3 "" H 3300 3350 50  0001 C CNN
-	1    3300 3350
-	1    0    0    -1
-$EndComp
-Text Notes 2500 3350 0    39   ~ 0
-Green
-Wire Wire Line
-	1800 3200 1950 3200
-Wire Wire Line
-	1950 3200 1950 3350
-Wire Wire Line
-	1950 3650 1950 3800
-Connection ~ 1950 3200
-Wire Wire Line
-	2250 3200 2250 3050
-Wire Wire Line
-	2250 3200 2400 3200
-Connection ~ 2250 3200
-Wire Wire Line
-	2700 3200 2850 3200
-Wire Wire Line
-	3150 3200 3300 3200
-Wire Wire Line
-	3300 3200 3300 3350
+P 1950 3300
+F 0 "#PWR02" H 1950 3050 50  0001 C CNN
+F 1 "GND" H 1955 3127 50  0000 C CNN
+F 2 "" H 1950 3300 50  0001 C CNN
+F 3 "" H 1950 3300 50  0001 C CNN
+	1    1950 3300
+	1    0    0    -1
+$EndComp
+Wire Wire Line
+	1800 2700 1950 2700
+Wire Wire Line
+	1950 2700 1950 2850
+Wire Wire Line
+	1950 3150 1950 3300
+Connection ~ 1950 2700
+Wire Wire Line
+	2250 2700 2250 2550
 $Comp
 L power:+12VA #PWR04
 U 1 1 5FB30BF8
-P 2250 3050
-F 0 "#PWR04" H 2250 2900 50  0001 C CNN
-F 1 "+12VA" H 2265 3223 50  0000 C CNN
-F 2 "" H 2250 3050 50  0001 C CNN
-F 3 "" H 2250 3050 50  0001 C CNN
-	1    2250 3050
-	1    0    0    -1
-$EndComp
-Wire Wire Line
-	2100 3200 2250 3200
-Wire Wire Line
-	1950 3200 2100 3200
-Connection ~ 2100 3200
-Wire Wire Line
-	2100 3200 2100 3350
+P 2250 2550
+F 0 "#PWR04" H 2250 2400 50  0001 C CNN
+F 1 "+12VA" H 2265 2723 50  0000 C CNN
+F 2 "" H 2250 2550 50  0001 C CNN
+F 3 "" H 2250 2550 50  0001 C CNN
+	1    2250 2550
+	1    0    0    -1
+$EndComp
+Wire Wire Line
+	2100 2700 2250 2700
+Wire Wire Line
+	1950 2700 2100 2700
+Connection ~ 2100 2700
+Wire Wire Line
+	2100 2700 2100 2850
 $Comp
 L MRDT_Connectors:Test_Point J2
 U 1 1 5FB1E588
-P 2100 3350
-F 0 "J2" H 2022 3389 60  0000 R CNN
-F 1 "Test_Point" H 2022 3495 60  0000 R CNN
-F 2 "TestPoint:TestPoint_Pad_2.0x2.0mm" H 2100 3300 60  0001 C CNN
-F 3 "" H 2100 3300 60  0001 C CNN
-	1    2100 3350
+P 2100 2850
+F 0 "J2" H 2022 2889 60  0000 R CNN
+F 1 "Test_Point" H 2022 2995 60  0000 R CNN
+F 2 "TestPoint:TestPoint_Pad_2.0x2.0mm" H 2100 2800 60  0001 C CNN
+F 3 "" H 2100 2800 60  0001 C CNN
+	1    2100 2850
 	-1   0    0    1
 $EndComp
@@
 U 1 1 5F8266E6
 P 2100 1650
-F 0 "J1" H 2022 1689 60  0000 R CNN
-F 1 "Test_Point" H 2022 1795 60  0000 R CNN
+F 0 "J1" H 2000 1850 60  0000 R CNN
+F 1 "Test_Point" H 2150 1950 60  0000 R CNN
 F 2 "TestPoint:TestPoint_Pad_2.0x2.0mm" H 2100 1600 60  0001 C CNN
 F 3 "" H 2100 1600 60  0001 C CNN
@@
 Connection ~ 6000 1950
 $Comp
-L power:+3.3V #PWR08
+L power:+3.3V #PWR06
 U 1 1 5FB6E12D
 P 6000 1200
-F 0 "#PWR08" H 6000 1050 50  0001 C CNN
+F 0 "#PWR06" H 6000 1050 50  0001 C CNN
 F 1 "+3.3V" H 6015 1373 50  0000 C CNN
 F 2 "" H 6000 1200 50  0001 C CNN
@@
 $EndComp
 $Comp
-L power:GND #PWR012
+L power:GND #PWR010
 U 1 1 5FB71B34
 P 8450 2200
-F 0 "#PWR012" H 8450 1950 50  0001 C CNN
+F 0 "#PWR010" H 8450 1950 50  0001 C CNN
 F 1 "GND" H 8455 2027 50  0000 C CNN
 F 2 "" H 8450 2200 50  0001 C CNN
@@
 5v Converter
 $Comp
-L power:+12VA #PWR010
+L power:+12VA #PWR08
 U 1 1 5FB8D1B3
 P 7200 1300
-F 0 "#PWR010" H 7200 1150 50  0001 C CNN
+F 0 "#PWR08" H 7200 1150 50  0001 C CNN
 F 1 "+12VA" H 7215 1473 50  0000 C CNN
 F 2 "" H 7200 1300 50  0001 C CNN
@@
 	1    0    0    -1
 $EndComp
+$Comp
+L power:+12L #PWR03
+U 1 1 5FB7DB5E
+P 2250 1350
+F 0 "#PWR03" H 2250 1200 50  0001 C CNN
+F 1 "+12L" H 2265 1523 50  0000 C CNN
+F 2 "" H 2250 1350 50  0001 C CNN
+F 3 "" H 2250 1350 50  0001 C CNN
+	1    2250 1350
+	1    0    0    -1
+$EndComp
+$Comp
+L power:+12L #PWR05
+U 1 1 5FB7E2F0
+P 4900 1200
+F 0 "#PWR05" H 4900 1050 50  0001 C CNN
+F 1 "+12L" H 4915 1373 50  0000 C CNN
+F 2 "" H 4900 1200 50  0001 C CNN
+F 3 "" H 4900 1200 50  0001 C CNN
+	1    4900 1200
+	1    0    0    -1
+$EndComp

Commit message: layout 16
Parts:
- added C5, C6: 10uF, Capacitor_SMD:C_0603_1608Metric_Pad1.05x0.95mm_HandSolder, symbol Device:C
- added U4: OKI, MRDT_Devices:OKI_Horizontal, symbol MRDT_Devices:OKI
Connections:
- net +12VA: now also C5.2, U4.1 (Vi)
- net +5V: now also C6.2, U4.3 (Vo)
- net GND: now also C5.1, C6.1, U4.2 (GND)
Changed lines of the file:
@@
+	1    0    0    -1
+$EndComp
+$Comp
+L power:+5V #PWR032
+U 1 1 5FB846E5
+P 8300 2700
+F 0 "#PWR032" H 8300 2550 50  0001 C CNN
+F 1 "+5V" H 8315 2873 50  0000 C CNN
+F 2 "" H 8300 2700 50  0001 C CNN
+F 3 "" H 8300 2700 50  0001 C CNN
+	1    8300 2700
+	1    0    0    -1
+$EndComp
+$Comp
+L power:GND #PWR033
+U 1 1 5FB846EB
+P 8450 3600
+F 0 "#PWR033" H 8450 3350 50  0001 C CNN
+F 1 "GND" H 8455 3427 50  0000 C CNN
+F 2 "" H 8450 3600 50  0001 C CNN
+F 3 "" H 8450 3600 50  0001 C CNN
+	1    8450 3600
+	1    0    0    -1
+$EndComp
+$Comp
+L MRDT_Devices:OKI U4
+U 1 1 5FB846F1
+P 7550 2950
+F 0 "U4" H 7600 2900 60  0001 C CNN
+F 1 "OKI" H 7750 3231 60  0000 C CNN
+F 2 "MRDT_Devices:OKI_Horizontal" H 7350 2850 60  0001 C CNN
+F 3 "" H 7350 2850 60  0001 C CNN
+	1    7550 2950
+	1    0    0    -1
+$EndComp
+Wire Wire Line
+	7200 2700 7200 2850
+Wire Wire Line
+	7200 2850 7350 2850
+$Comp
+L Device:C C5
+U 1 1 5FB846F9
+P 7200 3150
+F 0 "C5" V 6948 3150 50  0000 C CNN
+F 1 "10uF" V 7039 3150 50  0000 C CNN
+F 2 "Capacitor_SMD:C_0603_1608Metric_Pad1.05x0.95mm_HandSolder" H 7238 3000 50  0001 C CNN
+F 3 "~" H 7200 3150 50  0001 C CNN
+	1    7200 3150
+	-1   0    0    1
+$EndComp
+$Comp
+L Device:C C6
+U 1 1 5FB846FF
+P 8300 3150
+F 0 "C6" V 8048 3150 50  0000 C CNN
+F 1 "10uF" V 8139 3150 50  0000 C CNN
+F 2 "Capacitor_SMD:C_0603_1608Metric_Pad1.05x0.95mm_HandSolder" H 8338 3000 50  0001 C CNN
+F 3 "~" H 8300 3150 50  0001 C CNN
+	1    8300 3150
+	-1   0    0    1
+$EndComp
+Wire Wire Line
+	7200 3000 7200 2850
+Connection ~ 7200 2850
+Wire Wire Line
+	7200 3300 7200 3450
+Wire Wire Line
+	7200 3450 7750 3450
+Wire Wire Line
+	8300 3450 8300 3300
+Wire Wire Line
+	7750 3150 7750 3450
+Connection ~ 7750 3450
+Wire Wire Line
+	7750 3450 8300 3450
+Wire Wire Line
+	8300 3000 8300 2850
+Wire Wire Line
+	8300 2850 8150 2850
+Wire Wire Line
+	8300 2850 8300 2700
+Connection ~ 8300 2850
+Wire Wire Line
+	8300 3450 8450 3450
+Wire Wire Line
+	8450 3450 8450 3600
+Connection ~ 8300 3450
+$Comp
+L power:+12VA #PWR031
+U 1 1 5FB84714
+P 7200 2700
+F 0 "#PWR031" H 7200 2550 50  0001 C CNN
+F 1 "+12VA" H 7215 2873 50  0000 C CNN
+F 2 "" H 7200 2700 50  0001 C CNN
+F 3 "" H 7200 2700 50  0001 C CNN
+	1    7200 2700
 	1    0    0    -1
 $EndComp
