File: Hardware/gimble_board/GimbleBoard01.sch (KiCad schematic (older format))
At the start: 13 parts, among them J1 Test_Point, J2 Test_Point, U1 OKI, U2 OKI, U4 OKI

Commit message: layout 18
Parts:
- removed C5, C6: 10uF, Capacitor_SMD:C_0603_1608Metric_Pad1.05x0.95mm_HandSolder, symbol Device:C
Connections:
- wire segments 53 -> 45
Changed lines of the file:
@@
 L power:GND #PWR033
 U 1 1 5FB846EB
-P 8450 3600
-F 0 "#PWR033" H 8450 3350 50  0001 C CNN
-F 1 "GND" H 8455 3427 50  0000 C CNN
-F 2 "" H 8450 3600 50  0001 C CNN
-F 3 "" H 8450 3600 50  0001 C CNN
-	1    8450 3600
+P 7750 3300
+F 0 "#PWR033" H 7750 3050 50  0001 C CNN
+F 1 "GND" H 7755 3127 50  0000 C CNN
+F 2 "" H 7750 3300 50  0001 C CNN
+F 3 "" H 7750 3300 50  0001 C CNN
+	1    7750 3300
 	1    0    0    -1
 $EndComp
@@
 Wire Wire Line
 	7200 2850 7350 2850
-$Comp
-L Device:C C5
-U 1 1 5FB846F9
-P 7200 3150
-F 0 "C5" V 6948 3150 50  0000 C CNN
-F 1 "10uF" V 7039 3150 50  0000 C CNN
-F 2 "Capacitor_SMD:C_0603_1608Metric_Pad1.05x0.95mm_HandSolder" H 7238 3000 50  0001 C CNN
-F 3 "~" H 7200 3150 50  0001 C CNN
-	1    7200 3150
-	-1   0    0    1
-$EndComp
-$Comp
-L Device:C C6
-U 1 1 5FB846FF
-P 8300 3150
-F 0 "C6" V 8048 3150 50  0000 C CNN
-F 1 "10uF" V 8139 3150 50  0000 C CNN
-F 2 "Capacitor_SMD:C_0603_1608Metric_Pad1.05x0.95mm_HandSolder" H 8338 3000 50  0001 C CNN
-F 3 "~" H 8300 3150 50  0001 C CNN
-	1    8300 3150
-	-1   0    0    1
-$EndComp
-Wire Wire Line
-	7200 3000 7200 2850
-Connection ~ 7200 2850
-Wire Wire Line
-	7200 3300 7200 3450
-Wire Wire Line
-	7200 3450 7750 3450
-Wire Wire Line
-	8300 3450 8300 3300
-Wire Wire Line
-	7750 3150 7750 3450
-Connection ~ 7750 3450
-Wire Wire Line
-	7750 3450 8300 3450
-Wire Wire Line
-	8300 3000 8300 2850
 Wire Wire Line
 	8300 2850 8150 2850
 Wire Wire Line
 	8300 2850 8300 2700
-Connection ~ 8300 2850
-Wire Wire Line
-	8300 3450 8450 3450
-Wire Wire Line
-	8450 3450 8450 3600
-Connection ~ 8300 3450
 $Comp
 L power:+12VA #PWR031
@@
 	1    0    0    -1
 $EndComp
+Wire Wire Line
+	7750 3150 7750 3300
 $EndSCHEMATC
