File: GimbalBoard_Hardware/switches.sch (KiCad schematic (older format))
At the start: 0 parts

Commit message: swiches sheet
swithces subsheet with 3 toggle is done
Parts:
- added D? (x11): LED, symbol Device:LED
- added R? (x8): R, symbol Device:R
- added R? (x3): 330, symbol Device:R
- added SW? (x8): SW_Push, symbol Switch:SW_Push
- added SW?: SW_SP3T, symbol Switch:SW_SP3T
Connections:
- new net: D?.2 (A), R?.1 (x11)
- new net +3V3: SW?.1, SW?.1, SW?.1, SW?.1, SW?.1, SW?.1, SW?.1, SW?.1, SW?.3
- new net GND: D?.1 (K), D?.1 (K), D?.1 (K), D?.1 (K), D?.1 (K), D?.1 (K), D?.1 (K), D?.1 (K), D?.1 (K), D?.1 (K), D?.1 (K)
- new net Servo_1_SW: R?.2, SW?.2
- new net Servo_2_SW: R?.2, SW?.2
- new net Servo_3­_SW: R?.2, SW?.2
- new net Servo_4_SW: R?.2, SW?.2
- new net Servo_5_SW: R?.2, SW?.2
- new net Servo_6_SW: R?.2, SW?.2
- new net Servo_7_SW: R?.2, SW?.2
- new net Servo_8_SW: R?.2, SW?.2
- new net Servo_Digital_Control: R?.2, SW?.1
- new net Servo_Manual_Control_Left: R?.2, SW?.2
- new net Servo_Manual_Control_Right: R?.2, SW?.4
