File: GimbalBoard_Hardware/switches.sch (KiCad schematic (older format))
At the start: 31 parts, among them SW1 SW_Push, SW2 SW_Push, SW3 SW_Push, SW4 SW_Push, SW5 SW_Push, SW6 SW_Push, SW7 SW_Push, SW8 SW_Push, SW9 SW_SP3T

Commit message: Post PDR changes
Parts:
- removed D14: LED, symbol Device:LED
- removed R14: 43, symbol Device:R
- removed SW9: SW_SP3T, symbol Switch:SW_SP3T
- added SW9: SW_DPDT_x2, symbol Switch:SW_DPDT_x2
Connections:
- net 3.3VL: now also SW9.2 (B)
- net Servo_Manual_Control_Left: now also SW9.1 (A)
- net Servo_Manual_Control_Right: now also SW9.3 (C)
Changed lines of the file:
@@
 $Descr A4 11693 8268
 encoding utf-8
-Sheet 4 8
+Sheet 2 5
 Title ""
 Date ""
@@
 Wire Wire Line
 	3700 6850 3700 7000
-$Comp
-L Device:LED D14
-U 1 1 6161933E
-P 6600 1950
-F 0 "D14" H 6593 1695 50  0000 C CNN
-F 1 "LED" H 6593 1786 50  0000 C CNN
-F 2 "" H 6600 1950 50  0001 C CNN
-F 3 "~" H 6600 1950 50  0001 C CNN
-	1    6600 1950
-	-1   0    0    1
-$EndComp
-$Comp
-L Device:R R14
-U 1 1 6161A7C1
-P 6100 1950
-F 0 "R14" V 6000 1950 50  0000 C CNN
-F 1 "43" V 6100 1950 50  0000 C CNN
-F 2 "" V 6030 1950 50  0001 C CNN
-F 3 "~" H 6100 1950 50  0001 C CNN
-	1    6100 1950
-	0    1    1    0
-$EndComp
 Text HLabel 2650 1850 2    50   Output ~ 0
 Servo_1_SW
@@
 Text HLabel 2650 6450 2    50   Output ~ 0
 Servo_8_SW
-Text HLabel 6200 2200 2    50   Output ~ 0
-Servo_Digital_Control
-Wire Wire Line
-	4800 2050 4800 2300
-Wire Wire Line
-	4800 2300 5100 2300
-Wire Wire Line
-	5500 2200 5750 2200
-Wire Wire Line
-	5950 1950 5750 1950
-Connection ~ 5750 2200
-Wire Wire Line
-	5750 2200 6200 2200
-Wire Wire Line
-	6250 1950 6450 1950
-Wire Wire Line
-	5750 1950 5750 2200
-$Comp
-L Device:LED D15
-U 1 1 61657CB4
-P 6650 2500
-F 0 "D15" H 6643 2245 50  0000 C CNN
-F 1 "LED" H 6643 2336 50  0000 C CNN
-F 2 "" H 6650 2500 50  0001 C CNN
-F 3 "~" H 6650 2500 50  0001 C CNN
-	1    6650 2500
-	-1   0    0    1
-$EndComp
-$Comp
-L Device:LED D16
-U 1 1 61657CBA
-P 6650 3150
-F 0 "D16" H 6643 2895 50  0000 C CNN
-F 1 "LED" H 6643 2986 50  0000 C CNN
-F 2 "" H 6650 3150 50  0001 C CNN
-F 3 "~" H 6650 3150 50  0001 C CNN
-	1    6650 3150
-	-1   0    0    1
-$EndComp
-$Comp
-L Device:R R15
-U 1 1 61657CC0
-P 6150 2500
-F 0 "R15" V 6050 2500 50  0000 C CNN
-F 1 "43" V 6150 2500 50  0000 C CNN
-F 2 "" V 6080 2500 50  0001 C CNN
-F 3 "~" H 6150 2500 50  0001 C CNN
-	1    6150 2500
-	0    1    1    0
-$EndComp
-$Comp
-L Device:R R16
-U 1 1 61657CC6
-P 6150 3150
-F 0 "R16" V 6050 3150 50  0000 C CNN
-F 1 "43" V 6150 3150 50  0000 C CNN
-F 2 "" V 6080 3150 50  0001 C CNN
-F 3 "~" H 6150 3150 50  0001 C CNN
-	1    6150 3150
-	0    1    1    0
-$EndComp
-Text HLabel 6250 2750 2    50   Output ~ 0
-Servo_Manual_Control_Left
-Text HLabel 6250 3400 2    50   Output ~ 0
-Servo_Manual_Control_Right
-Wire Wire Line
-	6000 2500 5800 2500
-Connection ~ 5800 2750
-Wire Wire Line
-	5800 2750 6250 2750
-Wire Wire Line
-	6000 3150 5850 3150
-Wire Wire Line
-	6300 2500 6500 2500
-Wire Wire Line
-	6300 3150 6500 3150
-Wire Wire Line
-	7550 3150 6800 3150
-Wire Wire Line
-	5800 2500 5800 2750
-$Comp
-L Switch:SW_SP3T SW9
-U 1 1 6168F99A
-P 5300 2300
-F 0 "SW9" H 5300 2583 50  0000 C CNN
-F 1 "SW_SP3T" H 5300 2492 50  0000 C CNN
-F 2 "" H 4675 2475 50  0001 C CNN
-F 3 "~" H 4675 2475 50  0001 C CNN
-	1    5300 2300
-	1    0    0    -1
-$EndComp
-Wire Wire Line
-	5550 3400 5850 3400
-Wire Wire Line
-	5850 3150 5850 3400
-Connection ~ 5850 3400
-Wire Wire Line
-	5850 3400 6250 3400
-Wire Wire Line
-	5500 2300 5650 2300
-Wire Wire Line
-	5650 2300 5650 2750
-Wire Wire Line
-	5650 2750 5800 2750
-Wire Wire Line
-	5500 2400 5550 2400
-Wire Wire Line
-	5550 2400 5550 3400
-Connection ~ 7550 3150
-Wire Wire Line
-	7550 3150 7550 3700
-Wire Wire Line
-	6750 1950 7550 1950
-Wire Wire Line
-	7550 1950 7550 2500
-Wire Wire Line
-	6800 2500 7550 2500
-Connection ~ 7550 2500
-Wire Wire Line
-	7550 2500 7550 3150
 Text HLabel 1600 1900 1    50   Input ~ 0
 3.3VL
 Text HLabel 3700 7000 3    50   Input ~ 0
 GND
-Text HLabel 4800 2050 1    50   Input ~ 0
-3.3VL
-Text HLabel 7550 3700 3    50   Input ~ 0
-GND
-Text Notes 5750 1300 0    79   ~ 0
+Text Notes 5600 1350 0    79   ~ 0
 Digital/Manual Switch
 Text Notes 2050 1250 0    79   ~ 0
 Manual Servo Switches
+$Comp
+L Switch:SW_DPDT_x2 SW9
+U 1 1 617F83FD
+P 5000 2200
+F 0 "SW9" H 5000 2485 50  0000 C CNN
+F 1 "SW_DPDT_x2" H 5000 2394 50  0000 C CNN
+F 2 "" H 5000 2200 50  0001 C CNN
+F 3 "~" H 5000 2200 50  0001 C CNN
+	1    5000 2200
+	1    0    0    -1
+$EndComp
+Wire Wire Line
+	4500 1950 4500 2200
+Wire Wire Line
+	4500 2200 4800 2200
+$Comp
+L Device:LED D15
+U 1 1 617FDA6F
+P 6350 2300
+F 0 "D15" H 6343 2045 50  0000 C CNN
+F 1 "LED" H 6343 2136 50  0000 C CNN
+F 2 "" H 6350 2300 50  0001 C CNN
+F 3 "~" H 6350 2300 50  0001 C CNN
+	1    6350 2300
+	-1   0    0    1
+$EndComp
+$Comp
+L Device:LED D16
+U 1 1 617FDA75
+P 6350 3050
+F 0 "D16" H 6343 2795 50  0000 C CNN
+F 1 "LED" H 6343 2886 50  0000 C CNN
+F 2 "" H 6350 3050 50  0001 C CNN
+F 3 "~" H 6350 3050 50  0001 C CNN
+	1    6350 3050
+	-1   0    0    1
+$EndComp
+$Comp
+L Device:R R15
+U 1 1 617FDA7B
+P 5850 2300
+F 0 "R15" V 5750 2300 50  0000 C CNN
+F 1 "43" V 5850 2300 50  0000 C CNN
+F 2 "" V 5780 2300 50  0001 C CNN
+F 3 "~" H 5850 2300 50  0001 C CNN
+	1    5850 2300
+	0    1    1    0
+$EndComp
+$Comp
+L Device:R R16
+U 1 1 617FDA81
+P 5850 3050
+F 0 "R16" V 5750 3050 50  0000 C CNN
+F 1 "43" V 5850 3050 50  0000 C CNN
+F 2 "" V 5780 3050 50  0001 C CNN
+F 3 "~" H 5850 3050 50  0001 C CNN
+	1    5850 3050
+	0    1    1    0
+$EndComp
+Text HLabel 5950 2550 2    50   Output ~ 0
+Servo_Manual_Control_Left
+Text HLabel 5950 3300 2    50   Output ~ 0
+Servo_Manual_Control_Right
+Wire Wire Line
+	5700 2300 5500 2300
+Connection ~ 5500 2550
+Wire Wire Line
+	5500 2550 5950 2550
+Wire Wire Line
+	5700 3050 5550 3050
+Wire Wire Line
+	6000 2300 6200 2300
+Wire Wire Line
+	6000 3050 6200 3050
+Wire Wire Line
+	7250 3050 6500 3050
+Wire Wire Line
+	5500 2300 5500 2550
+Wire Wire Line
+	5250 3300 5550 3300
+Wire Wire Line
+	5550 3050 5550 3300
+Connection ~ 5550 3300
+Wire Wire Line
+	5550 3300 5950 3300
+Wire Wire Line
+	5200 2100 5350 2100
+Wire Wire Line
+	5350 2100 5350 2550
+Wire Wire Line
+	5350 2550 5500 2550
+Wire Wire Line
+	5200 2300 5250 2300
+Wire Wire Line
+	5250 2300 5250 3300
+Wire Wire Line
+	7250 3050 7250 3600
+Wire Wire Line
+	6500 2300 7250 2300
+Text HLabel 4500 1950 1    50   Input ~ 0
+3.3VL
+Text HLabel 7250 3600 3    50   Input ~ 0
+GND
+Wire Wire Line
+	7250 2300 7250 3050
+Connection ~ 7250 3050
 $EndSCHEMATC

Commit message: Added more footprints
I added more footprints. Not done yet. I'd like to come back when when I can verify with max about some of the other components.
Parts:
- D10, D11, D12, D13, D15, D16, D6, D7, D8, D9: footprint (none) -> LED_SMD:LED_0603_1608Metric_Pad1.05x0.95mm_HandSolder
- R10, R11, R12, R13, R15, R16, R6, R7, R8, R9: footprint (none) -> Resistor_SMD:R_0603_1608Metric_Pad0.98x0.95mm_HandSolder
Changed lines of the file:
@@
 F 0 "R6" V 2650 2250 50  0000 C CNN
 F 1 "43" V 2750 2250 50  0000 C CNN
-F 2 "" V 2680 2250 50  0001 C CNN
+F 2 "Resistor_SMD:R_0603_1608Metric_Pad0.98x0.95mm_HandSolder" V 2680 2250 50  0001 C CNN
 F 3 "~" H 2750 2250 50  0001 C CNN
 	1    2750 2250
@@
 F 0 "D6" H 3243 1995 50  0000 C CNN
 F 1 "LED" H 3243 2086 50  0000 C CNN
-F 2 "" H 3250 2250 50  0001 C CNN
+F 2 "LED_SMD:LED_0603_1608Metric_Pad1.05x0.95mm_HandSolder" H 3250 2250 50  0001 C CNN
 F 3 "~" H 3250 2250 50  0001 C CNN
 	1    3250 2250
@@
 F 0 "R7" V 2650 2950 50  0000 C CNN
 F 1 "43" V 2750 2950 50  0000 C CNN
-F 2 "" V 2680 2950 50  0001 C CNN
+F 2 "Resistor_SMD:R_0603_1608Metric_Pad0.98x0.95mm_HandSolder" V 2680 2950 50  0001 C CNN
 F 3 "~" H 2750 2950 50  0001 C CNN
 	1    2750 2950
@@
 F 0 "D7" H 3243 2695 50  0000 C CNN
 F 1 "LED" H 3243 2786 50  0000 C CNN
-F 2 "" H 3250 2950 50  0001 C CNN
+F 2 "LED_SMD:LED_0603_1608Metric_Pad1.05x0.95mm_HandSolder" H 3250 2950 50  0001 C CNN
 F 3 "~" H 3250 2950 50  0001 C CNN
 	1    3250 2950
@@
 F 0 "R8" V 2650 3600 50  0000 C CNN
 F 1 "43" V 2750 3600 50  0000 C CNN
-F 2 "" V 2680 3600 50  0001 C CNN
+F 2 "Resistor_SMD:R_0603_1608Metric_Pad0.98x0.95mm_HandSolder" V 2680 3600 50  0001 C CNN
 F 3 "~" H 2750 3600 50  0001 C CNN
 	1    2750 3600
@@
 F 0 "D8" H 3243 3345 50  0000 C CNN
 F 1 "LED" H 3243 3436 50  0000 C CNN
-F 2 "" H 3250 3600 50  0001 C CNN
+F 2 "LED_SMD:LED_0603_1608Metric_Pad1.05x0.95mm_HandSolder" H 3250 3600 50  0001 C CNN
 F 3 "~" H 3250 3600 50  0001 C CNN
 	1    3250 3600
@@
 F 0 "R9" V 2650 4250 50  0000 C CNN
 F 1 "43" V 2750 4250 50  0000 C CNN
-F 2 "" V 2680 4250 50  0001 C CNN
+F 2 "Resistor_SMD:R_0603_1608Metric_Pad0.98x0.95mm_HandSolder" V 2680 4250 50  0001 C CNN
 F 3 "~" H 2750 4250 50  0001 C CNN
 	1    2750 4250
@@
 F 0 "D9" H 3243 3995 50  0000 C CNN
 F 1 "LED" H 3243 4086 50  0000 C CNN
-F 2 "" H 3250 4250 50  0001 C CNN
+F 2 "LED_SMD:LED_0603_1608Metric_Pad1.05x0.95mm_HandSolder" H 3250 4250 50  0001 C CNN
 F 3 "~" H 3250 4250 50  0001 C CNN
 	1    3250 4250
@@
 F 0 "R10" V 2650 4900 50  0000 C CNN
 F 1 "43" V 2750 4900 50  0000 C CNN
-F 2 "" V 2680 4900 50  0001 C CNN
+F 2 "Resistor_SMD:R_0603_1608Metric_Pad0.98x0.95mm_HandSolder" V 2680 4900 50  0001 C CNN
 F 3 "~" H 2750 4900 50  0001 C CNN
 	1    2750 4900
@@
 F 0 "D10" H 3243 4645 50  0000 C CNN
 F 1 "LED" H 3243 4736 50  0000 C CNN
-F 2 "" H 3250 4900 50  0001 C CNN
+F 2 "LED_SMD:LED_0603_1608Metric_Pad1.05x0.95mm_HandSolder" H 3250 4900 50  0001 C CNN
 F 3 "~" H 3250 4900 50  0001 C CNN
 	1    3250 4900
@@
 F 0 "R11" V 2650 5550 50  0000 C CNN
 F 1 "43" V 2750 5550 50  0000 C CNN
-F 2 "" V 2680 5550 50  0001 C CNN
+F 2 "Resistor_SMD:R_0603_1608Metric_Pad0.98x0.95mm_HandSolder" V 2680 5550 50  0001 C CNN
 F 3 "~" H 2750 5550 50  0001 C CNN
 	1    2750 5550
@@
 F 0 "D11" H 3243 5295 50  0000 C CNN
 F 1 "LED" H 3243 5386 50  0000 C CNN
-F 2 "" H 3250 5550 50  0001 C CNN
+F 2 "LED_SMD:LED_0603_1608Metric_Pad1.05x0.95mm_HandSolder" H 3250 5550 50  0001 C CNN
 F 3 "~" H 3250 5550 50  0001 C CNN
 	1    3250 5550
@@
 F 0 "R12" V 2650 6200 50  0000 C CNN
 F 1 "43" V 2750 6200 50  0000 C CNN
-F 2 "" V 2680 6200 50  0001 C CNN
+F 2 "Resistor_SMD:R_0603_1608Metric_Pad0.98x0.95mm_HandSolder" V 2680 6200 50  0001 C CNN
 F 3 "~" H 2750 6200 50  0001 C CNN
 	1    2750 6200
@@
 F 0 "D12" H 3243 5945 50  0000 C CNN
 F 1 "LED" H 3243 6036 50  0000 C CNN
-F 2 "" H 3250 6200 50  0001 C CNN
+F 2 "LED_SMD:LED_0603_1608Metric_Pad1.05x0.95mm_HandSolder" H 3250 6200 50  0001 C CNN
 F 3 "~" H 3250 6200 50  0001 C CNN
 	1    3250 6200
@@
 F 0 "R13" V 2650 6850 50  0000 C CNN
 F 1 "43" V 2750 6850 50  0000 C CNN
-F 2 "" V 2680 6850 50  0001 C CNN
+F 2 "Resistor_SMD:R_0603_1608Metric_Pad0.98x0.95mm_HandSolder" V 2680 6850 50  0001 C CNN
 F 3 "~" H 2750 6850 50  0001 C CNN
 	1    2750 6850
@@
 F 0 "D13" H 3243 6595 50  0000 C CNN
 F 1 "LED" H 3243 6686 50  0000 C CNN
-F 2 "" H 3250 6850 50  0001 C CNN
+F 2 "LED_SMD:LED_0603_1608Metric_Pad1.05x0.95mm_HandSolder" H 3250 6850 50  0001 C CNN
 F 3 "~" H 3250 6850 50  0001 C CNN
 	1    3250 6850
@@
 F 0 "D15" H 6343 2045 50  0000 C CNN
 F 1 "LED" H 6343 2136 50  0000 C CNN
-F 2 "" H 6350 2300 50  0001 C CNN
+F 2 "LED_SMD:LED_0603_1608Metric_Pad1.05x0.95mm_HandSolder" H 6350 2300 50  0001 C CNN
 F 3 "~" H 6350 2300 50  0001 C CNN
 	1    6350 2300
@@
 F 0 "D16" H 6343 2795 50  0000 C CNN
 F 1 "LED" H 6343 2886 50  0000 C CNN
-F 2 "" H 6350 3050 50  0001 C CNN
+F 2 "LED_SMD:LED_0603_1608Metric_Pad1.05x0.95mm_HandSolder" H 6350 3050 50  0001 C CNN
 F 3 "~" H 6350 3050 50  0001 C CNN
 	1    6350 3050
@@
 F 0 "R15" V 5750 2300 50  0000 C CNN
 F 1 "43" V 5850 2300 50  0000 C CNN
-F 2 "" V 5780 2300 50  0001 C CNN
+F 2 "Resistor_SMD:R_0603_1608Metric_Pad0.98x0.95mm_HandSolder" V 5780 2300 50  0001 C CNN
 F 3 "~" H 5850 2300 50  0001 C CNN
 	1    5850 2300
@@
 F 0 "R16" V 5750 3050 50  0000 C CNN
 F 1 "43" V 5850 3050 50  0000 C CNN
-F 2 "" V 5780 3050 50  0001 C CNN
+F 2 "Resistor_SMD:R_0603_1608Metric_Pad0.98x0.95mm_HandSolder" V 5780 3050 50  0001 C CNN
 F 3 "~" H 5850 3050 50  0001 C CNN
 	1    5850 3050

Commit message: Footprints finished
the footprints are finished. the RJ45 connector has been added for eithernet.
the net is in the layout thing but I haven't moved anything yet
Parts:
- SW1, SW2, SW3, SW4, SW5, SW6, SW7, SW8: footprint (none) -> Button_Switch_SMD:SW_SPST_EVPBF
- SW9: footprint (none) -> MRDT_Switches:2P2T_Switch_GrayHill_Series76
Changed lines of the file:
@@
 F 0 "SW1" H 2100 2535 50  0000 C CNN
 F 1 "SW_Push" H 2100 2444 50  0000 C CNN
-F 2 "" H 2100 2450 50  0001 C CNN
+F 2 "Button_Switch_SMD:SW_SPST_EVPBF" H 2100 2450 50  0001 C CNN
 F 3 "~" H 2100 2450 50  0001 C CNN
 	1    2100 2250
@@
 F 0 "SW2" H 2100 3235 50  0000 C CNN
 F 1 "SW_Push" H 2100 3144 50  0000 C CNN
-F 2 "" H 2100 3150 50  0001 C CNN
+F 2 "Button_Switch_SMD:SW_SPST_EVPBF" H 2100 3150 50  0001 C CNN
 F 3 "~" H 2100 3150 50  0001 C CNN
 	1    2100 2950
@@
 F 0 "SW3" H 2100 3885 50  0000 C CNN
 F 1 "SW_Push" H 2100 3794 50  0000 C CNN
-F 2 "" H 2100 3800 50  0001 C CNN
+F 2 "Button_Switch_SMD:SW_SPST_EVPBF" H 2100 3800 50  0001 C CNN
 F 3 "~" H 2100 3800 50  0001 C CNN
 	1    2100 3600
@@
 F 0 "SW4" H 2100 4535 50  0000 C CNN
 F 1 "SW_Push" H 2100 4444 50  0000 C CNN
-F 2 "" H 2100 4450 50  0001 C CNN
+F 2 "Button_Switch_SMD:SW_SPST_EVPBF" H 2100 4450 50  0001 C CNN
 F 3 "~" H 2100 4450 50  0001 C CNN
 	1    2100 4250
@@
 F 0 "SW5" H 2100 5185 50  0000 C CNN
 F 1 "SW_Push" H 2100 5094 50  0000 C CNN
-F 2 "" H 2100 5100 50  0001 C CNN
+F 2 "Button_Switch_SMD:SW_SPST_EVPBF" H 2100 5100 50  0001 C CNN
 F 3 "~" H 2100 5100 50  0001 C CNN
 	1    2100 4900
@@
 F 0 "SW6" H 2100 5835 50  0000 C CNN
 F 1 "SW_Push" H 2100 5744 50  0000 C CNN
-F 2 "" H 2100 5750 50  0001 C CNN
+F 2 "Button_Switch_SMD:SW_SPST_EVPBF" H 2100 5750 50  0001 C CNN
 F 3 "~" H 2100 5750 50  0001 C CNN
 	1    2100 5550
@@
 F 0 "SW7" H 2100 6485 50  0000 C CNN
 F 1 "SW_Push" H 2100 6394 50  0000 C CNN
-F 2 "" H 2100 6400 50  0001 C CNN
+F 2 "Button_Switch_SMD:SW_SPST_EVPBF" H 2100 6400 50  0001 C CNN
 F 3 "~" H 2100 6400 50  0001 C CNN
 	1    2100 6200
@@
 F 0 "SW8" H 2100 7135 50  0000 C CNN
 F 1 "SW_Push" H 2100 7044 50  0000 C CNN
-F 2 "" H 2100 7050 50  0001 C CNN
+F 2 "Button_Switch_SMD:SW_SPST_EVPBF" H 2100 7050 50  0001 C CNN
 F 3 "~" H 2100 7050 50  0001 C CNN
 	1    2100 6850
@@
 F 0 "SW9" H 5000 2485 50  0000 C CNN
 F 1 "SW_DPDT_x2" H 5000 2394 50  0000 C CNN
-F 2 "" H 5000 2200 50  0001 C CNN
+F 2 "MRDT_Switches:2P2T_Switch_GrayHill_Series76" H 5000 2200 50  0001 C CNN
 F 3 "~" H 5000 2200 50  0001 C CNN
 	1    5000 2200
