File: GimbalBoard_Hardware/switches.sch (KiCad schematic (older format))
At the start: 29 parts, among them SW1 SW_Push, SW2 SW_Push, SW3 SW_Push, SW4 SW_Push, SW5 SW_Push, SW6 SW_Push, SW7 SW_Push, SW8 SW_Push, SW9 SW_DPDT_x2

Commit message: after review
some changes needed but yeah
Parts:
- removed SW9: SW_DPDT_x2, MRDT_Switches:2P2T_Switch_GrayHill_Series76, symbol Switch:SW_DPDT_x2
- added SW9: 3P1T, MRDT_Switches:3P1T_Switch, symbol MRDT_Switches:3P1T
Connections:
- net 3.3VL: now also SW9.1, SW9.3, SW9.5
- net Servo_Manual_Control_Left: now also SW9.6
- net Servo_Manual_Control_Right: now also SW9.2
- no-connect marks 0 -> 1
Changed lines of the file:
@@
 Text Notes 2050 1250 0    79   ~ 0
 Manual Servo Switches
-$Comp
-L Switch:SW_DPDT_x2 SW9
-U 1 1 617F83FD
-P 5000 2200
-F 0 "SW9" H 5000 2485 50  0000 C CNN
-F 1 "SW_DPDT_x2" H 5000 2394 50  0000 C CNN
-F 2 "MRDT_Switches:2P2T_Switch_GrayHill_Series76" H 5000 2200 50  0001 C CNN
-F 3 "~" H 5000 2200 50  0001 C CNN
-	1    5000 2200
-	1    0    0    -1
-$EndComp
 Wire Wire Line
-	4500 1950 4500 2200
-Wire Wire Line
-	4500 2200 4800 2200
+	4200 1850 4200 2100
 $Comp
 L Device:LED D15
@@
 	5550 3300 5950 3300
 Wire Wire Line
-	5200 2100 5350 2100
-Wire Wire Line
-	5350 2100 5350 2550
-Wire Wire Line
 	5350 2550 5500 2550
-Wire Wire Line
-	5200 2300 5250 2300
 Wire Wire Line
 	5250 2300 5250 3300
@@
 Wire Wire Line
 	6500 2300 7250 2300
-Text HLabel 4500 1950 1    50   Input ~ 0
+Text HLabel 4200 1850 1    50   Input ~ 0
 3.3VL
 Text HLabel 7250 3600 3    50   Input ~ 0
@@
 	7250 2300 7250 3050
 Connection ~ 7250 3050
+Wire Wire Line
+	5200 2300 5250 2300
+Wire Wire Line
+	4200 2100 4400 2100
+$Comp
+L MRDT_Switches:3P1T SW9
+U 1 1 61A05A6E
+P 4700 2400
+F 0 "SW9" H 4850 3187 60  0000 C CNN
+F 1 "3P1T" H 4850 3081 60  0000 C CNN
+F 2 "MRDT_Switches:3P1T_Switch" H 4450 2450 60  0001 C CNN
+F 3 "" H 4450 2450 60  0001 C CNN
+	1    4700 2400
+	1    0    0    -1
+$EndComp
+Wire Wire Line
+	5350 1900 5200 1900
+Wire Wire Line
+	5350 1900 5350 2550
+Wire Wire Line
+	4500 1900 4400 1900
+Wire Wire Line
+	4400 1900 4400 2100
+Connection ~ 4400 2100
+Wire Wire Line
+	4400 2100 4500 2100
+Wire Wire Line
+	4400 2100 4400 2300
+Wire Wire Line
+	4400 2300 4500 2300
+NoConn ~ 5200 2100
 $EndSCHEMATC

Commit message: ethernet fixed.
the ethernet is fixed. as well as the switch footprint association issue.
I'm not certain that the current footprint being used matches an actual switch. also this edit does not have the 3x2 microfit connectors
Connections:
- net 3.3VL: no longer SW9.3
- no-connect marks 1 -> 2
Changed lines of the file:
@@
 Connection ~ 4400 2100
-Wire Wire Line
-	4400 2100 4500 2100
 Wire Wire Line
 	4400 2100 4400 2300
@@
 	4400 2300 4500 2300
 NoConn ~ 5200 2100
+NoConn ~ 4500 2100
 $EndSCHEMATC

Commit message: the correct switch, and some decals
some decals and the correct switch
Parts:
- removed SW9: 3P1T, MRDT_Switches:3P1T_Switch, symbol MRDT_Switches:3P1T
- added SW9: SW_DPDT_x2, Button_Switch_THT:SW_Slide_1P2T_CK_OS102011MS2Q, symbol Switch:SW_DPDT_x2
Connections:
- net 3.3VL: now also SW9.2 (B)
- net Servo_Manual_Control_Left: now also SW9.1 (A)
- net Servo_Manual_Control_Right: now also SW9.3 (C)
- no-connect marks 2 -> 0
Changed lines of the file:
@@
 Manual Servo Switches
 Wire Wire Line
-	4200 1850 4200 2100
+	4200 1850 4200 2000
 $Comp
 L Device:LED D15
@@
 	5350 2550 5500 2550
 Wire Wire Line
-	5250 2300 5250 3300
-Wire Wire Line
 	7250 3050 7250 3600
 Wire Wire Line
@@
 Connection ~ 7250 3050
 Wire Wire Line
-	5200 2300 5250 2300
+	5350 1900 5200 1900
 Wire Wire Line
-	4200 2100 4400 2100
+	5350 1900 5350 2550
 $Comp
-L MRDT_Switches:3P1T SW9
-U 1 1 61A05A6E
-P 4700 2400
-F 0 "SW9" H 4850 3187 60  0000 C CNN
-F 1 "3P1T" H 4850 3081 60  0000 C CNN
-F 2 "MRDT_Switches:3P1T_Switch" H 4450 2450 60  0001 C CNN
-F 3 "" H 4450 2450 60  0001 C CNN
-	1    4700 2400
+L Switch:SW_DPDT_x2 SW9
+U 1 1 61AA101E
+P 5000 2000
+F 0 "SW9" H 5000 2285 50  0000 C CNN
+F 1 "SW_DPDT_x2" H 5000 2194 50  0000 C CNN
+F 2 "Button_Switch_THT:SW_Slide_1P2T_CK_OS102011MS2Q" H 5000 2000 50  0001 C CNN
+F 3 "~" H 5000 2000 50  0001 C CNN
+	1    5000 2000
 	1    0    0    -1
 $EndComp
 Wire Wire Line
-	5350 1900 5200 1900
+	5250 3300 5250 2100
 Wire Wire Line
-	5350 1900 5350 2550
+	5250 2100 5200 2100
 Wire Wire Line
-	4500 1900 4400 1900
-Wire Wire Line
-	4400 1900 4400 2100
-Connection ~ 4400 2100
-Wire Wire Line
-	4400 2100 4400 2300
-Wire Wire Line
-	4400 2300 4500 2300
-NoConn ~ 5200 2100
-NoConn ~ 4500 2100
+	4800 2000 4200 2000
 $EndSCHEMATC
