File: GimbalBoard_Hardware/Molex.sch (KiCad schematic (older format))
At the start: 8 parts

Commit message: fixed h-labels in molex sheet
Connections:
- net Servo_1_PWM: no longer Conn2.3, Conn3.3, Conn4.3, Conn5.3, Conn6.3, Conn7.3, Conn8.3
- new net Servo_2_PWM: Conn2.3
- new net Servo_3_PWM: Conn3.3
- new net Servo_4_PWM: Conn4.3
- new net Servo_5_PWM: Conn5.3
- new net Servo_6_PWM: Conn6.3
- new net Servo_7_PWM: Conn7.3
- new net Servo_8_PWM: Conn8.3
Changed lines of the file:
@@
 Wire Wire Line
 	3500 6050 4100 6050
-Connection ~ 4100 6050
-Wire Wire Line
-	4100 6050 4100 6450
 Text HLabel 4250 1750 2    50   Input ~ 0
 Servo_1_PWM
 Text HLabel 4250 2350 2    50   Input ~ 0
-Servo_1_PWM
+Servo_2_PWM
 Text HLabel 4250 2950 2    50   Input ~ 0
-Servo_1_PWM
+Servo_3_PWM
 Text HLabel 4250 3550 2    50   Input ~ 0
-Servo_1_PWM
+Servo_4_PWM
 Text HLabel 4250 4150 2    50   Input ~ 0
-Servo_1_PWM
+Servo_5_PWM
 Text HLabel 4250 4750 2    50   Input ~ 0
-Servo_1_PWM
+Servo_6_PWM
 Text HLabel 4250 5350 2    50   Input ~ 0
-Servo_1_PWM
+Servo_7_PWM
 Text HLabel 4250 5950 2    50   Input ~ 0
-Servo_1_PWM
+Servo_8_PWM
 Wire Wire Line
 	3500 1750 4250 1750
@@
 Text HLabel 3950 1300 1    50   Input ~ 0
 +5V
-Text HLabel 4100 6450 3    50   Input ~ 0
-GND
+Connection ~ 4100 6050
+Wire Wire Line
+	4100 6050 4100 6450
+$Comp
+L power:GND #PWR?
+U 1 1 615FA9B5
+P 4100 6450
+F 0 "#PWR?" H 4100 6200 50  0001 C CNN
+F 1 "GND" H 4105 6277 50  0000 C CNN
+F 2 "" H 4100 6450 50  0001 C CNN
+F 3 "" H 4100 6450 50  0001 C CNN
+	1    4100 6450
+	1    0    0    -1
+$EndComp
 $EndSCHEMATC
