File: GimbalBoard_Hardware/Molex.sch (KiCad schematic (older format))
At the start: 8 parts

Commit message: added text
Connections:
- net +5V renamed +5VA
Changed lines of the file:
@@
 $Descr A4 11693 8268
 encoding utf-8
-Sheet 6 8
+Sheet 5 8
 Title ""
 Date ""
@@
 	3500 5950 4250 5950
 Text HLabel 3950 1300 1    50   Input ~ 0
-+5V
++5VA
 Connection ~ 4100 6050
 Wire Wire Line

Commit message: added more text
Other:
- note added: "Molex SL Connectors"
- moved on the sheet: Conn1, Conn2, Conn3, Conn4, Conn5, Conn6, Conn7, Conn8
Changed lines of the file:
@@
 L MRDT_Connectors:Molex_SL_03 Conn1
 U 1 1 615E1A75
-P 3300 1700
-F 0 "Conn1" H 3150 1500 60  0000 L CNN
-F 1 "Molex_SL_03" H 2850 1600 60  0000 L CNN
-F 2 "" H 3300 1700 60  0001 C CNN
-F 3 "" H 3300 1700 60  0001 C CNN
-	1    3300 1700
+P 3400 2400
+F 0 "Conn1" H 3250 2200 60  0000 L CNN
+F 1 "Molex_SL_03" H 2950 2300 60  0000 L CNN
+F 2 "" H 3400 2400 60  0001 C CNN
+F 3 "" H 3400 2400 60  0001 C CNN
+	1    3400 2400
 	-1   0    0    1
 $EndComp
@@
 L MRDT_Connectors:Molex_SL_03 Conn2
 U 1 1 615E7ABD
-P 3300 2300
-F 0 "Conn2" H 3150 2100 60  0000 L CNN
-F 1 "Molex_SL_03" H 2850 2200 60  0000 L CNN
-F 2 "" H 3300 2300 60  0001 C CNN
-F 3 "" H 3300 2300 60  0001 C CNN
-	1    3300 2300
+P 3400 3000
+F 0 "Conn2" H 3250 2800 60  0000 L CNN
+F 1 "Molex_SL_03" H 2950 2900 60  0000 L CNN
+F 2 "" H 3400 3000 60  0001 C CNN
+F 3 "" H 3400 3000 60  0001 C CNN
+	1    3400 3000
 	-1   0    0    1
 $EndComp
@@
 L MRDT_Connectors:Molex_SL_03 Conn3
 U 1 1 615E7D2A
-P 3300 2900
-F 0 "Conn3" H 3150 2700 60  0000 L CNN
-F 1 "Molex_SL_03" H 2850 2800 60  0000 L CNN
-F 2 "" H 3300 2900 60  0001 C CNN
-F 3 "" H 3300 2900 60  0001 C CNN
-	1    3300 2900
+P 3400 3600
+F 0 "Conn3" H 3250 3400 60  0000 L CNN
+F 1 "Molex_SL_03" H 2950 3500 60  0000 L CNN
+F 2 "" H 3400 3600 60  0001 C CNN
+F 3 "" H 3400 3600 60  0001 C CNN
+	1    3400 3600
 	-1   0    0    1
 $EndComp
@@
 L MRDT_Connectors:Molex_SL_03 Conn4
 U 1 1 615E800F
-P 3300 3500
-F 0 "Conn4" H 3150 3300 60  0000 L CNN
-F 1 "Molex_SL_03" H 2850 3400 60  0000 L CNN
-F 2 "" H 3300 3500 60  0001 C CNN
-F 3 "" H 3300 3500 60  0001 C CNN
-	1    3300 3500
+P 3400 4200
+F 0 "Conn4" H 3250 4000 60  0000 L CNN
+F 1 "Molex_SL_03" H 2950 4100 60  0000 L CNN
+F 2 "" H 3400 4200 60  0001 C CNN
+F 3 "" H 3400 4200 60  0001 C CNN
+	1    3400 4200
 	-1   0    0    1
 $EndComp
@@
 L MRDT_Connectors:Molex_SL_03 Conn5
 U 1 1 615E82F1
-P 3300 4100
-F 0 "Conn5" H 3150 3900 60  0000 L CNN
-F 1 "Molex_SL_03" H 2850 4000 60  0000 L CNN
-F 2 "" H 3300 4100 60  0001 C CNN
-F 3 "" H 3300 4100 60  0001 C CNN
-	1    3300 4100
+P 3400 4800
+F 0 "Conn5" H 3250 4600 60  0000 L CNN
+F 1 "Molex_SL_03" H 2950 4700 60  0000 L CNN
+F 2 "" H 3400 4800 60  0001 C CNN
+F 3 "" H 3400 4800 60  0001 C CNN
+	1    3400 4800
 	-1   0    0    1
 $EndComp
@@
 L MRDT_Connectors:Molex_SL_03 Conn6
 U 1 1 615E860E
-P 3300 4700
-F 0 "Conn6" H 3150 4500 60  0000 L CNN
-F 1 "Molex_SL_03" H 2850 4600 60  0000 L CNN
-F 2 "" H 3300 4700 60  0001 C CNN
-F 3 "" H 3300 4700 60  0001 C CNN
-	1    3300 4700
+P 3400 5400
+F 0 "Conn6" H 3250 5200 60  0000 L CNN
+F 1 "Molex_SL_03" H 2950 5300 60  0000 L CNN
+F 2 "" H 3400 5400 60  0001 C CNN
+F 3 "" H 3400 5400 60  0001 C CNN
+	1    3400 5400
 	-1   0    0    1
 $EndComp
@@
 L MRDT_Connectors:Molex_SL_03 Conn7
 U 1 1 615E87E0
-P 3300 5300
-F 0 "Conn7" H 3150 5100 60  0000 L CNN
-F 1 "Molex_SL_03" H 2850 5200 60  0000 L CNN
-F 2 "" H 3300 5300 60  0001 C CNN
-F 3 "" H 3300 5300 60  0001 C CNN
-	1    3300 5300
+P 3400 6000
+F 0 "Conn7" H 3250 5800 60  0000 L CNN
+F 1 "Molex_SL_03" H 2950 5900 60  0000 L CNN
+F 2 "" H 3400 6000 60  0001 C CNN
+F 3 "" H 3400 6000 60  0001 C CNN
+	1    3400 6000
 	-1   0    0    1
 $EndComp
@@
 L MRDT_Connectors:Molex_SL_03 Conn8
 U 1 1 615E89E0
-P 3300 5900
-F 0 "Conn8" H 3150 5700 60  0000 L CNN
-F 1 "Molex_SL_03" H 2850 5800 60  0000 L CNN
-F 2 "" H 3300 5900 60  0001 C CNN
-F 3 "" H 3300 5900 60  0001 C CNN
-	1    3300 5900
-	-1   0    0    1
-$EndComp
-Wire Wire Line
-	3500 6150 3950 6150
-Wire Wire Line
-	3950 6150 3950 5550
-Wire Wire Line
-	3500 5550 3950 5550
-Connection ~ 3950 5550
-Wire Wire Line
-	3950 5550 3950 4950
-Wire Wire Line
-	3500 4950 3950 4950
-Connection ~ 3950 4950
-Wire Wire Line
-	3950 4950 3950 4350
-Wire Wire Line
-	3500 4350 3950 4350
-Connection ~ 3950 4350
-Wire Wire Line
-	3950 4350 3950 3750
-Wire Wire Line
-	3500 3750 3950 3750
-Connection ~ 3950 3750
-Wire Wire Line
-	3950 3750 3950 3150
-Wire Wire Line
-	3500 3150 3950 3150
-Connection ~ 3950 3150
-Wire Wire Line
-	3950 3150 3950 2550
-Wire Wire Line
-	3500 2550 3950 2550
-Connection ~ 3950 2550
-Wire Wire Line
-	3950 2550 3950 1950
-Wire Wire Line
-	3500 1950 3950 1950
-Connection ~ 3950 1950
-Wire Wire Line
-	3950 1950 3950 1300
-Wire Wire Line
-	3500 1850 4100 1850
-Wire Wire Line
-	4100 1850 4100 2450
-Wire Wire Line
-	3500 2450 4100 2450
-Connection ~ 4100 2450
-Wire Wire Line
-	4100 2450 4100 3050
-Wire Wire Line
-	3500 3050 4100 3050
-Connection ~ 4100 3050
-Wire Wire Line
-	4100 3050 4100 3650
-Wire Wire Line
-	3500 3650 4100 3650
-Connection ~ 4100 3650
-Wire Wire Line
-	4100 3650 4100 4250
-Wire Wire Line
-	3500 4250 4100 4250
-Connection ~ 4100 4250
-Wire Wire Line
-	4100 4250 4100 4850
-Wire Wire Line
-	3500 4850 4100 4850
-Connection ~ 4100 4850
-Wire Wire Line
-	4100 4850 4100 5450
-Wire Wire Line
-	3500 5450 4100 5450
-Connection ~ 4100 5450
-Wire Wire Line
-	4100 5450 4100 6050
-Wire Wire Line
-	3500 6050 4100 6050
-Text HLabel 4250 1750 2    50   Input ~ 0
+P 3400 6600
+F 0 "Conn8" H 3250 6400 60  0000 L CNN
+F 1 "Molex_SL_03" H 2950 6500 60  0000 L CNN
+F 2 "" H 3400 6600 60  0001 C CNN
+F 3 "" H 3400 6600 60  0001 C CNN
+	1    3400 6600
+	-1   0    0    1
+$EndComp
+Wire Wire Line
+	3600 6850 4050 6850
+Wire Wire Line
+	4050 6850 4050 6250
+Wire Wire Line
+	3600 6250 4050 6250
+Connection ~ 4050 6250
+Wire Wire Line
+	4050 6250 4050 5650
+Wire Wire Line
+	3600 5650 4050 5650
+Connection ~ 4050 5650
+Wire Wire Line
+	4050 5650 4050 5050
+Wire Wire Line
+	3600 5050 4050 5050
+Connection ~ 4050 5050
+Wire Wire Line
+	4050 5050 4050 4450
+Wire Wire Line
+	3600 4450 4050 4450
+Connection ~ 4050 4450
+Wire Wire Line
+	4050 4450 4050 3850
+Wire Wire Line
+	3600 3850 4050 3850
+Connection ~ 4050 3850
+Wire Wire Line
+	4050 3850 4050 3250
+Wire Wire Line
+	3600 3250 4050 3250
+Connection ~ 4050 3250
+Wire Wire Line
+	4050 3250 4050 2650
+Wire Wire Line
+	3600 2650 4050 2650
+Connection ~ 4050 2650
+Wire Wire Line
+	4050 2650 4050 2000
+Wire Wire Line
+	3600 2550 4200 2550
+Wire Wire Line
+	4200 2550 4200 3150
+Wire Wire Line
+	3600 3150 4200 3150
+Connection ~ 4200 3150
+Wire Wire Line
+	4200 3150 4200 3750
+Wire Wire Line
+	3600 3750 4200 3750
+Connection ~ 4200 3750
+Wire Wire Line
+	4200 3750 4200 4350
+Wire Wire Line
+	3600 4350 4200 4350
+Connection ~ 4200 4350
+Wire Wire Line
+	4200 4350 4200 4950
+Wire Wire Line
+	3600 4950 4200 4950
+Connection ~ 4200 4950
+Wire Wire Line
+	4200 4950 4200 5550
+Wire Wire Line
+	3600 5550 4200 5550
+Connection ~ 4200 5550
+Wire Wire Line
+	4200 5550 4200 6150
+Wire Wire Line
+	3600 6150 4200 6150
+Connection ~ 4200 6150
+Wire Wire Line
+	4200 6150 4200 6750
+Wire Wire Line
+	3600 6750 4200 6750
+Text HLabel 4350 2450 2    50   Input ~ 0
 Servo_1_PWM
-Text HLabel 4250 2350 2    50   Input ~ 0
+Text HLabel 4350 3050 2    50   Input ~ 0
 Servo_2_PWM
-Text HLabel 4250 2950 2    50   Input ~ 0
+Text HLabel 4350 3650 2    50   Input ~ 0
 Servo_3_PWM
-Text HLabel 4250 3550 2    50   Input ~ 0
+Text HLabel 4350 4250 2    50   Input ~ 0
 Servo_4_PWM
-Text HLabel 4250 4150 2    50   Input ~ 0
+Text HLabel 4350 4850 2    50   Input ~ 0
 Servo_5_PWM
-Text HLabel 4250 4750 2    50   Input ~ 0
+Text HLabel 4350 5450 2    50   Input ~ 0
 Servo_6_PWM
-Text HLabel 4250 5350 2    50   Input ~ 0
+Text HLabel 4350 6050 2    50   Input ~ 0
 Servo_7_PWM
-Text HLabel 4250 5950 2    50   Input ~ 0
+Text HLabel 4350 6650 2    50   Input ~ 0
 Servo_8_PWM
 Wire Wire Line
-	3500 1750 4250 1750
-Wire Wire Line
-	3500 2350 4250 2350
-Wire Wire Line
-	3500 2950 4250 2950
-Wire Wire Line
-	3500 3550 4250 3550
-Wire Wire Line
-	3500 4150 4250 4150
-Wire Wire Line
-	3500 4750 4250 4750
-Wire Wire Line
-	3500 5350 4250 5350
-Wire Wire Line
-	3500 5950 4250 5950
-Text HLabel 3950 1300 1    50   Input ~ 0
+	3600 2450 4350 2450
+Wire Wire Line
+	3600 3050 4350 3050
+Wire Wire Line
+	3600 3650 4350 3650
+Wire Wire Line
+	3600 4250 4350 4250
+Wire Wire Line
+	3600 4850 4350 4850
+Wire Wire Line
+	3600 5450 4350 5450
+Wire Wire Line
+	3600 6050 4350 6050
+Wire Wire Line
+	3600 6650 4350 6650
+Text HLabel 4050 2000 1    50   Input ~ 0
 +5VA
-Connection ~ 4100 6050
-Wire Wire Line
-	4100 6050 4100 6450
-Text HLabel 4100 6450 3    50   Input ~ 0
+Connection ~ 4200 6750
+Wire Wire Line
+	4200 6750 4200 7150
+Text HLabel 4200 7150 3    50   Input ~ 0
 GND
+Text Notes 3350 1350 0    79   ~ 0
+Molex SL Connectors
 $EndSCHEMATC
