File: GimbalBoard_Hardware/GimbalBoard_Hardware.sch (KiCad schematic (older format))
At the start: 3 parts

Commit message: added more text
Changed lines of the file:
@@
 F11 "+5VA" I R 8750 4200 50
 $EndSheet
-Wire Wire Line
-	1400 1900 2300 1900
 Connection ~ 1400 1900
 Wire Wire Line
-	1550 2500 2550 2500
+	1550 2500 2300 2500
 Connection ~ 1550 2500
 Wire Wire Line
@@
 Wire Wire Line
 	2400 1900 2550 1900
-Connection ~ 2300 1900
-Wire Wire Line
-	2300 1900 2400 1900
 Wire Wire Line
 	1550 3100 1800 3100
@@
 	2300 3900 2550 3900
 Wire Wire Line
-	2300 1900 2300 3900
-Wire Wire Line
 	3850 3750 3700 3750
 Wire Wire Line
@@
 Wire Wire Line
 	2350 4150 2550 4150
+Wire Wire Line
+	1400 1900 2400 1900
+Wire Wire Line
+	2300 3900 2300 2500
+Connection ~ 2300 2500
+Wire Wire Line
+	2300 2500 2550 2500
 $EndSCHEMATC
