File: GimbalBoard_Hardware/5V-buck-converter.sch (KiCad schematic (older format))
At the start: 4 parts

Commit message: connected everything up and changed power to accomodate teensy instead of tiva
Connections:
- net +5V renamed +5VA
Changed lines of the file:
@@
 $Descr A4 11693 8268
 encoding utf-8
-Sheet 4 7
+Sheet 3 8
 Title ""
 Date ""
@@
 Power_Input_Act
 Text HLabel 6850 3550 2    50   Output ~ 0
-+5V
++5VA
 $Comp
 L power:GND #PWR?

Commit message: added h-labels
Changed lines of the file:
@@
-$EndComp
-$Comp
-L power:GND #PWR?
-U 1 1 6160A8C4
-P 5850 2900
-AR Path="/6160A8C4" Ref="#PWR?"  Part="1"
-AR Path="/615B83A4/6160A8C4" Ref="#PWR?"  Part="1"
-AR Path="/61606E20/6160A8C4" Ref="#PWR?"  Part="1"
-F 0 "#PWR?" H 5850 2650 50  0001 C CNN
-F 1 "GND" H 5855 2727 50  0000 C CNN
-F 2 "" H 5850 2900 50  0001 C CNN
-F 3 "" H 5850 2900 50  0001 C CNN
-	1    5850 2900
-	1    0    0    -1
 $EndComp
 $Comp
@@
 Text HLabel 6850 3550 2    50   Output ~ 0
 +5VA
-$Comp
-L power:GND #PWR?
-U 1 1 6160A8D8
-P 5850 4250
-F 0 "#PWR?" H 5850 4000 50  0001 C CNN
-F 1 "GND" H 5855 4077 50  0000 C CNN
-F 2 "" H 5850 4250 50  0001 C CNN
-F 3 "" H 5850 4250 50  0001 C CNN
-	1    5850 4250
-	1    0    0    -1
-$EndComp
 Wire Wire Line
 	6250 2600 6500 2600
@@
 Wire Wire Line
 	4800 3550 5200 3550
+Text HLabel 5850 2900 3    50   Input ~ 0
+GND
+Text HLabel 5850 4250 3    50   Input ~ 0
+GND
 $EndSCHEMATC

Commit message: added more text
Other:
- note added: "5VA Converter"
Changed lines of the file:
@@
 Text HLabel 5850 4250 3    50   Input ~ 0
 GND
+Text Notes 5400 2100 0    79   ~ 0
+5VA Converter
 $EndSCHEMATC

Commit message: added labels, numbered everything, added no connection to pins. Still can't get past a couple pf errors in the electrical rules check
Parts:
- C1, C2: renamed from C?; value C -> 10uF
- gave numbers to parts that had none: 2
Other:
- note removed: "5VA Converter"
Changed lines of the file:
@@
 AR Path="/6160A8B8" Ref="U?"  Part="1"
 AR Path="/615B83A4/6160A8B8" Ref="U?"  Part="1"
-AR Path="/61606E20/6160A8B8" Ref="U?"  Part="1"
-F 0 "U?" H 5700 3600 60  0001 C CNN
+AR Path="/61606E20/6160A8B8" Ref="U2"  Part="1"
+F 0 "U2" H 5850 4050 60  0000 C CNN
 F 1 "OKI" H 5850 3931 60  0000 C CNN
 F 2 "" H 5450 3550 60  0001 C CNN
@@
 AR Path="/6160A8BE" Ref="U?"  Part="1"
 AR Path="/615B83A4/6160A8BE" Ref="U?"  Part="1"
-AR Path="/61606E20/6160A8BE" Ref="U?"  Part="1"
-F 0 "U?" H 5700 2650 60  0001 C CNN
+AR Path="/61606E20/6160A8BE" Ref="U1"  Part="1"
+F 0 "U1" H 5850 3100 60  0000 C CNN
 F 1 "OKI" H 5850 2981 60  0000 C CNN
 F 2 "" H 5450 2600 60  0001 C CNN
 F 3 "" H 5450 2600 60  0001 C CNN
 	1    5650 2700
-	1    0    0    -1
-$EndComp
-$Comp
-L Device:C C?
-U 1 1 6160A8CA
-P 5200 3950
-AR Path="/6160A8CA" Ref="C?"  Part="1"
-AR Path="/615B83A4/6160A8CA" Ref="C?"  Part="1"
-AR Path="/61606E20/6160A8CA" Ref="C?"  Part="1"
-F 0 "C?" H 5315 3996 50  0000 L CNN
-F 1 "C" H 5315 3905 50  0000 L CNN
-F 2 "" H 5238 3800 50  0001 C CNN
-F 3 "~" H 5200 3950 50  0001 C CNN
-	1    5200 3950
-	1    0    0    -1
-$EndComp
-$Comp
-L Device:C C?
-U 1 1 6160A8D0
-P 6500 3950
-AR Path="/6160A8D0" Ref="C?"  Part="1"
-AR Path="/615B83A4/6160A8D0" Ref="C?"  Part="1"
-AR Path="/61606E20/6160A8D0" Ref="C?"  Part="1"
-F 0 "C?" H 6615 3996 50  0000 L CNN
-F 1 "C" H 6615 3905 50  0000 L CNN
-F 2 "" H 6538 3800 50  0001 C CNN
-F 3 "~" H 6500 3950 50  0001 C CNN
-	1    6500 3950
 	1    0    0    -1
 $EndComp
@@
 Wire Wire Line
 	4800 3550 5200 3550
-Text HLabel 5850 2900 3    50   Input ~ 0
+Text HLabel 5850 2900 3    50   Output ~ 0
 GND
-Text HLabel 5850 4250 3    50   Input ~ 0
+Text HLabel 5850 4250 3    50   Output ~ 0
 GND
-Text Notes 5400 2100 0    79   ~ 0
-5VA Converter
+$Comp
+L Device:C C?
+U 1 1 6160A8D0
+P 6500 3950
+AR Path="/6160A8D0" Ref="C?"  Part="1"
+AR Path="/615B83A4/6160A8D0" Ref="C?"  Part="1"
+AR Path="/61606E20/6160A8D0" Ref="C2"  Part="1"
+F 0 "C2" H 6615 3996 50  0000 L CNN
+F 1 "10uF" H 6615 3905 50  0000 L CNN
+F 2 "" H 6538 3800 50  0001 C CNN
+F 3 "~" H 6500 3950 50  0001 C CNN
+	1    6500 3950
+	1    0    0    -1
+$EndComp
+$Comp
+L Device:C C?
+U 1 1 6160A8CA
+P 5200 3950
+AR Path="/6160A8CA" Ref="C?"  Part="1"
+AR Path="/615B83A4/6160A8CA" Ref="C?"  Part="1"
+AR Path="/61606E20/6160A8CA" Ref="C1"  Part="1"
+F 0 "C1" H 5315 3996 50  0000 L CNN
+F 1 "10uF" H 5315 3905 50  0000 L CNN
+F 2 "" H 5238 3800 50  0001 C CNN
+F 3 "~" H 5200 3950 50  0001 C CNN
+	1    5200 3950
+	1    0    0    -1
+$EndComp
 $EndSCHEMATC
