File: GimbalBoard_Hardware/Act_Buck_Converter.sch (KiCad schematic (older format))
At the start: 4 parts, among them U1 OKI, U2 OKI

Commit message: updated labels and file names
Other:
- note added: "12VA to 5VA Converter"
Changed lines of the file:
@@
 	1    0    0    -1
 $EndComp
+Text Notes 5250 2050 0    79   ~ 0
+12VA to 5VA Converter
 $EndSCHEMATC
