File: GimbalBoard_Hardware/Log_Buck_Converter.sch (KiCad schematic (older format))
At the start: 6 parts, among them U3 OKI, U4 OKI

Commit message: updated labels and file names
Other:
- note added: "12VL to 3.3VL Converter"
- note added: "12VL to 5VL Converter"
- note removed: "3.3VL Converter"
- note removed: "5VL Converter"
Changed lines of the file:
@@
 Wire Wire Line
 	4900 3600 5150 3600
-Text Notes 5350 1250 0    79   ~ 0
-3.3VL Converter
-Text Notes 5500 3100 0    79   ~ 0
-5VL Converter
+Text Notes 5150 1250 0    79   ~ 0
+12VL to 3.3VL Converter
+Text Notes 5250 3100 0    79   ~ 0
+12VL to 5VL Converter
 Text HLabel 4900 1750 0    50   Input ~ 0
 Power_Input_Log
