File: GimbalBoard_Hardware/Servo_Indicators.sch (KiCad schematic (older format))
At the start: 32 parts, among them Q1 Q_NMOS_GDS, Q2 Q_NMOS_GDS, Q3 Q_NMOS_GDS, Q4 Q_NMOS_GDS, Q5 Q_NMOS_GDS, Q6 Q_NMOS_GDS, Q7 Q_NMOS_GDS, Q8 Q_NMOS_GDS

Commit message: sheet has been reviewed
schematic has been reviewed. and resister values have been changed. as well as a ground being added
Parts:
- R17, R18, R19, R20, R21, R22, R23, R24: value 510 -> 100
