File: GimbalBoard_Hardware/servo-connectors2.sch (KiCad schematic (older format))
At the start: 40 parts, among them Q1 Q_NMOS_GDS, Q2 Q_NMOS_GDS, Q3 Q_NMOS_GDS, Q4 Q_NMOS_GDS, Q5 Q_NMOS_GDS, Q6 Q_NMOS_GDS, Q7 Q_NMOS_GDS, Q8 Q_NMOS_GDS

Commit message: Added more footprints
I added more footprints. Not done yet. I'd like to come back when when I can verify with max about some of the other components.
Parts:
- D17, D18, D19, D20, D21, D22, D23, D24: footprint (none) -> LED_SMD:LED_0603_1608Metric_Pad1.05x0.95mm_HandSolder
- R17, R18, R19, R20, R21, R22, R23, R24, R25, R26, R27, R28, R29, R30, R31, R32: footprint (none) -> Resistor_SMD:R_0603_1608Metric_Pad0.98x0.95mm_HandSolder
Changed lines of the file:
@@
 F 0 "R25" V 2000 1350 50  0000 C CNN
 F 1 "510" V 2100 1350 50  0000 C CNN
-F 2 "" V 2030 1350 50  0001 C CNN
+F 2 "Resistor_SMD:R_0603_1608Metric_Pad0.98x0.95mm_HandSolder" V 2030 1350 50  0001 C CNN
 F 3 "~" H 2100 1350 50  0001 C CNN
 	1    2100 1350
@@
 F 0 "R26" V 2000 2100 50  0000 C CNN
 F 1 "510" V 2100 2100 50  0000 C CNN
-F 2 "" V 2030 2100 50  0001 C CNN
+F 2 "Resistor_SMD:R_0603_1608Metric_Pad0.98x0.95mm_HandSolder" V 2030 2100 50  0001 C CNN
 F 3 "~" H 2100 2100 50  0001 C CNN
 	1    2100 2100
@@
 F 0 "R27" V 2000 2850 50  0000 C CNN
 F 1 "510" V 2100 2850 50  0000 C CNN
-F 2 "" V 2030 2850 50  0001 C CNN
+F 2 "Resistor_SMD:R_0603_1608Metric_Pad0.98x0.95mm_HandSolder" V 2030 2850 50  0001 C CNN
 F 3 "~" H 2100 2850 50  0001 C CNN
 	1    2100 2850
@@
 F 0 "R28" V 2000 3600 50  0000 C CNN
 F 1 "510" V 2100 3600 50  0000 C CNN
-F 2 "" V 2030 3600 50  0001 C CNN
+F 2 "Resistor_SMD:R_0603_1608Metric_Pad0.98x0.95mm_HandSolder" V 2030 3600 50  0001 C CNN
 F 3 "~" H 2100 3600 50  0001 C CNN
 	1    2100 3600
@@
 F 0 "R29" V 2000 4350 50  0000 C CNN
 F 1 "510" V 2100 4350 50  0000 C CNN
-F 2 "" V 2030 4350 50  0001 C CNN
+F 2 "Resistor_SMD:R_0603_1608Metric_Pad0.98x0.95mm_HandSolder" V 2030 4350 50  0001 C CNN
 F 3 "~" H 2100 4350 50  0001 C CNN
 	1    2100 4350
@@
 F 0 "R30" V 2000 5100 50  0000 C CNN
 F 1 "510" V 2100 5100 50  0000 C CNN
-F 2 "" V 2030 5100 50  0001 C CNN
+F 2 "Resistor_SMD:R_0603_1608Metric_Pad0.98x0.95mm_HandSolder" V 2030 5100 50  0001 C CNN
 F 3 "~" H 2100 5100 50  0001 C CNN
 	1    2100 5100
@@
 F 0 "R31" V 2000 5850 50  0000 C CNN
 F 1 "510" V 2100 5850 50  0000 C CNN
-F 2 "" V 2030 5850 50  0001 C CNN
+F 2 "Resistor_SMD:R_0603_1608Metric_Pad0.98x0.95mm_HandSolder" V 2030 5850 50  0001 C CNN
 F 3 "~" H 2100 5850 50  0001 C CNN
 	1    2100 5850
@@
 F 0 "R32" V 2000 6600 50  0000 C CNN
 F 1 "510" V 2100 6600 50  0000 C CNN
-F 2 "" V 2030 6600 50  0001 C CNN
+F 2 "Resistor_SMD:R_0603_1608Metric_Pad0.98x0.95mm_HandSolder" V 2030 6600 50  0001 C CNN
 F 3 "~" H 2100 6600 50  0001 C CNN
 	1    2100 6600
@@
 F 0 "R24" V 2750 6900 50  0000 C CNN
 F 1 "100" V 2850 6900 50  0000 C CNN
-F 2 "" V 2780 6900 50  0001 C CNN
+F 2 "Resistor_SMD:R_0603_1608Metric_Pad0.98x0.95mm_HandSolder" V 2780 6900 50  0001 C CNN
 F 3 "~" H 2850 6900 50  0001 C CNN
 	1    2850 6900
@@
 F 0 "D24" H 2350 7000 50  0000 C CNN
 F 1 "LED" H 2350 6800 50  0000 C CNN
-F 2 "" H 2350 6900 50  0001 C CNN
+F 2 "LED_SMD:LED_0603_1608Metric_Pad1.05x0.95mm_HandSolder" H 2350 6900 50  0001 C CNN
 F 3 "~" H 2350 6900 50  0001 C CNN
 	1    2350 6900
@@
 F 0 "R23" V 2750 6150 50  0000 C CNN
 F 1 "100" V 2850 6150 50  0000 C CNN
-F 2 "" V 2780 6150 50  0001 C CNN
+F 2 "Resistor_SMD:R_0603_1608Metric_Pad0.98x0.95mm_HandSolder" V 2780 6150 50  0001 C CNN
 F 3 "~" H 2850 6150 50  0001 C CNN
 	1    2850 6150
@@
 F 0 "D23" H 2350 6250 50  0000 C CNN
 F 1 "LED" H 2350 6050 50  0000 C CNN
-F 2 "" H 2350 6150 50  0001 C CNN
+F 2 "LED_SMD:LED_0603_1608Metric_Pad1.05x0.95mm_HandSolder" H 2350 6150 50  0001 C CNN
 F 3 "~" H 2350 6150 50  0001 C CNN
 	1    2350 6150
@@
 F 0 "R22" V 2750 5400 50  0000 C CNN
 F 1 "100" V 2850 5400 50  0000 C CNN
-F 2 "" V 2780 5400 50  0001 C CNN
+F 2 "Resistor_SMD:R_0603_1608Metric_Pad0.98x0.95mm_HandSolder" V 2780 5400 50  0001 C CNN
 F 3 "~" H 2850 5400 50  0001 C CNN
 	1    2850 5400
@@
 F 0 "D22" H 2350 5500 50  0000 C CNN
 F 1 "LED" H 2350 5300 50  0000 C CNN
-F 2 "" H 2350 5400 50  0001 C CNN
+F 2 "LED_SMD:LED_0603_1608Metric_Pad1.05x0.95mm_HandSolder" H 2350 5400 50  0001 C CNN
 F 3 "~" H 2350 5400 50  0001 C CNN
 	1    2350 5400
@@
 F 0 "D21" H 2350 4750 50  0000 C CNN
 F 1 "LED" H 2350 4550 50  0000 C CNN
-F 2 "" H 2350 4650 50  0001 C CNN
+F 2 "LED_SMD:LED_0603_1608Metric_Pad1.05x0.95mm_HandSolder" H 2350 4650 50  0001 C CNN
 F 3 "~" H 2350 4650 50  0001 C CNN
 	1    2350 4650
@@
 F 0 "R21" V 2750 4650 50  0000 C CNN
 F 1 "100" V 2850 4650 50  0000 C CNN
-F 2 "" V 2780 4650 50  0001 C CNN
+F 2 "Resistor_SMD:R_0603_1608Metric_Pad0.98x0.95mm_HandSolder" V 2780 4650 50  0001 C CNN
 F 3 "~" H 2850 4650 50  0001 C CNN
 	1    2850 4650
@@
 F 0 "R20" V 2750 3900 50  0000 C CNN
 F 1 "100" V 2850 3900 50  0000 C CNN
-F 2 "" V 2780 3900 50  0001 C CNN
+F 2 "Resistor_SMD:R_0603_1608Metric_Pad0.98x0.95mm_HandSolder" V 2780 3900 50  0001 C CNN
 F 3 "~" H 2850 3900 50  0001 C CNN
 	1    2850 3900
@@
 F 0 "D20" H 2350 4000 50  0000 C CNN
 F 1 "LED" H 2350 3800 50  0000 C CNN
-F 2 "" H 2350 3900 50  0001 C CNN
+F 2 "LED_SMD:LED_0603_1608Metric_Pad1.05x0.95mm_HandSolder" H 2350 3900 50  0001 C CNN
 F 3 "~" H 2350 3900 50  0001 C CNN
 	1    2350 3900
@@
 F 0 "R19" V 2750 3150 50  0000 C CNN
 F 1 "100" V 2850 3150 50  0000 C CNN
-F 2 "" V 2780 3150 50  0001 C CNN
+F 2 "Resistor_SMD:R_0603_1608Metric_Pad0.98x0.95mm_HandSolder" V 2780 3150 50  0001 C CNN
 F 3 "~" H 2850 3150 50  0001 C CNN
 	1    2850 3150
@@
 F 0 "D19" H 2350 3250 50  0000 C CNN
 F 1 "LED" H 2350 3050 50  0000 C CNN
-F 2 "" H 2350 3150 50  0001 C CNN
+F 2 "LED_SMD:LED_0603_1608Metric_Pad1.05x0.95mm_HandSolder" H 2350 3150 50  0001 C CNN
 F 3 "~" H 2350 3150 50  0001 C CNN
 	1    2350 3150
@@
 F 0 "R18" V 2750 2400 50  0000 C CNN
 F 1 "100" V 2850 2400 50  0000 C CNN
-F 2 "" V 2780 2400 50  0001 C CNN
+F 2 "Resistor_SMD:R_0603_1608Metric_Pad0.98x0.95mm_HandSolder" V 2780 2400 50  0001 C CNN
 F 3 "~" H 2850 2400 50  0001 C CNN
 	1    2850 2400
@@
 F 0 "D18" H 2350 2500 50  0000 C CNN
 F 1 "LED" H 2350 2300 50  0000 C CNN
-F 2 "" H 2350 2400 50  0001 C CNN
+F 2 "LED_SMD:LED_0603_1608Metric_Pad1.05x0.95mm_HandSolder" H 2350 2400 50  0001 C CNN
 F 3 "~" H 2350 2400 50  0001 C CNN
 	1    2350 2400
@@
 F 0 "R17" V 2750 1650 50  0000 C CNN
 F 1 "100" V 2850 1650 50  0000 C CNN
-F 2 "" V 2780 1650 50  0001 C CNN
+F 2 "Resistor_SMD:R_0603_1608Metric_Pad0.98x0.95mm_HandSolder" V 2780 1650 50  0001 C CNN
 F 3 "~" H 2850 1650 50  0001 C CNN
 	1    2850 1650
@@
 F 0 "D17" H 2350 1750 50  0000 C CNN
 F 1 "LED" H 2350 1550 50  0000 C CNN
-F 2 "" H 2350 1650 50  0001 C CNN
+F 2 "LED_SMD:LED_0603_1608Metric_Pad1.05x0.95mm_HandSolder" H 2350 1650 50  0001 C CNN
 F 3 "~" H 2350 1650 50  0001 C CNN
 	1    2350 1650

Commit message: Footprints finished
the footprints are finished. the RJ45 connector has been added for eithernet.
the net is in the layout thing but I haven't moved anything yet
Parts:
- Conn1, Conn2, Conn3, Conn4, Conn5, Conn6, Conn7, Conn8: footprint (none) -> MRDT_Connectors:MOLEX_SL_03_Horizontal
- Q1, Q2, Q3, Q4, Q5, Q6, Q7, Q8: footprint (none) -> Package_TO_SOT_SMD:SOT-23
Changed lines of the file:
@@
 F 0 "Q8" V 1999 6800 50  0000 C CNN
 F 1 "Q_NMOS_GDS" V 2090 6800 50  0000 C CNN
-F 2 "" H 1950 6900 50  0001 C CNN
+F 2 "Package_TO_SOT_SMD:SOT-23" H 1950 6900 50  0001 C CNN
 F 3 "~" H 1750 6800 50  0001 C CNN
 	1    1750 6800
@@
 F 0 "Q7" V 1999 6050 50  0000 C CNN
 F 1 "Q_NMOS_GDS" V 2090 6050 50  0000 C CNN
-F 2 "" H 1950 6150 50  0001 C CNN
+F 2 "Package_TO_SOT_SMD:SOT-23" H 1950 6150 50  0001 C CNN
 F 3 "~" H 1750 6050 50  0001 C CNN
 	1    1750 6050
@@
 F 0 "Q6" V 1999 5300 50  0000 C CNN
 F 1 "Q_NMOS_GDS" V 2090 5300 50  0000 C CNN
-F 2 "" H 1950 5400 50  0001 C CNN
+F 2 "Package_TO_SOT_SMD:SOT-23" H 1950 5400 50  0001 C CNN
 F 3 "~" H 1750 5300 50  0001 C CNN
 	1    1750 5300
@@
 F 0 "Q5" V 1999 4550 50  0000 C CNN
 F 1 "Q_NMOS_GDS" V 2090 4550 50  0000 C CNN
-F 2 "" H 1950 4650 50  0001 C CNN
+F 2 "Package_TO_SOT_SMD:SOT-23" H 1950 4650 50  0001 C CNN
 F 3 "~" H 1750 4550 50  0001 C CNN
 	1    1750 4550
@@
 F 0 "Q4" V 1999 3800 50  0000 C CNN
 F 1 "Q_NMOS_GDS" V 2090 3800 50  0000 C CNN
-F 2 "" H 1950 3900 50  0001 C CNN
+F 2 "Package_TO_SOT_SMD:SOT-23" H 1950 3900 50  0001 C CNN
 F 3 "~" H 1750 3800 50  0001 C CNN
 	1    1750 3800
@@
 F 0 "Q3" V 1999 3050 50  0000 C CNN
 F 1 "Q_NMOS_GDS" V 2090 3050 50  0000 C CNN
-F 2 "" H 1950 3150 50  0001 C CNN
+F 2 "Package_TO_SOT_SMD:SOT-23" H 1950 3150 50  0001 C CNN
 F 3 "~" H 1750 3050 50  0001 C CNN
 	1    1750 3050
@@
 F 0 "Q2" V 1999 2300 50  0000 C CNN
 F 1 "Q_NMOS_GDS" V 2090 2300 50  0000 C CNN
-F 2 "" H 1950 2400 50  0001 C CNN
+F 2 "Package_TO_SOT_SMD:SOT-23" H 1950 2400 50  0001 C CNN
 F 3 "~" H 1750 2300 50  0001 C CNN
 	1    1750 2300
@@
 F 0 "Q1" V 1999 1550 50  0000 C CNN
 F 1 "Q_NMOS_GDS" V 2090 1550 50  0000 C CNN
-F 2 "" H 1950 1650 50  0001 C CNN
+F 2 "Package_TO_SOT_SMD:SOT-23" H 1950 1650 50  0001 C CNN
 F 3 "~" H 1750 1550 50  0001 C CNN
 	1    1750 1550
@@
 F 0 "Conn8" H 5650 6000 60  0000 L CNN
 F 1 "Molex_SL_03" H 5350 6100 60  0000 L CNN
-F 2 "" H 5800 6200 60  0001 C CNN
+F 2 "MRDT_Connectors:MOLEX_SL_03_Horizontal" H 5800 6200 60  0001 C CNN
 F 3 "" H 5800 6200 60  0001 C CNN
 	1    5800 6200
@@
 F 0 "Conn7" H 5650 5400 60  0000 L CNN
 F 1 "Molex_SL_03" H 5350 5500 60  0000 L CNN
-F 2 "" H 5800 5600 60  0001 C CNN
+F 2 "MRDT_Connectors:MOLEX_SL_03_Horizontal" H 5800 5600 60  0001 C CNN
 F 3 "" H 5800 5600 60  0001 C CNN
 	1    5800 5600
@@
 F 0 "Conn6" H 5650 4800 60  0000 L CNN
 F 1 "Molex_SL_03" H 5350 4900 60  0000 L CNN
-F 2 "" H 5800 5000 60  0001 C CNN
+F 2 "MRDT_Connectors:MOLEX_SL_03_Horizontal" H 5800 5000 60  0001 C CNN
 F 3 "" H 5800 5000 60  0001 C CNN
 	1    5800 5000
@@
 F 0 "Conn5" H 5650 4200 60  0000 L CNN
 F 1 "Molex_SL_03" H 5350 4300 60  0000 L CNN
-F 2 "" H 5800 4400 60  0001 C CNN
+F 2 "MRDT_Connectors:MOLEX_SL_03_Horizontal" H 5800 4400 60  0001 C CNN
 F 3 "" H 5800 4400 60  0001 C CNN
 	1    5800 4400
@@
 F 0 "Conn4" H 5650 3600 60  0000 L CNN
 F 1 "Molex_SL_03" H 5350 3700 60  0000 L CNN
-F 2 "" H 5800 3800 60  0001 C CNN
+F 2 "MRDT_Connectors:MOLEX_SL_03_Horizontal" H 5800 3800 60  0001 C CNN
 F 3 "" H 5800 3800 60  0001 C CNN
 	1    5800 3800
@@
 F 0 "Conn3" H 5650 3000 60  0000 L CNN
 F 1 "Molex_SL_03" H 5350 3100 60  0000 L CNN
-F 2 "" H 5800 3200 60  0001 C CNN
+F 2 "MRDT_Connectors:MOLEX_SL_03_Horizontal" H 5800 3200 60  0001 C CNN
 F 3 "" H 5800 3200 60  0001 C CNN
 	1    5800 3200
@@
 F 0 "Conn2" H 5650 2400 60  0000 L CNN
 F 1 "Molex_SL_03" H 5350 2500 60  0000 L CNN
-F 2 "" H 5800 2600 60  0001 C CNN
+F 2 "MRDT_Connectors:MOLEX_SL_03_Horizontal" H 5800 2600 60  0001 C CNN
 F 3 "" H 5800 2600 60  0001 C CNN
 	1    5800 2600
@@
 F 0 "Conn1" H 5650 1800 60  0000 L CNN
 F 1 "Molex_SL_03" H 5350 1900 60  0000 L CNN
-F 2 "" H 5800 2000 60  0001 C CNN
+F 2 "MRDT_Connectors:MOLEX_SL_03_Horizontal" H 5800 2000 60  0001 C CNN
 F 3 "" H 5800 2000 60  0001 C CNN
 	1    5800 2000

Commit message: ethernet fixed.
the ethernet is fixed. as well as the switch footprint association issue.
I'm not certain that the current footprint being used matches an actual switch. also this edit does not have the 3x2 microfit connectors
Parts:
- added Conn10, Conn11, Conn12, Conn13: Molex_uF_D_06, MRDT_Connectors:MOLEX_uF_D_06_Horizontal, symbol MRDT_Connectors:Molex_uF_D_06
Changed lines of the file:
@@
 	1    0    0    -1
 $EndComp
+Wire Wire Line
+	5600 1750 5150 1750
+Wire Wire Line
+	5600 1850 5000 1850
+Text HLabel 4850 1950 0    50   Input ~ 0
+Servo_1_PWM
+Wire Wire Line
+	5600 1950 4850 1950
+Text HLabel 5150 1500 1    50   Input ~ 0
++5VA
+Text Notes 4550 1000 0    79   ~ 0
+Molex SL Connectors
+Wire Wire Line
+	5150 1500 5150 1750
+Connection ~ 5150 1750
+Text HLabel 5000 6450 3    50   Input ~ 0
+GND
+Text HLabel 4850 6150 0    50   Input ~ 0
+Servo_8_PWM
+Connection ~ 5000 6050
+Wire Wire Line
+	5000 6050 5000 6450
+Wire Wire Line
+	5600 6150 4850 6150
+Wire Wire Line
+	5600 6050 5000 6050
+Wire Wire Line
+	5600 5950 5150 5950
 $Comp
 L MRDT_Connectors:Molex_SL_03 Conn?
@@
 	1    0    0    -1
 $EndComp
+Text HLabel 4850 5550 0    50   Input ~ 0
+Servo_7_PWM
+Connection ~ 5000 5450
+Wire Wire Line
+	5000 6050 5000 5450
+Wire Wire Line
+	5150 5350 5150 5950
+Connection ~ 5150 5350
+Wire Wire Line
+	5600 5550 4850 5550
+Wire Wire Line
+	5600 5450 5000 5450
+Wire Wire Line
+	5600 5350 5150 5350
+Text HLabel 4850 4950 0    50   Input ~ 0
+Servo_6_PWM
+Connection ~ 5000 4850
+Wire Wire Line
+	5000 5450 5000 4850
+Wire Wire Line
+	5150 4750 5150 5350
+Connection ~ 5150 4750
+Wire Wire Line
+	5600 4950 4850 4950
+Wire Wire Line
+	5600 4850 5000 4850
+Wire Wire Line
+	5600 4750 5150 4750
 $Comp
 L MRDT_Connectors:Molex_SL_03 Conn?
@@
 	1    0    0    -1
 $EndComp
+Text HLabel 4850 4350 0    50   Input ~ 0
+Servo_5_PWM
+Connection ~ 5000 4250
+Wire Wire Line
+	5000 4850 5000 4250
+Wire Wire Line
+	5150 4150 5150 4750
+Connection ~ 5150 4150
+Wire Wire Line
+	5600 4350 4850 4350
+Wire Wire Line
+	5600 4250 5000 4250
+Wire Wire Line
+	5600 4150 5150 4150
 $Comp
 L MRDT_Connectors:Molex_SL_03 Conn?
@@
 	1    0    0    -1
 $EndComp
+Text HLabel 4850 3750 0    50   Input ~ 0
+Servo_4_PWM
+Connection ~ 5000 3650
+Wire Wire Line
+	5000 4250 5000 3650
+Wire Wire Line
+	5150 3550 5150 4150
+Connection ~ 5150 3550
+Wire Wire Line
+	5600 3750 4850 3750
+Wire Wire Line
+	5600 3650 5000 3650
+Wire Wire Line
+	5600 3550 5150 3550
 $Comp
 L MRDT_Connectors:Molex_SL_03 Conn?
@@
 	1    0    0    -1
 $EndComp
+Text HLabel 4850 3150 0    50   Input ~ 0
+Servo_3_PWM
+Connection ~ 5150 2950
+Wire Wire Line
+	5150 2950 5150 3550
+Wire Wire Line
+	5000 3650 5000 3050
+Connection ~ 5000 3050
+Wire Wire Line
+	5600 2950 5150 2950
+Wire Wire Line
+	5600 3050 5000 3050
+Wire Wire Line
+	5600 3150 4850 3150
 $Comp
 L MRDT_Connectors:Molex_SL_03 Conn?
@@
 	1    0    0    -1
 $EndComp
+Text HLabel 4850 2550 0    50   Input ~ 0
+Servo_2_PWM
+Connection ~ 5000 2450
+Wire Wire Line
+	5000 3050 5000 2450
+Wire Wire Line
+	5150 2350 5150 2950
+Connection ~ 5150 2350
+Wire Wire Line
+	5150 1750 5150 2350
+Wire Wire Line
+	5000 2450 5000 1850
+Wire Wire Line
+	5600 2550 4850 2550
+Wire Wire Line
+	5600 2450 5000 2450
+Wire Wire Line
+	5600 2350 5150 2350
 $Comp
 L MRDT_Connectors:Molex_SL_03 Conn?
@@
 	1    0    0    -1
 $EndComp
-Wire Wire Line
-	5600 1750 5150 1750
-Wire Wire Line
-	5150 1750 5150 2350
-Wire Wire Line
-	5600 2350 5150 2350
-Connection ~ 5150 2350
-Wire Wire Line
-	5150 2350 5150 2950
-Wire Wire Line
-	5600 2950 5150 2950
-Connection ~ 5150 2950
-Wire Wire Line
-	5150 2950 5150 3550
-Wire Wire Line
-	5600 3550 5150 3550
-Connection ~ 5150 3550
-Wire Wire Line
-	5150 3550 5150 4150
-Wire Wire Line
-	5600 4150 5150 4150
-Connection ~ 5150 4150
-Wire Wire Line
-	5150 4150 5150 4750
-Wire Wire Line
-	5600 4750 5150 4750
-Connection ~ 5150 4750
-Wire Wire Line
-	5150 4750 5150 5350
-Wire Wire Line
-	5600 5350 5150 5350
-Connection ~ 5150 5350
-Wire Wire Line
-	5150 5350 5150 5950
-Wire Wire Line
-	5600 5950 5150 5950
-Wire Wire Line
-	5600 6050 5000 6050
-Wire Wire Line
-	5000 6050 5000 5450
-Wire Wire Line
-	5600 5450 5000 5450
-Connection ~ 5000 5450
-Wire Wire Line
-	5000 5450 5000 4850
-Wire Wire Line
-	5600 4850 5000 4850
-Connection ~ 5000 4850
-Wire Wire Line
-	5000 4850 5000 4250
-Wire Wire Line
-	5600 4250 5000 4250
-Connection ~ 5000 4250
-Wire Wire Line
-	5000 4250 5000 3650
-Wire Wire Line
-	5600 3650 5000 3650
-Connection ~ 5000 3650
-Wire Wire Line
-	5000 3650 5000 3050
-Wire Wire Line
-	5600 3050 5000 3050
-Connection ~ 5000 3050
-Wire Wire Line
-	5000 3050 5000 2450
-Wire Wire Line
-	5600 2450 5000 2450
-Connection ~ 5000 2450
-Wire Wire Line
-	5000 2450 5000 1850
-Wire Wire Line
-	5600 1850 5000 1850
-Text HLabel 4850 1950 0    50   Input ~ 0
-Servo_1_PWM
-Text HLabel 4850 2550 0    50   Input ~ 0
-Servo_2_PWM
-Text HLabel 4850 3150 0    50   Input ~ 0
-Servo_3_PWM
-Text HLabel 4850 3750 0    50   Input ~ 0
-Servo_4_PWM
-Text HLabel 4850 4350 0    50   Input ~ 0
-Servo_5_PWM
-Text HLabel 4850 4950 0    50   Input ~ 0
-Servo_6_PWM
-Text HLabel 4850 5550 0    50   Input ~ 0
-Servo_7_PWM
-Text HLabel 4850 6150 0    50   Input ~ 0
-Servo_8_PWM
-Wire Wire Line
-	5600 6150 4850 6150
-Wire Wire Line
-	5600 5550 4850 5550
-Wire Wire Line
-	5600 4950 4850 4950
-Wire Wire Line
-	5600 4350 4850 4350
-Wire Wire Line
-	5600 3750 4850 3750
-Wire Wire Line
-	5600 3150 4850 3150
-Wire Wire Line
-	5600 2550 4850 2550
-Wire Wire Line
-	5600 1950 4850 1950
-Text HLabel 5150 1500 1    50   Input ~ 0
-+5VA
-Wire Wire Line
-	5000 6050 5000 6450
-Text HLabel 5000 6450 3    50   Input ~ 0
-GND
-Text Notes 4550 1000 0    79   ~ 0
-Molex SL Connectors
-Connection ~ 5000 6050
-Wire Wire Line
-	5150 1500 5150 1750
-Connection ~ 5150 1750
+$Comp
+L MRDT_Connectors:Molex_uF_D_06 Conn10
+U 1 1 61A57BF2
+P 7000 2600
+F 0 "Conn10" H 7128 3158 60  0000 L CNN
+F 1 "Molex_uF_D_06" H 7128 3052 60  0000 L CNN
+F 2 "MRDT_Connectors:MOLEX_uF_D_06_Horizontal" H 7000 2900 60  0001 C CNN
+F 3 "" H 7000 2900 60  0001 C CNN
+	1    7000 2600
+	1    0    0    -1
+$EndComp
+$Comp
+L MRDT_Connectors:Molex_uF_D_06 Conn11
+U 1 1 61A58E08
+P 7000 3400
+F 0 "Conn11" H 7128 3958 60  0000 L CNN
+F 1 "Molex_uF_D_06" H 7128 3852 60  0000 L CNN
+F 2 "MRDT_Connectors:MOLEX_uF_D_06_Horizontal" H 7000 3700 60  0001 C CNN
+F 3 "" H 7000 3700 60  0001 C CNN
+	1    7000 3400
+	1    0    0    -1
+$EndComp
+$Comp
+L MRDT_Connectors:Molex_uF_D_06 Conn12
+U 1 1 61A5BF21
+P 7050 4200
+F 0 "Conn12" H 7178 4758 60  0000 L CNN
+F 1 "Molex_uF_D_06" H 7178 4652 60  0000 L CNN
+F 2 "MRDT_Connectors:MOLEX_uF_D_06_Horizontal" H 7050 4500 60  0001 C CNN
+F 3 "" H 7050 4500 60  0001 C CNN
+	1    7050 4200
+	1    0    0    -1
+$EndComp
+$Comp
+L MRDT_Connectors:Molex_uF_D_06 Conn13
+U 1 1 61A5F2E6
+P 7050 5000
+F 0 "Conn13" H 7178 5558 60  0000 L CNN
+F 1 "Molex_uF_D_06" H 7178 5452 60  0000 L CNN
+F 2 "MRDT_Connectors:MOLEX_uF_D_06_Horizontal" H 7050 5300 60  0001 C CNN
+F 3 "" H 7050 5300 60  0001 C CNN
+	1    7050 5000
+	1    0    0    -1
+$EndComp
 $EndSCHEMATC
