File: Hardware/Gimbal_Board_2023.kicad_pcb (KiCad board)
At the start: 2 copper layers, 115.1 x 84.8 mm, 74 parts, among them J1 6P6C, J2 RJ45_LED_Shielded, Q1 Q_NMOS_GDS, Q2 Q_NMOS_GDS, Q3 Q_NMOS_GDS, Q4 Q_NMOS_GDS, Q5 Q_NMOS_GDS, Q6 Q_NMOS_GDS, Q7 Q_NMOS_GDS, SW1 SW_Push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

Commit message: Redid header
Parts:
- moved G*** 1.73 mm to (84.4, 95.3)
Other:
- board text added: "Gimbal Board, Rev 1 Mars Rover Design Team Missouri S&T, 2023 Tyler Nguyen, Aden Standefer"
- board text removed: "Gimbal Board, 2023 Rev 1 Mars Rover Design Team Tyler Nguyen & Aden Standefer"
Changed lines of the file:
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@@
   )
   (footprint "Gimbal_Board_Library:z-sig-Tyler-Nguyen" (layer "F.Cu")
-    (at 83.566 93.795406)
+    (at 84.384432 95.319406)
     (attr board_only exclude_from_pos_files exclude_from_bom)
     (fp_text reference "G***" (at 0 0) (layer "F.SilkS")
@@
     (effects (font (size 1.524 1.524) (thickness 0.254)))
   )
-  (gr_text "Gimbal Board, 2023 Rev 1\nMars Rover Design Team\nTyler Nguyen & Aden Standefer" (at 84.836 84.328) (layer "F.SilkS")
+  (gr_text "Gimbal Board, Rev 1\nMars Rover Design Team\nMissouri S&T,  2023\nTyler Nguyen, Aden Standefer" (at 84.836 84.328) (layer "F.SilkS")
     (effects (font (size 1.5 1.5) (thickness 0.3)))
   )

Commit message: redrew edgecuts and finished board
Routing:
- net +3.3V: track 218.3 -> 216.4 mm
- net Servo_3_PWM: track 28.7 -> 28.6 mm, vias 1 -> 2
- net Servo_1_SW: vias 4 -> 2
- net GND: vias 1 -> 9
Other:
- board size 115.1 x 84.8 mm -> 112 x 81.8 mm
